File: proj/light_controller/v1.0/light_controller.brd (EAGLE design)
At the start: 101.6 x 85.1 mm, 112 parts, among them J1 0022232051, U1 RCD-24-0.70, U10 ADM2481BRWZ-RL7, U11 DAC5578SPW, U12 CY8C4124PVI-432, U13 PHOTONH, U2 RCD-24-0.70, U3 RCD-24-0.70, U4 RCD-24-0.70, U5 RCD-24-0.70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

Commit message: initial design changes for light controller v1.1
Other:
- board text removed: "Light Controller v1 MIT OpenAg This board controls x6, 24V LED channels up to 700mA each. It has a dedicated microcontroller (PSOC 4100) with optional headers for a Particle Photon. We are believers in the power of open source hardware / software to make future food production systems accessible to all. Being so, we freely share all hardware design files and supporting software on our GitHub (Ope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"
Changed lines of the file:
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@@
 <?xml version="1.0" encoding="utf-8"?>
 <!DOCTYPE eagle SYSTEM "eagle.dtd">
-<eagle version="8.4.1">
+<eagle version="8.4.3">
 <drawing>
 <settings>
@@
 <text x="98.552" y="44.704" size="1.27" layer="21" rot="R90">Light Controller v1
 MIT OpenAg</text>
-<text x="99.06" y="9.398" size="1.27" layer="22" rot="MR0">Light Controller v1
-MIT OpenAg
-This board controls x6, 24V LED channels up to 700mA each. It has a dedicated
-microcontroller (PSOC 4100) with optional headers for a Particle Photon.
-We are believers in the power of open source hardware / software to make
-future food production systems accessible to all. Being so, we freely share all
-hardware design files and supporting software on our GitHub (OpenAgInitiative).
-The design files for this board are located in the following GitHub repository:
-    https://github.com/OpenAgInitiative/openag_light_controller
-All boards we develop exclusively utilize parts from our eagle parts library. We
-do this to maximize component reuse and ensure part verification.
-The OpenAg eagle library is located in the following GitHub repository:
-    https://github.com/OpenAgInitiative/openag_eagle_library
-Whenever possible, we strive to create re-usable and modular elements throughout all of our designs.
-The OpenAg eagle design blocks are located in the following GitHub repository:
-    https://github.com/OpenAgInitiative/openag_eagle_design_blocks
-We are always looking for more collaborators aligned with our ideologies! Want
-to get involved?
-    Join the forum: http://forum.openag.media.mit.edu/
-    Visit the wiki: https://wiki.openag.media.mit.edu/
-</text>
 </plain>
 <attributes>
@@
 <attribute name="NAME" x="91.186" y="56.642" size="0.635" layer="25"/>
 <attribute name="POPULATE" value="YES" x="91.567" y="54.991" size="1.778" layer="27" rot="R270" display="off"/>
+<attribute name="VALUE" value="330pF" x="91.567" y="54.991" size="1.778" layer="27" rot="R270" display="off"/>
 <attribute name="VALUE" x="89.662" y="55.626" size="1.27" layer="27" rot="R270"/>
-<attribute name="VALUE" value="330pF" x="91.567" y="54.991" size="1.778" layer="27" rot="R270" display="off"/>
 <attribute name="VERIFIED" value="NO" x="91.567" y="54.991" size="1.778" layer="27" rot="R270" display="off"/>
 </element>
