File: proj/light_controller/v1.1 - Copy/light_controller.brd (EAGLE design)
At the start: 127 x 127 mm, 119 parts, among them J1 0022232051, J2 RJ12, J3 RJ12, J4 1377G2, J5 RJ12, J6 RJ12, U1 RCD-24-0.70/VREF, U10 ADM2481BRWZ-RL7, U11 PHOTONH, U12 TLV70433DBVR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

Commit message: pushing to avoid any loss of work
Parts:
- added J7: OPENAG-I2C-HEADER, openag-connectors:OPENAG-I2C-HEADER
- moved R56 120.7 mm to (145.7, 80.8)
- moved R60 120.7 mm to (155.8, 80.8)
- moved SJ_A1 120.7 mm to (155.8, 85.7)
- moved SJ_A5 120.7 mm to (145.7, 85.7)
- moved R57 120.7 mm to (148.2, 80.8)
- moved R61 120.7 mm to (158.4, 80.8)
- moved SJ_A0 120.7 mm to (158.4, 85.7)
- moved SJ_A4 120.7 mm to (148.2, 85.7)
- moved R58 120.7 mm to (150.7, 80.8)
- moved R59 120.7 mm to (153.3, 80.8)
- moved SJ_A2 120.7 mm to (153.3, 85.7)
- moved SJ_A3 120.7 mm to (150.7, 85.7)
- moved C21 116.2 mm to (-7.62, -21.6)
- moved R28 102.7 mm to (-6.86, -13.5), turned to 0 degrees
- moved R29 102.3 mm to (-6.86, -16.3)
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Connections:
- new net VCC: C21.1, SJ_A0.1, SJ_A1.1, SJ_A2.1, SJ_A3.1, SJ_A4.1, SJ_A5.1, U14.28
- net +3V3: no longer C21.1, SJ_A0.1, SJ_A1.1, SJ_A2.1, SJ_A3.1, SJ_A4.1, SJ_A5.1, U14.28
- net 485_5V: no longer J6.2
- net 485_A: no longer J6.3
- net 485_B: no longer J6.4
- net 485_GND: no longer J6.1, J6.6
- net DIM1: now also U7.4; no longer U7.7
- net DIM2: now also U7.5; no longer U7.6
- net DIM3: now also U7.6; no longer U7.5
- net DIM4: now also U7.7; no longer U7.4
- net I2C_3V3: now also J6.5, J7.3V3
- net I2C_GND: now also J6.1, J7.GND
- net I2C_IO: now also J6.2
- net I2C_SCL: now also J6.3, J7.SCL
- net I2C_SDA: now also J6.4, J7.SDA
- net PWM1: now also U14.7; no longer U14.12
- net PWM2: now also U14.8; no longer U14.11
- net PWM3: now also U14.9; no longer U14.10
- net PWM4: now also U14.10; no longer U14.9
- net PWM5: now also U14.11; no longer U14.8
- net PWM6: now also U14.12; no longer U14.7
Routing:
- net PWM6: track 166.3 -> 0.00 mm
- net PWM5: track 148.3 -> 0.00 mm
- net PHOTON_SCL: track 0.00 -> 135.2 mm
- net PHOTON_SDA: track 0.00 -> 131.7 mm
- net PWM4: track 130.2 -> 0.00 mm
- net PHOTON_TX: track 0.10 -> 120.4 mm
- net PHOTON_RX: track 0.00 -> 118.0 mm
- net PWM3: track 112.2 -> 0.00 mm
- net PHOTON_A0: track 0.00 -> 106.3 mm
- net DIM3: track 137.9 -> 39.6 mm, vias 1 -> 2
- net DIM2: track 156.6 -> 58.9 mm, vias 1 -> 2
- net DIM1: track 175.5 -> 79.0 mm, vias 1 -> 2
- net PWM2: track 94.1 -> 0.00 mm
- net DIM4: track 118.9 -> 32.8 mm, vias 1 -> 2
- net PWM1: track 79.8 -> 0.00 mm
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- removed copper zone on layer 1, net +3V3
- removed copper zone on layer 1, net DAC_!CLR!
- removed copper zone on layer 1, net REG_3V3
- removed copper zone on layer 1, net SCL
- removed copper zone on layer 1, net SDA
Other:
- board size 127 x 127 mm -> 114.3 x 114.3 mm
- board text added: "PCA9685"
- board text added: "Use V+ for servo supply"
- board text removed: "24V / GND Anderson Powerpole Connector"
- board text removed: "24V-to-3.3V Regulator"
- board text removed: "3.3V"
- board text removed: "6-Channel 24V, 700mA (per channel) Current Regulator Module w/I2C Controlled Dimming via PWM or Analog Signaling"
- board text removed: "CLR"
- board text removed: "EDGE"
- board text removed: "NC"
- board text removed: "SCL"
- board text removed: "SDA"
