File: proj/edu_brain/v1.0/edu_brain.brd (EAGLE design)
At the start: 50.9 x 31.8 mm, 5 parts

Commit message: sent light controller v1.1 to fab house
Parts:
- added U$5: (no value), openag-valves:UMBRELLA-VALVE-21.5MM
- added U1: BEAGLEBONE_OUTLINE, openag-microcontrollers:BEAGLEBONE_SHIELD
- moved U$3 355.0 mm to (288.3, 288.3)
- moved U$2 287.7 mm to (3.81, 288.3), turned to 270 degrees
- moved U$4 285.5 mm to (288.3, 3.81), turned to 90 degrees
- moved FRAME1 203.6 mm to (247.7, 19.1), flipped to the top
Connections:
- new net AIN0: U1.85
- new net GND: U1.1, U1.2, U1.47, U1.48, U1.89, U1.90, U1.91, U1.92
- new net SYS_5V: U1.53
- new net VDD_3V3EXP: U1.49, U1.50
- new net VDD_5V: U1.51, U1.52
Other:
- board size 50.9 x 31.8 mm -> 292.1 x 292.1 mm
- board text added: "LIGHT"
