File: proj/edu_brain/v1.0/edu_brain.sch (EAGLE design)
At the start: 120 parts, among them J1 0022232051, J2 RJ12, J3 RJ12, J4 1377G2, J5 RJ12, J6 RJ12, J7 OPENAG-I2C-HEADER, U1 RCD-24-0.70/VREF, U10 ADM2481BRWZ-RL7, U11 PHOTONH, U12 TLV70433DBVR, U14 PCA9685, U2 RCD-24-0.70/VREF, U3 RCD-24-0.70/VREF, U4 RCD-24-0.70/VREF, U5 RCD-24-0.70/VREF, U6 RCD-24-0.70/VREF, U7 DAC5578SPW, U8 ISO1540DR, U9 CY8C4124PVI-432

Commit message: sent light controller v1.1 to fab house
Parts:
- removed C1, C10, C11, C13, C14, C16, C17, C2, C4, C5, C7, C8: 10nF, openag-capacitors:10NF-C0603C103K5RACTU
- removed C12, C15, C18, C3, C6, C9: 100uF, openag-capacitors:100UF-EEE-1HA101UP
- removed C19, C26, C27, C28, C30, C31, C38: 0.1uF, openag-capacitors:0.1UF-C0603C104K5RACTU
- removed C20, C32, C33: 1uF, openag-capacitors:1UF-CL10A105KB8NNNC
- removed C21, C24, C25, C36: 10uF, openag-capacitors:10UF-GMK212BBJ106KG-T
- removed C29, C34, C37: 4.7uF, openag-capacitors:4.7UF-CL21A475KBQNNNE
- removed CH1+, CH1-, CH2+, CH2-, CH3+, CH3-, CH4+, CH4-, CH5+, CH5-, CH6+, CH6-: (no value), openag-wirepads:3,17/1,3
- removed CR2: SMAJ26A-13-F, openag-diodes:SMAJ26A-13-F
- removed D1: APT1608CGCK, openag-diodes:APT1608CGCK
- removed F2: SST 7, openag-fuses:SST_7
- removed J1: 0022232051, openag-connectors:MINI-PROG3-5POS-MATING-CONNECTOR
- removed J2, J3, J5, J6: RJ12, openag-connectors:A-2004-1-4-LP-N-R
- removed J4: 1377G2, openag-connectors:1377G21377G2
- removed J7: OPENAG-I2C-HEADER, openag-connectors:OPENAG-I2C-HEADER
- removed L1, L2, L3, L4, L5, L6: 120uH, openag-inductors:120UH-74404064121
- removed R1, R15, R16, R17, R18, R19, R2, R20, R21, R22, R23, R24, R25, R3, R4, R5: 0 OHM, openag-resistors:0OHM-RC0603JR-070RL
- removed R10, R11, R12, R13, R14, R26, R28, R6, R7, R8, R9: 1K, openag-resistors:1K-ERJ-PB3D1001V
- removed R27: 100 OHM, openag-resistors:100OHM-RC0603JR-07100RL
- removed R29: 3.9K, openag-resistors:3.9K-RC0603JR-073K9L
- removed R56, R57, R58, R59, R60, R61, R62: 10K, openag-resistors:10K-ERJ-3EKF1002V
- removed SJ_A0, SJ_A1, SJ_A2, SJ_A3, SJ_A4, SJ_A5: (no value), openag-connectors:SOLDERJUMPERREFLOW_NOPASTE
- removed SW1: (no value), openag-switches:BF3-1020
- removed U10: ADM2481BRWZ-RL7, openag-isolators:ADM2481BRWZ-RL7
- removed U11: PHOTONH, openag-microcontrollers:PHOTONHPHOTONH
- removed U12: TLV70433DBVR, openag-regulators:TLV70433DBVRDBV5-M
- removed U14: PCA9685, openag-pwm:PCA9685PW/Q900,118
- removed U2, U3, U4, U5, U6: RCD-24-0.70/VREF, openag-regulators:RCD-24-0.70/VREF
- removed U7: DAC5578SPW, openag-dacs:DAC5578SPW
- removed U8: ISO1540DR, openag-isolators:ISO1540DR
- removed U9: CY8C4124PVI-432, openag-microcontrollers:CY8C4124PVI-432
- FRAME1: DESCRIPTION (none) -> Top Brain for PFC-EDU; TITLE Light Controller -> EDU Brain; URL https://github.com/OpenAgInitiative/openag_eagle/proj/light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 -> https://github.com/OpenAgInitiative/openag_eagle/proj/edu_b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; VER 1.1 -> (none)
- U1: value RCD-24-0.70/VREF -> BEAGLEBONE_OUTLINE; device openag-regulators:RCD-24-0.70/VREF -> openag-microcontrollers:BEAGLEBONE_OUTLINE
Connections:
- removed net +24V: C12.1(+), C15.1(+), C18.1(+), C19.1, C3.1(+), C36.1, C37.1, C38.1, C6.1(+), C9.1(+), CR2.P$2, F2.2, L1.1, L2.1, L3.1, L4.1, L5.1, L6.1, U12.IN
- removed net +3V3: C25.1, C27.1, C28.1, C29.1, R10.2, R11.2, R14.1, R17.2, R26.1, R27.2, R28.2, R3.1, R6.1, R7.1, R8.1, R9.1, SW1.P, U10.VDD1, U7.AVDD, U8.VCC2
- removed net 2.6V: R28.1, R29.2, U7.VREF_IN
- removed net 24V_IN: F2.1, J4.V+
- removed net 485_5V: C26.1, J5.2, U10.VDD2
- removed net 485_A: J5.3, U10.A
- removed net 485_B: J5.4, U10.B
- removed net 485_GND: C26.2, J5.1, J5.6, U10.GND2
- removed net A0: R61.2, SJ_A0.2, U14.A0
- removed net A1: R60.2, SJ_A1.2, U14.A1
- removed net A2: R59.2, SJ_A2.2, U14.A2
- removed net A3: R58.2, SJ_A3.2, U14.A3
- removed net A4: R57.2, SJ_A4.2, U14.A4
- removed net A5: R56.2, SJ_A5.2, U14.A5
- removed net CH1+: CH1+.P, U1.+VOUT
- removed net CH1-: C2.1, CH1-.P, U1.-VOUT
- removed net CH2+: CH2+.P, U2.+VOUT
- removed net CH2-: C5.1, CH2-.P, U2.-VOUT
- removed net CH3+: CH3+.P, U3.+VOUT
- removed net CH3-: C8.1, CH3-.P, U3.-VOUT
- removed net CH4+: CH4+.P, U4.+VOUT
- removed net CH4-: C11.1, CH4-.P, U4.-VOUT
- removed net CH5+: CH5+.P, U5.+VOUT
- removed net CH5-: C14.1, CH5-.P, U5.-VOUT
- removed net CH6+: CH6+.P, U6.+VOUT
- removed net CH6-: C17.1, CH6-.P, U6.-VOUT
- removed net DAC_!CLR!: R24.2, R25.2, SW1.S, U7.!CLR!
- removed net DIM1: R6.2, U1.ANALOGUE_DIM, U7.VOUT_A
- removed net DIM2: R7.2, U2.ANALOGUE_DIM, U7.VOUT_C
- removed net DIM3: R8.2, U3.ANALOGUE_DIM, U7.VOUT_E
- removed net DIM4: R9.2, U4.ANALOGUE_DIM, U7.VOUT_G
- removed net DIM5: R14.2, U5.ANALOGUE_DIM, U7.VOUT_H
- removed net DIM6: R26.2, U6.ANALOGUE_DIM, U7.VOUT_F
- removed net GND: C1.2, C10.2, C11.2, C12.2(-), C13.2, C14.2, C15.2(-), C16.2, C17.2, C18.2(-), C19.2, C2.2, C20.2, C21.2, C25.2, C27.2, C28.2, C29.2, C3.2(-), C30.2, C31.2, C32.2, C33.2, C34.2, C36.2, C37.2, C38.2, C4.2, C5.2, C6.2(-), C7.2, C8.2, C9.2(-), CR2.P$1, D1.C, J1.GND, J4.GND, R29.1, R56.1, R57.1, R58.1, R59.1, R60.1, R61.1, R62.2, U1.GND, U10.GND1, U11.GND@2, U11.GND@21, U12.GND, U14.EXTCLK, U14.GND, U2.GND, U3.GND, U4.GND, U5.GND, U6.GND, U7.!LDAC!, U7.GND, U8.GND2, U9.VSS
- removed net I2C_3V3: C24.1, J2.5, J3.5, J6.5, J7.3V3, R12.2, R13.2, U8.VCC1
- removed net I2C_GND: C24.2, J2.1, J3.1, J6.1, J7.GND, U8.GND1
- removed net I2C_IO: J2.2, J3.2, J6.2
- removed net I2C_SCL: J2.3, J3.3, J6.3, J7.SCL, R12.1, U8.SCL1
- removed net I2C_SDA: J2.4, J3.4, J6.4, J7.SDA, R13.1, U8.SDA1
- removed net N$1: C1.1, L1.2, U1.+VIN
- removed net N$2: C4.1, L2.2, U2.+VIN
- removed net N$23: C33.1, U9.VCCD
- removed net N$3: D1.A, R27.1
- removed net N$4: C7.1, L3.2, U3.+VIN
- removed net N$5: C10.1, L4.2, U4.+VIN
- removed net N$6: C13.1, L5.2, U5.+VIN
- removed net N$7: C16.1, L6.2, U6.+VIN
- removed net N$8: C30.1, C34.1, R17.1, U11.3V3
- removed net OE: R62.1, U14.#OE
- removed net P0[7]: R25.1, U9.P0[7]
- removed net P2[6]: R20.1, U9.P2[6]
- removed net P2[7]: R21.1, U9.P2[7]
- removed net PHOTON_A0: R24.1, U11.A0
- removed net PHOTON_D2: R23.1, U11.D2
- removed net PHOTON_D3: R22.1, U11.D3
- removed net PHOTON_D4: U11.D4
- removed net PHOTON_RX: R18.1, U11.RX
- removed net PHOTON_SCL: R5.1, U11.D1
- removed net PHOTON_SDA: R4.1, U11.D0
- removed net PHOTON_TX: R19.1, U11.TX
- removed net PWM1: U1.PWM/ON/OFF, U14.PWM1
- removed net PWM2: U14.PWM2, U2.PWM/ON/OFF
- removed net PWM3: U14.PWM3, U3.PWM/ON/OFF
- removed net PWM4: U14.PWM4, U4.PWM/ON/OFF
- removed net PWM5: U14.PWM5, U5.PWM/ON/OFF
- removed net PWM6: U14.PWM6, U6.PWM/ON/OFF
- removed net REG_3V3: C20.1, U12.OUT
- removed net SCB0_I2C_SCL: R2.1, U9.P4[0]
- removed net SCB0_I2C_SDA: R1.1, U9.P4[1]
- removed net SCB1_RX[0]: R15.1, U9.P3[0]
- removed net SCB1_TX[0]: R16.1, U9.P3[1]
- removed net SCL: R10.1, R2.2, R5.2, U14.SCL, U7.SCL, U8.SCL2
- removed net SDA: R1.2, R11.1, R4.2, U14.SDA, U7.SDA, U8.SDA2
- removed net SWD_CLK[0]: J1.SCLK, U9.P3[3]
- removed net SWD_IO[0]: J1.SDAT, U9.P3[2]
- removed net UART_!RE!: R21.2, R23.2, U10.!RE!
- removed net UART_DE: R20.2, R22.2, U10.DE
- removed net UART_RX: R15.2, R18.2, U10.RXD
- removed net UART_TX: R16.2, R19.2, U10.TXD
- removed net VCC: C21.1, SJ_A0.1, SJ_A1.1, SJ_A2.1, SJ_A3.1, SJ_A4.1, SJ_A5.1, U14.VDD
- removed net VDDD: C31.1, C32.1, J1.VTARG, R3.2, U9.VDDD
- removed net XRES: J1.XRES, U9.XRES
Other:
- note removed: "1 + A5 + A4 + A3 + A2 + A1 +A1 + RW"
- note removed: "24V Power Conditioning"
- note removed: "24V Powerpole Connector"
- note removed: "24V-0.7A Current Regulators"
- note removed: "3.3V Indicator LED"
- note removed: "3.3V Interrupt Switch"
- note removed: "3.3V, 150mA Linear Regulator"
- note removed: "I2C Address ="
- note removed: "I2C Header Connector"
- note removed: "I2C Isolator"
- note removed: "I2C to 8-Channel 8-Bit DAC"
- note removed: "Notes: - GND !LDAC! for syncronous mode - Broadcast I2C Addr = 0x47 - ADDR0=Low, I2C Addr=0x48 - ADDR0=High, I2C Addr=0x4A - ADDR0=Float, I2C Addr=0x4C"
- note removed: "Open = 0 / Closed = 1"
- note removed: "PCA9685 16-Channel I2C DAC"
- note removed: "PSOC 4100 Microcontroller"
- note removed: "PSOC 4100 Programming Header"
- note removed: "Photon Microcontroller"
- note removed: "RJ12 Connectors"
- note removed: "RS485 Isolator"
