File: proj/light_controller/v1.1/light_controller.sch (EAGLE design)
At the start: 119 parts, among them J1 0022232051, J2 RJ12, J3 RJ12, J4 1377G2, J5 RJ12, J6 RJ12, U1 RCD-24-0.70/VREF, U10 ADM2481BRWZ-RL7, U11 PHOTONH, U12 TLV70433DBVR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

Commit message: explored new modularity concept for light controller
Parts:
- added R30, R31, R32, R33: 0 OHM, openag-resistors:0OHM-RC0603JR-070RL
Connections:
- net I2C_SCL renamed SCL1
- net I2C_SDA renamed SDA1
- removed net SCB1_RX[0]: R15.1, U9.P3[0]
- removed net SCB1_TX[0]: R16.1, U9.P3[1]
- new net SCB1_RX[0]_SCL[0]: R15.1, R31.1, U9.P3[0]
- new net SCB1_TX[0]_SDA[0]: R16.1, R30.1, U9.P3[1]
- new net SCL2: R10.1, R31.2, R33.1, U8.SCL2
- new net SDA2: R11.1, R30.2, R32.1, U8.SDA2
- net PHOTON_D2: now also R22.1; no longer R23.1
- net PHOTON_D3: now also R23.1; no longer R22.1
- net SCL: now also R33.2; no longer R10.1, U8.SCL2
- net SDA: now also R32.2; no longer R11.1, U8.SDA2
Other:
- note added: "PCA9685 16-Channel I2C PWM Driver"
- note removed: "PCA9685 16-Channel I2C DAC"
- moved on the sheet: C24, C25, C31, C32, C33, R1, R10, R11, R12, R13, R15, R16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

Commit message: majority of design changes done for light controller v1.1
Parts:
- added J7: OPENAG-I2C-HEADER, openag-connectors:OPENAG-I2C-HEADER
- added J8: JUMPER, openag-connectors:100-MIL-HEADER-JUMPER
- J2, J3, J5, J6: value RJ12 -> A-2004-1-4-LP-N-R
- SW1: value (none) -> BF3-1020
Connections:
- net +3V3: now also J8.2
- net I2C_3V3: now also J7.3V3
- net I2C_GND: now also J7.GND
- net REG_3V3: now also J8.1
- net SCL1: now also J7.SCL
- net SDA1: now also J7.SDA
Other:
- note added: "24V / GND Anderson Powerpole Connector"
- note added: "24V-to-3.3V Regulator w/3v3 Enable Jumper"
- note added: "3.3V Interrupt Jumper"
- note added: "6-Channel 24V, 700mA (per channel) Current Regulator Module w/I2C Controlled Dimming via PWM or Analog Signaling"
- note added: "Changelog: - adjusted RS485 IC has footprint - adjusted CH5 LED connections label - updated 1uf capacitor package - added pullups to dimmer driver - added fancy openag logo - added rj12 connectors for i2c and rs485 - added powerpole power connector - replaced 10uf w/10nf caps on dimmer circuit - added power status leds - added pushbutton to clear dacs - added linear 3v3 regulator - adjusted curre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"
- note added: "I2C Connector Pair w/Isolation and Inter-I2C Connection Option"
- note added: "I2C Header"
- note added: "Inter-I2C Connect Option"
- note added: "PSOC4100 Microcontroller w/Optional Dual Channel I2C and/or RS485 Connections"
- note added: "Photon w/Optional I2C + RS485 Connections"
- note added: "RS485 Connection Pair w/UART Transceiver"
- note removed: "3.3V Interrupt Switch"
- moved on the sheet: C1, C10, C11, C12, C13, C14, C15, C16, C17, C18, C19, C2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

Commit message: sent light controller v1.1 to fab house
Parts:
- FRAME1: DESCRIPTION (none) -> Controls 6 channels of 24V, 700mA for LED strings that can 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
- J2, J3: value A-2004-1-4-LP-N-R -> OPENAG-I2C-RJ12; device openag-connectors:A-2004-1-4-LP-N-R -> openag-connectors:OPENAG-I2C-RJ12
- J5, J6: value A-2004-1-4-LP-N-R -> OPENAG-RS485-RJ12; device openag-connectors:A-2004-1-4-LP-N-R -> openag-connectors:OPENAG-RS485-RJ12
Changed lines of the file:
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@@
 <layer number="1" name="Top" color="4" fill="1" visible="no" active="no"/>
 <layer number="2" name="Route2" color="1" fill="3" visible="no" active="no"/>
+<layer number="3" name="Route3" color="4" fill="3" visible="no" active="no"/>
+<layer number="4" name="Route4" color="1" fill="4" visible="no" active="no"/>
+<layer number="5" name="Route5" color="4" fill="4" visible="no" active="no"/>
+<layer number="6" name="Route6" color="1" fill="8" visible="no" active="no"/>
+<layer number="7" name="Route7" color="4" fill="8" visible="no" active="no"/>
+<layer number="8" name="Route8" color="1" fill="2" visible="no" active="no"/>
+<layer number="9" name="Route9" color="4" fill="2" visible="no" active="no"/>
+<layer number="10" name="Route10" color="1" fill="7" visible="no" active="no"/>
+<layer number="11" name="Route11" color="4" fill="7" visible="no" active="no"/>
+<layer number="12" name="Route12" color="1" fill="5" visible="no" active="no"/>
+<layer number="13" name="Route13" color="4" fill="5" visible="no" active="no"/>
+<layer number="14" name="Route14" color="1" fill="6" visible="no" active="no"/>
 <layer number="15" name="Route15" color="4" fill="6" visible="no" active="no"/>
 <layer number="16" name="Bottom" color="1" fill="1" visible="no" active="no"/>
@@
 <part name="FRAME1" library="openag-frames" deviceset="DOCFIELD" device="">
 <attribute name="AUTHOR" value="JR"/>
-<attribute name="DESCRIPTION" value=""/>
+<attribute name="DESCRIPTION" value="Controls 6 channels of 24V, 700mA for LED strings that can be interfaced via i2c, rs485, and/or wifi."/>
 <attribute name="TITLE" value="Light Controller"/>
 <attribute name="URL" value="https://github.com/OpenAgInitiative/openag_eagle/proj/light_controller"/>
 <attribute name="VER" value="1.1"/>
 </part>
-<part name="J2" library="openag-connectors" deviceset="A-2004-1-4-LP-N-R" device="" value="A-2004-1-4-LP-N-R"/>
-<part name="J3" library="openag-connectors" deviceset="A-2004-1-4-LP-N-R" device="" value="A-2004-1-4-LP-N-R"/>
+<part name="J2" library="openag-connectors" deviceset="OPENAG-I2C-RJ12" device="" value="OPENAG-I2C-RJ12"/>
+<part name="J3" library="openag-connectors" deviceset="OPENAG-I2C-RJ12" device="" value="OPENAG-I2C-RJ12"/>
 <part name="J4" library="openag-connectors" deviceset="1377G2" device="1377G2" value="1377G2"/>
 <part name="GND10" library="openag-supply" deviceset="GND" device=""/>
@@
 <part name="R26" library="openag-resistors" deviceset="1K-ERJ-PB3D1001V" device="" value="1K"/>
 <part name="+3V1" library="openag-supply" deviceset="+3V3" device=""/>
-<part name="J5" library="openag-connectors" deviceset="A-2004-1-4-LP-N-R" device="" value="A-2004-1-4-LP-N-R"/>
+<part name="J5" library="openag-connectors" deviceset="OPENAG-RS485-RJ12" device="" value="OPENAG-RS485-RJ12"/>
 <part name="D1" library="openag-diodes" deviceset="APT1608CGCK" device="" value="APT1608CGCK"/>
 <part name="R27" library="openag-resistors" deviceset="100OHM-RC0603JR-07100RL" device="" value="100 OHM"/>
@@
 <part name="+3V10" library="openag-supply" deviceset="+3V3" device=""/>
 <part name="+3V11" library="openag-supply" deviceset="+3V3" device=""/>
-<part name="J6" library="openag-connectors" deviceset="A-2004-1-4-LP-N-R" device="" value="A-2004-1-4-LP-N-R"/>
+<part name="J6" library="openag-connectors" deviceset="OPENAG-RS485-RJ12" device="" value="OPENAG-RS485-RJ12"/>
 <part name="R30" library="openag-resistors" deviceset="0OHM-RC0603JR-070RL" device="" value="0 OHM"/>
 <part name="R31" library="openag-resistors" deviceset="0OHM-RC0603JR-070RL" device="" value="0 OHM"/>
@@
 <instance part="J2" gate="G$1" x="-17.78" y="591.82" smashed="yes">
 <attribute name="NAME" x="-27.432" y="601.472" size="1.27" layer="95"/>
-<attribute name="VALUE" x="-22.86" y="574.548" size="1.27" layer="96"/>
 </instance>
 <instance part="J3" gate="G$1" x="-50.8" y="591.82" smashed="yes">
 <attribute name="NAME" x="-60.452" y="601.726" size="1.27" layer="95"/>
-<attribute name="VALUE" x="-55.88" y="574.548" size="1.27" layer="96"/>
 </instance>
 <instance part="J4" gate="G$1" x="271.78" y="586.74"/>
@@
 <instance part="J5" gate="G$1" x="172.72" y="591.82" smashed="yes">
 <attribute name="NAME" x="162.814" y="601.726" size="1.27" layer="95"/>
-<attribute name="VALUE" x="167.64" y="574.04" size="1.27" layer="96"/>
 </instance>
 <instance part="D1" gate="G$1" x="106.68" y="393.7" rot="R270"/>
@@
 <instance part="J6" gate="G$1" x="139.7" y="591.82" smashed="yes">
 <attribute name="NAME" x="129.794" y="601.726" size="1.27" layer="95"/>
-<attribute name="VALUE" x="134.62" y="574.04" size="1.27" layer="96"/>
 </instance>
 <instance part="R30" gate="G$1" x="-213.36" y="548.64"/>
