File: proj/modules/24V_to_ADJ_1A_switching_regulator/24V_to_1V8_1A_switching_regulator/24V_to_1V8_1A_switching_regulator.brd (EAGLE design)
At the start: 10 parts, among them U1 MIC4680YM-TR

Commit message: cleaned up values and added 1.8V and 3.3V output options
Parts:
- R2: value 976 Ohm -> 6.49K
Other:
- board text added: "24V-to-3V3@1A Switching Regulator w/Indicator LED + Enable"
- board text removed: "24V-to-5V@1A Switching Regulator w/Indicator LED + Enable"
Changed lines of the file:
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@@
 <wire x1="0.635" y1="17.145" x2="6.0325" y2="17.145" width="0.1524" layer="21" style="shortdash"/>
 <wire x1="7.9375" y1="17.145" x2="18.415" y2="17.145" width="0.1524" layer="21" style="shortdash"/>
-<text x="0" y="18.288" size="0.762" layer="21">24V-to-5V@1A Switching Regulator w/Indicator LED + Enable</text>
+<text x="0" y="18.288" size="0.762" layer="21">24V-to-3V3@1A Switching Regulator w/Indicator LED + Enable</text>
 <text x="14.732" y="9.398" size="0.762" layer="21">Enable</text>
 <wire x1="14.224" y1="10.414" x2="18.288" y2="10.414" width="0.1524" layer="21"/>
@@
 </element>
 <element name="R1" library="openag-resistors" package="RC0603N" value="3.01K" x="26.416" y="7.62" rot="R90"/>
-<element name="R2" library="openag-resistors" package="RC0603N" value="976 Ohm" x="26.416" y="4.572" smashed="yes" rot="R90">
+<element name="R2" library="openag-resistors" package="RC0603N" value="6.49K" x="26.416" y="4.572" smashed="yes" rot="R90">
 <attribute name="NAME" x="25.5905" y="3.4417" size="0.762" layer="25" ratio="6" rot="SR90"/>
-<attribute name="VALUE" value="976 Ohm" x="27.94" y="3.048" size="0.762" layer="27" ratio="6" rot="R90"/>
+<attribute name="VALUE" value="6.49K" x="27.94" y="3.048" size="0.762" layer="27" ratio="6" rot="R90"/>
 </element>
 <element name="R3" library="openag-resistors" package="RC0603N" value="100 OHM" x="22.987" y="8.382" smashed="yes">
