File: proj/modules/24V_to_ADJ_1A_switching_regulator/24V_to_1V8_1A_switching_regulator/24V_to_1V8_1A_switching_regulator.sch (EAGLE design)
At the start: 10 parts, among them U1 MIC4680YM-TR

Commit message: cleaned up values and added 1.8V and 3.3V output options
Parts:
- R2: value 976 Ohm -> 6.49K; device openag-resistors:982OHM-RC0603FR-07976RL -> openag-resistors:6.49K-RC0603FR-076K49L
Other:
- note added: "24V to 3V3@1A Switching Regulator w/Indicator LED + Enable"
- note removed: "24V to 5V@1A Switching Regulator w/Indicator LED + Enable"
Changed lines of the file:
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@@
 <part name="D1" library="openag-diodes" deviceset="B260A-13-F" device="" value="B260A-13-F"/>
 <part name="R1" library="openag-resistors" deviceset="3.01K-RC0603FR-073K01L" device="" value="3.01K"/>
-<part name="R2" library="openag-resistors" deviceset="982OHM-RC0603FR-07976RL" device="" value="976 Ohm"/>
+<part name="R2" library="openag-resistors" deviceset="6.49K-RC0603FR-076K49L" device="" value="6.49K"/>
 <part name="GND1" library="openag-supply" deviceset="GND" device=""/>
 <part name="P+1" library="openag-supply" deviceset="+24V" device=""/>
@@
 <sheet>
 <plain>
-<text x="0" y="40.64" size="3.81" layer="97">24V to 5V@1A Switching Regulator
+<text x="0" y="40.64" size="3.81" layer="97">24V to 3V3@1A Switching Regulator
 w/Indicator LED + Enable</text>
 <wire x1="0" y1="38.1" x2="114.3" y2="38.1" width="0.254" layer="97"/>
