File: proj/nodes/t6713/v2.0/t6713.sch (EAGLE design)
At the start: 1 part

Commit message: cleaned up design blocks, added co2 sensor node v2.0
Parts:
- added C1, C4: 0.1uF, openag-capacitors:0.1UF-C0603C104K5RACTU
- added C2: 10uF, openag-capacitors:10UF-GMK212BBJ106KG-T
- added C3: 15uF, openag-capacitors:15UF-TPSD156K035R0100
- added C5: 220uF, openag-capacitors:220UF-TPSY227K010R0100
- added D2, D4: APT1608CGCK, openag-diodes:APT1608CGCK
- added D3: B260A-13-F, openag-diodes:B260A-13-F
- added F1: 0448.400MR, openag-fuses:0438.375WR
- added J3, J4: 54602-908LF, openag_connector:OPENAG-V1-RJ45PTH
- added L2: 68uH, openag-inductors:68UH-UP2B-680-R
- added R1, R8: 100 OHM, openag-resistors:100OHM-RC0603JR-07100RL
- added R16, R17, R18, R19, R20, R21, R22, R23: NV, openag-resistors:R0603
- added R2, R9: 0 OHM, openag-resistors:0OHM-RC0603JR-070RL
- added R3: 4.7K, openag-resistors:4.7K-RC1206JR-074K7L
- added R6: 3.01K, openag-resistors:3.01K-RC0603FR-073K01L
- added R7: 976 Ohm, openag-resistors:982OHM-RC0603FR-07976RL
- added U1: T6713-5K, openag-sensors:T6713-5K
- added U2: LM2937IMP3.3NOPB, openag-regulators:LM2937IMP-3.3/NOPB
- added U4: MIC4680YM-TR, openag-regulators:MIC4680YM-TR
- added U5: PCA9615DPJ, openag-buffers:PCA9615DPJ
- FRAME1: AUTHOR (none) -> JR; TITLE Example Template! -> T6713 Sensor Node; URL https://github.com/OpenAgInitiative/openag_eagle/proj/templ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 -> github.com/OpenAgInitiative/openag_eagle/proj/nodes; VER (none) -> 2.0
Connections:
- new net +24V: C3.1(+), J3.+24V, J4.+24V, U4.IN
- new net +3V3: C4.1, R2.2, R22.2, R23.2, R3.1, U1.V++, U5.VDD_(A)
- new net +5V: C1.1, R18.1, R19.2, R9.2, U2.IN, U5.VDD_(B)
- new net DSCLM: J3.DSCLM, J4.DSCLM, R20.2, R21.1, U5.DSCLM
- new net DSCLP: J3.DSCLP, J4.DSCLP, R19.1, R21.2, U5.DSCLP
- new net DSDAM: J3.DSDAM, J4.DSDAM, R16.1, R17.2, U5.DSDAM
- new net DSDAP: J3.DSDAP, J4.DSDAP, R17.1, R18.2, U5.DSDAP
- new net GND: C1.2, C2.2, C3.2(-), C4.2, C5.2(-), D2.C, D3.21, D4.C, J3.GND, J4.GND, R16.2, R20.1, R7.1, U1.CTRL/TEST, U1.GND, U2.GND, U4.GND, U4.SHDN, U5.VSS
- new net N$4: D3.12, L2.1, R6.1, R7.2, U4.FB, U4.SW
- new net N$6: D2.A, R1.1
- new net N$7: C2.1, F1.1, U2.OUT
- new net N$8: D4.A, R8.1
- new net N$9: C5.1(+), L2.2, R6.2, R8.2, R9.1
- new net REG_3V3_400MA: F1.2, R1.2, R2.1
- new net SCL: R23.1, R3.2, U1.RX/SCL, U5.SCL
- new net SDA: R22.1, U1.TX/SDA, U5.SDA
- new net USBM: J3.USBM, J4.USBM
- new net USBP: J3.USBP, J4.USBP
Other:
- note added: "24V to 5V@1A Switching Regulator w/Indicator LED + Enable"
- note added: "3.3V Enable Resistor"
- note added: "3.3V Indicator LED"
- note added: "3.3V, 400mA Regulator"
- note added: "5-26V to 3.3V@400mA Regulator w/3v3 Enable, Indicator LED & Fuse"
- note added: "Notes - See app note p.6 for i2c details - SDA has internal 4.7k pullup - SCL needs external 4.7k pullup - For I2C, ground pin 6 - I2C address default is 0x15"
- note added: "RJ45 Connector w/dI2C Buffer"
- note added: "RJ45 Connectors"
- note added: "T6713 CO2 Sensor"
- note added: "dI2C Buffer"
