File: proj/sensor-nodes/light/v1.0/light.sch (EAGLE design)
At the start: 48 parts, among them J1 54602-908LF, J2 54602-908LF, J3 OPENAG-I2C-RJ12, J4 OPENAG-I2C-RJ12, U2 PCA9615DPJ, U3 MIC4680YM-TR, U4 LM2937IMP3.3NOPB

Commit message: extracted design blocks from light controller
Parts:
- removed J3, J4: OPENAG-I2C-RJ12, openag-connectors:OPENAG-I2C-RJ12
- removed TP1, TP2, TP3, TP5: TPTP06R, openag-testpads:TPTP06R
- added C2, C7: 0.1uF, openag-capacitors:0.1UF-C0603C104K5RACTU
- added TP13, TP14, TP19, TP20, TP21, TP22, TP6, TP7: TPTP06R, openag-testpads:TPTP06R
- added U5: APDS-9250, openag-sensors:APDS-9250
- added U7: TSL2591, openag-sensors:TSL25911FN
- FRAME1: TITLE RJ12 Adapter -> Light Sensor Node
Connections:
- removed net IO: J4.2
- net +3V3: now also C2.1, C7.1, TP14.TP, TP21.TP, U5.VDD, U7.VDD; no longer J3.5, J4.5, TP1.TP
- net GND: now also C2.2, C7.2, TP13.TP, TP22.TP, U5.GND, U7.GND; no longer J3.1, J4.1, TP5.TP
- net SCL: now also TP20.TP, TP6.TP, U5.SCL, U7.SCL; no longer J3.3, J4.3, TP3.TP
- net SDA: now also TP19.TP, TP7.TP, U5.SDA, U7.SDA; no longer J3.4, J4.4, TP2.TP
Other:
- note added: "APDS-9250 Light Sensor"
- note added: "Note -I2C Addr is 0x29"
- note added: "Note: - I2C Addr is 0x52"
- note added: "TSL2591 Light Intensity Sensor"
- note removed: "RJ12 Connectors Chainable"

Commit message: added light and rj12 nodes, started working on light controller v2
Parts:
- removed C2, C7: 0.1uF, openag-capacitors:0.1UF-C0603C104K5RACTU
- removed L2: 68uH, openag-inductors:68UH-UP2B-680-R
- removed SJ4: (no value), openag-connectors:SOLDERJUMPERREFLOW_NOPASTE
- removed TP13, TP14, TP19, TP20, TP21, TP22, TP31: TPTP06R, openag-testpads:TPTP06R
- removed U5: APDS-9250, openag-sensors:APDS-9250
- removed U7: TSL2591, openag-sensors:TSL25911FN
- added C1, C3: 0.1uF, openag-capacitors:0.1UF-C0603C104K5RACTU
- added L1: 68uH, openag-inductors:68UH-UP2B-680-R
- added SJ2: (no value), openag-connectors:SOLDERJUMPERREFLOW_NOPASTE
- added TP15, TP16, TP17, TP18, TP3, TP5: TPTP06R, openag-testpads:TPTP06R
- added U1: APDS-9250, openag-sensors:APDS-9250
- added U6: TSL2591, openag-sensors:TSL25911FN
- C4: device openag-capacitors:15UF-TPSD156K035R0100 -> openag-capacitors:15UF-C2012X5R1V156M125AC
- D4: value B260A-13-F -> SBR2A40P1-7; device openag-diodes:B260A-13-F -> openag-diodes:SBR2A40P1-7
- R13, R15, R16, R17: value NV -> 600; device openag-resistors:R0603 -> openag-resistors:600OHM-RC0603FR-07604RL
- R14, R19: value NV -> 120; device openag-resistors:R0603 -> openag-resistors:120OHM-RC0603FR-07120RL
- R2, R7: value 100 OHM -> 100
- R20, R21: value NV -> 10K; device openag-resistors:R0603 -> openag-resistors:10K-ERJ-3EKF1002V
Connections:
- net +24V: now also C4.1, TP7.TP; no longer C4.1(+), TP12.TP
- net +3V3: now also C1.1, C3.1, TP12.TP, TP17.TP, U1.VDD, U6.VDD; no longer C2.1, C7.1, TP14.TP, TP21.TP, U5.VDD, U7.VDD
- net +5V: now also SJ2.2, TP5.TP; no longer SJ4.2, TP10.TP
- net GND: now also C1.2, C3.2, C4.2, TP18.TP, TP6.TP, U1.GND, U4.TAB, U6.GND; no longer C2.2, C4.2(-), C7.2, TP13.TP, TP22.TP, TP31.TP, U5.GND, U7.GND
- net N$31: now also L1.1; no longer L2.1
- net N$33: now also L1.2, SJ2.1; no longer L2.2, SJ4.1
- net SCL: now also TP16.TP, TP3.TP, U1.SCL, U6.SCL; no longer TP20.TP, TP6.TP, U5.SCL, U7.SCL
- net SDA: now also TP10.TP, TP15.TP, U1.SDA, U6.SDA; no longer TP19.TP, TP7.TP, U5.SDA, U7.SDA
Other:
- note added: "3.3V@400mA Regulator"
- note removed: "3.3V, 400mA Regulator"
- moved on the sheet: C4, C5, D5, R5, R6, R7, TP10, TP11, TP12, TP6, TP7, U3
