File: proj/PFC_EDU/V1.0/Electrical/LED_Array.sch (EAGLE design)
At the start: 24 parts

Commit message: PFC EDU PCB
Parts:
- renumbered LED1 to CH2-2, LED10 to CH6-3, LED11 to CH6-2, LED12 to CH6-1, LED13 to CH1-4, LED14 to CH1-3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
Connections:
- new net T: CH1-1.THERM, CH1-2.THERM, CH1-3.THERM, CH1-4.THERM, CH2-1.THERM, CH2-2.THERM, CH2-3.THERM, CH2-4.THERM, CH3-1.THERM, CH3-2.THERM, CH3-3.THERM, CH3-4.THERM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
Other:
- note added: "6 Channel 4 LED Series"
