File: proj/PFC_EDU/V1.0/Electrical/PFCEDU_V1.sch (EAGLE design)
At the start: 76 parts, among them IC2 PCA9615DP, IC3 PCA9615DP, J1 87583-2010BLF, J2 54602-908LF, J3 54602-908LF, T1 R-78E5.0-1.0, U1 TCA9548APWRPW24-M, U10 HPP845E034R5, U11 SHT25, U12 T6713-5K, U9 CCS811

Commit message: PFCEDU SCH AND BRD
Parts:
- removed FRAME2: (no value), openag-frames:DOCFIELD
- removed J1: 87583-2010BLF, openag-connectors:87583-2010BLF
- added C44, C45, C47, C48, C50, C51, C53, C54, C56, C57, C59, C60: 10nF, openag-capacitors:10NF-C0603C103K5RACTU
- added C46, C49, C52, C55, C58, C61: 100uF, openag-capacitors:100UF-EEE-1HA101UP
- added C64: 0.1uF, openag-capacitors:0.1UF-C0603C104K5RACTU
- added C65: 4.7uF, openag-capacitors:4.7UF-CL21A475KBQNNNE
- added C71: 10uF, openag-capacitors:10UF-GMK212BBJ106KG-T
- added CH1+1, CH1-1, CH2+1, CH2-1, CH3+1, CH3-1, CH4+1, CH4-1, CH5+1, CH5-1, CH6+1, CH6-1: (no value), openag-wirepads:3,17/1,3
- added L10, L11, L12, L13, L7, L9: 120uH, openag-inductors:120UH-74404064121
- added R100, R101, R102, R103, R104, R105, R106: 10K, openag-resistors:10K-ERJ-3EKF1002V
- added R109, R94, R95, R96, R97, R98, R99: 1K, openag-resistors:1K-ERJ-PB3D1001V
- added R110: 0 OHM, openag-resistors:0OHM-RC0603JR-070RL
- added SJ_A18, SJ_A19, SJ_A20, SJ_A21, SJ_A22, SJ_A23, SJ_A24, SJ_A25, SJ_A26, SJ_A27, SJ_A28, SJ_A29, SJ_A34, SJ_A35: (no value), openag-connectors:SOLDERJUMPERREFLOW_NOPASTE
- added U20, U21, U22, U23, U24, U25: RCD-24-0.70/VREF, openag-regulators:RCD-24-0.70/VREF
- added U27: DAC5578SPW, openag-dacs:DAC5578SPW
- added U30: PCA9685, openag-pwm:PCA9685PW/Q900,118
Connections:
- new net !LDAC!: R110.2, U27.!LDAC!
- new net A0: R105.2, SJ_A18.2, U30.A0
- new net A1: R104.2, SJ_A19.2, U30.A1
- new net A2: R103.2, SJ_A20.2, U30.A2
- new net A3: R102.2, SJ_A21.2, U30.A3
- new net A4: R101.2, SJ_A22.2, U30.A4
- new net A5: R100.2, SJ_A23.2, U30.A5
- new net ADDR0: SJ_A34.2, SJ_A35.2, U27.ADDR0
- new net CH1+: CH1+1.P, U20.+VOUT
- new net CH1-: C45.1, CH1-1.P, U20.-VOUT
- new net CH2+: CH2+1.P, U21.+VOUT
- new net CH2-: C48.1, CH2-1.P, U21.-VOUT
- new net CH3+: CH3+1.P, U22.+VOUT
- new net CH3-: C51.1, CH3-1.P, U22.-VOUT
- new net CH4+: CH4+1.P, U23.+VOUT
- new net CH4-: C54.1, CH4-1.P, U23.-VOUT
- new net CH5+: CH5+1.P, U24.+VOUT
- new net CH5-: C57.1, CH5-1.P, U24.-VOUT
- new net CH6+: CH6+1.P, U25.+VOUT
- new net CH6-: C60.1, CH6-1.P, U25.-VOUT
- new net DAC_!CLR!: R109.2, U27.!CLR!
- new net DIM1: R94.2, U20.ANALOGUE_DIM, U27.VOUT_G
- new net DIM2: R95.2, U21.ANALOGUE_DIM, U27.VOUT_E
- new net DIM3: R96.2, U22.ANALOGUE_DIM, U27.VOUT_C
- new net DIM4: R97.2, U23.ANALOGUE_DIM, U27.VOUT_A
- new net DIM5: R98.2, U24.ANALOGUE_DIM, U27.VOUT_H
- new net DIM6: R99.2, U25.ANALOGUE_DIM, U27.VOUT_F
- new net N$38: C44.1, L7.2, SJ_A24.1, U20.+VIN
- new net N$39: C47.1, L9.2, SJ_A25.1, U21.+VIN
- new net N$40: C50.1, L10.2, SJ_A26.1, U22.+VIN
- new net N$41: C53.1, L11.2, SJ_A27.1, U23.+VIN
- new net N$44: C56.1, L12.2, SJ_A28.1, U24.+VIN
- new net N$45: C59.1, L13.2, SJ_A29.1, U25.+VIN
- new net OE: R106.1, U30.#OE
- new net PWM1: U20.PWM/ON/OFF, U30.PWM6
- new net PWM2: U21.PWM/ON/OFF, U30.PWM5
- new net PWM3: U22.PWM/ON/OFF, U30.PWM4
- new net PWM4: U23.PWM/ON/OFF, U30.PWM3
- new net PWM5: U24.PWM/ON/OFF, U30.PWM2
- new net PWM6: U25.PWM/ON/OFF, U30.PWM1
- net +24V: now also C46.1(+), C49.1(+), C52.1(+), C55.1(+), C58.1(+), C61.1(+), L10.1, L11.1, L12.1, L13.1, L7.1, L9.1, SJ_A24.2, SJ_A25.2, SJ_A26.2, SJ_A27.2, SJ_A28.2, SJ_A29.2
- net +3V3: now also C64.1, C65.1, C71.1, R109.1, R94.1, R95.1, R96.1, R97.1, R98.1, R99.1, SJ_A18.1, SJ_A19.1, SJ_A20.1, SJ_A21.1, SJ_A22.1, SJ_A23.1, SJ_A34.1, U27.AVDD, U27.VREF_IN, U30.VDD
- net GND: now also C44.2, C45.2, C46.2(-), C47.2, C48.2, C49.2(-), C50.2, C51.2, C52.2(-), C53.2, C54.2, C55.2(-), C56.2, C57.2, C58.2(-), C59.2, C60.2, C61.2(-), C64.2, C65.2, C71.2, R100.1, R101.1, R102.1, R103.1, R104.1, R105.1, R106.2, R110.1, SJ_A35.1, U20.GND, U21.GND, U22.GND, U23.GND, U24.GND, U25.GND, U27.GND, U30.EXTCLK, U30.GND; no longer J1.1
- net SC3: now also U27.SCL, U30.SCL
- net SD3: now also U27.SDA, U30.SDA
- net USBM1: no longer J1.3
- net USBP1: no longer J1.2
Other:
- note added: "1 + A5 + A4 + A3 + A2 + A1 +A1 + RW"
- note added: "24V-0.7A Current Regulators"
- note added: "6-Channel 24V, 700mA (per channel) Current Regulator Module w/I2C Controlled Dimming via PWM or Analog Signaling"
- note added: "I2C Address ="
- note added: "I2C to 8-Channel 8-Bit DAC"
- note added: "Notes: - GND !LDAC! for syncronous mode - Broadcast I2C Addr = 0x47 - ADDR0=Low, I2C Addr=0x48 - ADDR0=High, I2C Addr=0x4A - ADDR0=Float, I2C Addr=0x4C"
- note added: "Open = 0 / Closed = 1"
- note added: "PCA9685 16-Channel I2C PWM Driver"
- note removed: "USB header"
- moved on the sheet: C1, C11, C14, C15, C9, D1, D2, D3, D4, F11, F12, R10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

Commit message: PFC EDU PCB
Parts:
- added CH1-6, CH1-7, CH1-8, CH1-9, CH2-6, CH2-7, CH2-8, CH2-9, CH3-6, CH3-7, CH3-8, CH3-9, CH4-6, CH4-7, CH4-8, CH4-9, CH5-6, CH5-7, CH5-8, CH5-9, CH6-6, CH6-7, CH6-8, CH6-9: XP-E, Tomaszewski:LED_W/THERM-XP-E
Connections:
- new net N$159: CH5-7.C, CH5-8.A
- new net N$160: CH5-6.C, CH5-7.A
- new net N$29: CH2-8.C, CH2-9.A
- new net N$31: CH2-7.C, CH2-8.A
- new net N$32: CH2-6.C, CH2-7.A
- new net N$33: CH4-8.C, CH4-9.A
- new net N$34: CH4-7.C, CH4-8.A
- new net N$35: CH4-6.C, CH4-7.A
- new net N$36: CH6-8.C, CH6-9.A
- new net N$37: CH6-7.C, CH6-8.A
- new net N$46: CH6-6.C, CH6-7.A
- new net N$47: CH1-8.C, CH1-9.A
- new net N$48: CH1-7.C, CH1-8.A
- new net N$81: CH1-6.C, CH1-7.A
- new net N$82: CH3-8.C, CH3-9.A
- new net N$83: CH3-7.C, CH3-8.A
- new net N$84: CH3-6.C, CH3-7.A
- new net N$85: CH5-8.C, CH5-9.A
- new net T1: CH1-6.THERM, CH1-7.THERM, CH1-8.THERM, CH1-9.THERM, CH2-6.THERM, CH2-7.THERM, CH2-8.THERM, CH2-9.THERM, CH3-6.THERM, CH3-7.THERM, CH3-8.THERM, CH3-9.THERM, CH4-6.THERM, CH4-7.THERM, CH4-8.THERM, CH4-9.THERM, CH5-6.THERM, CH5-7.THERM, CH5-8.THERM, CH5-9.THERM, CH6-6.THERM, CH6-7.THERM, CH6-8.THERM, CH6-9.THERM
- net CH1+: now also CH1-6.A
- net CH1-: now also CH1-9.C
- net CH2+: now also CH2-6.A
- net CH2-: now also CH2-9.C
- net CH3+: now also CH3-6.A
- net CH3-: now also CH3-9.C
- net CH4+: now also CH4-6.A
- net CH4-: now also CH4-9.C
- net CH5+: now also CH5-6.A
- net CH5-: now also CH5-9.C
- net CH6+: now also CH6-6.A
- net CH6-: now also CH6-9.C
Other:
- note added: "6 Channel 4 LED Series"

Commit message: PFC EDU PCB
Parts:
- added C21: 0.1uF, openag-capacitors:0.1UF-C0603C104K5RACTU
- added C22: 10uF, openag-capacitors:10UF-GMK212BBJ106KG-T
- added D8: APT1608CGCK, openag-diodes:APT1608CGCK
- added F1: 0448.400MR, openag-fuses:0438.375WR
- added R44: 100, openag-resistors:100OHM-RC0603JR-07100RL
- added SJ1: (no value), openag-connectors:SOLDERJUMPERREFLOW_NOPASTE
- added TP61, TP62, TP63: TPTP06R, openag-testpads:TPTP06R
- added U17: LM2937IMP3.3NOPB, openag-regulators:LM2937IMP-3.3/NOPB
- ATTRIBUTES: DESCRIPTION Nervous System -> PFC EDU; TITLE Nervous System -> PFC EDU; VER 2.0 -> (none)
- R10, R11, R12: value 100 OHM -> 100
Connections:
- new net N$179: D8.A, R44.1
- new net N$180: C22.1, F1.1, U17.OUT
- new net REG_3V3_400MA: F1.2, R44.2, SJ1.1
- net +3V3: now also SJ1.2, TP63.TP
- net +5V: now also C21.1, TP62.TP, U17.IN
- net GND: now also C21.2, C22.2, D8.C, TP61.TP, U17.GND, U17.TAB
Other:
- note added: "3.3V Enable Jumper"
- note added: "3.3V@400mA Regulator"
- note added: "5-26V to 3.3V@400mA Regulator w/3v3 Enable, Indicator LED & Fuse"

Commit message: PFC EDU
Parts:
- added C5: .1uF, rcl:C-USC0603
- added PAD1, PAD10, PAD2, PAD3, PAD4, PAD5, PAD6, PAD7, PAD8, PAD9: WIREPAD3,81/1,3, wirepad:WIREPAD3,81/1,3
- added PAD11, PAD12, PAD13, PAD14: (no value), wirepad:SMD2
- added Q1, Q2, Q3: MMBT2222A, transistor-npn:BCF30SMD
- added R13, R34, R35, R36, R38, R41: (no value), rcl:R-US_R0805W
- added R14, R15, R32, R33, R37, R39, R40: 10K, SparkFun-Resistors:10KOHM-1/10W-1%(0603)0603
- added T2: R-78E12.0-1.0, R-78E5.0-1.0:R-78E5.0-1.0
- added U2, U3, U5: STD12NF06LT4, OpenAG_I2C:STD12NF06LT4
- added U4: PCF8574APWRPW20-M, IO_Expander:PCF8574APWRPW20-M
Connections:
- new net +12V: PAD2.P, PAD4.P, PAD6.P, PAD7.P, PAD8.P, R13.2, R34.2, R38.2, T2.+VOUT
- new net A0_IO: R14.1, R33.2, U4.A0
- new net A1_IO: R15.1, R32.2, U4.A1
- new net MOS1: PAD3.P, U3.2
- new net MOS2: PAD1.P, U2.2
- new net MOS3: PAD5.P, U5.2
- new net N$13: R37.1, U4.!INT
- new net N$14: Q2.C, R34.1, U2.1
- new net N$15: Q2.B, R35.1
- new net N$16: Q3.C, R38.1, U5.1
- new net N$17: Q3.B, R41.1
- new net N$5: Q1.C, R13.1, U3.1
- new net N$9: Q1.B, R36.1
- new net P0_IO: R35.2, U4.P0
- new net P1_IO: U4.P1
- new net P2_IO: U4.P2
- new net P3_IO: U4.P3
- new net P4_IO: U4.P4
- new net P5_IO: U4.P5
- new net P6_IO: R41.2, U4.P6
- new net P7_IO: R36.2, U4.P7
- net +24V: now also T2.+VIN
- net +3V3: now also C5.1, F1.2, R14.2, R15.2, R37.2, R39.2, R40.2, U4.VCC
- net +5V: now also PAD11.P
- net GND: now also C5.2, PAD10.P, PAD14.P, PAD9.P, Q1.E, Q2.E, Q3.E, R32.1, R33.1, T2.GND, U2.3, U3.3, U4.A2, U4.GND, U5.3
- net REG_3V3_400MA: no longer F1.2
- net SC4: now also PAD13.P
- net SC5: now also R39.1, U4.SCL
- net SD4: now also PAD12.P
- net SD5: now also R40.1, U4.SDA
