File: proj/light-controller/v2.0/light_controller.sch (EAGLE design)
At the start: 146 parts, among them J1 0022232051, J2 OPENAG-I2C-RJ12, J3 OPENAG-I2C-RJ12, J4 1377G2, J5 OPENAG-RS485-RJ12, J6 OPENAG-RS485-RJ12, J7 OPENAG-I2C-HEADER, U1 RCD-24-0.70/VREF, U10 ADM2481BRWZ-RL7, U11 PHOTONH, U12 TLV70433DBVR, U13 LM2937IMP3.3NOPB, U14 PCA9685, U2 RCD-24-0.70/VREF, U3 RCD-24-0.70/VREF, U4 RCD-24-0.70/VREF, U5 RCD-24-0.70/VREF, U6 RCD-24-0.70/VREF, U7 DAC5578SPW, U8 ISO1540DR, U9 CY8C4124PVI-432

Commit message: added light and rj12 nodes, started working on light controller v2
Parts:
- removed C19: 0.1uF, openag-capacitors:0.1UF-C0603C104K5RACTU
- removed C20: 1uF, openag-capacitors:1UF-CL10A105KB8NNNC
- removed C24, C25: 10uF, openag-capacitors:10UF-GMK212BBJ106KG-T
- removed C37: 4.7uF, openag-capacitors:4.7UF-CL21A475KBQNNNE
- removed CR2: SMAJ26A-13-F, openag-diodes:SMAJ26A-13-F
- removed D2: APT1608CGCK, openag-diodes:APT1608CGCK
- removed F1: F0402G0R15FNTR, openag-fuses:F0402G0R15FNTR
- removed F3: 0448.400MR, openag-fuses:0438.375WR
- removed J2, J3: OPENAG-I2C-RJ12, openag-connectors:OPENAG-I2C-RJ12
- removed R10, R12: 1K, openag-resistors:1K-ERJ-PB3D1001V
- removed R27, R37: 100 OHM, openag-resistors:100OHM-RC0603JR-07100RL
- removed R36, R38: 0 OHM, openag-resistors:0OHM-RC0603JR-070RL
- removed U13: LM2937IMP3.3NOPB, openag-regulators:LM2937IMP-3.3/NOPB
- removed U8: ISO1540DR, openag-isolators:ISO1540DR
- added C35: 15uF, openag-capacitors:15UF-C2012X5R1V156M125AC
- added C39: 4.7uF, openag-capacitors:4.7UF-CL21A475KBQNNNE
- added C40: 0.1uF, openag-capacitors:0.1UF-C0603C104K5RACTU
- added D5, D8: APT1608CGCK, openag-diodes:APT1608CGCK
- added D6: SMAJ26A, openag-diodes:SMAJ26A-13-F
- added D7: SBR2A40P1-7, openag-diodes:SBR2A40P1-7
- added F5: SST 7, openag-fuses:SST_7
- added F6: (no value), fuse:GSH15
- added J10, J9: PJ-036AH, openag-connectors:PJ-036AH-SMT-TR
- added J8: 54602-908LF, openag_connector:OPENAG-V1-RJ45PTH
- added L8: 68uH, openag-inductors:68UH-UP2B-680-R
- added R40: 100 OHM, openag-resistors:100OHM-RC0603JR-07100RL
- added R42, R44, R45, R46: 600, openag-resistors:600OHM-RC0603FR-07604RL
- added R43, R47: 120, openag-resistors:120OHM-RC0603FR-07120RL
- added R48, R49: 10K, openag-resistors:10K-ERJ-3EKF1002V
- added SJ1, SJ3: (no value), openag-connectors:SOLDERJUMPERREFLOW_NOPASTE
- added TP1, TP10, TP12, TP13, TP14, TP15, TP16, TP17, TP2, TP3, TP4, TP5, TP6, TP7: TPTP06R, openag-testpads:TPTP06R
- added U15: PCA9615DPJ, openag-buffers:PCA9615DPJ
- added U16: MIC4680YM-TR, openag-regulators:MIC4680YM-TR
- C36: value 10uF -> 220uF; device openag-capacitors:10UF-GMK212BBJ106KG-T -> openag-capacitors:220UF-TPSY227K010R0100
- C38: value 0.1uF -> 10uF; device openag-capacitors:0.1UF-C0603C104K5RACTU -> openag-capacitors:10UF-GMK212BBJ106KG-T
- F2: value SST 7 -> 0448.400MR; device openag-fuses:SST_7 -> openag-fuses:0438.375WR
- J4: value 1377G2 -> 54602-908LF; device openag-connectors:1377G21377G2 -> openag_connector:OPENAG-V1-RJ45PTH
- R11: value 1K -> 100 OHM; device openag-resistors:1K-ERJ-PB3D1001V -> openag-resistors:100OHM-RC0603JR-07100RL
- R13: value 1K -> 3.01K; device openag-resistors:1K-ERJ-PB3D1001V -> openag-resistors:3.01K-RC0603FR-073K01L
- R32: value 0 OHM -> 976 Ohm; device openag-resistors:0OHM-RC0603JR-070RL -> openag-resistors:982OHM-RC0603FR-07976RL
- R33: value 0 OHM -> 100 OHM; device openag-resistors:0OHM-RC0603JR-070RL -> openag-resistors:100OHM-RC0603JR-07100RL
- U12: value TLV70433DBVR -> LM2937IMP3.3NOPB; device openag-regulators:TLV70433DBVRDBV5-M -> openag-regulators:LM2937IMP-3.3/NOPB
Connections:
- removed net I2C_IO: J2.2, J3.2
- removed net N$3: D1.A, R27.1
- removed net N$9: C20.1, F1.1, U12.OUT
- removed net REG_3V3_150MA: F1.2, R36.1, R37.2
- new net +5V: R44.1, R45.2, SJ1.2, TP12.TP, TP7.TP, U15.VDD_(B)
- new net DSCLM: J4.DSCLM, J8.DSCLM, R46.2, R47.1, U15.DSCLM
- new net DSCLP: J4.DSCLP, J8.DSCLP, R45.1, R47.2, U15.DSCLP
- new net DSDAM: J4.DSDAM, J8.DSDAM, R42.1, R43.2, U15.DSDAM
- new net DSDAP: J4.DSDAP, J8.DSDAP, R43.1, R44.2, U15.DSDAP
- new net LIN_REG_VIN: C22.1, TP16.TP, U12.IN
- new net N$11: D7.12, L8.1, R13.1, R32.2, U16.FB, U16.SW
- new net N$22: D8.A, R33.1
- new net N$24: C36.1(+), L8.2, R13.2, R33.2, SJ1.1
- new net N$26: D5.A, R40.1
- new net USBM: J4.USBM, J8.USBM
- new net USBP: J4.USBP, J8.USBP
- net +24V: now also C35.1, C39.1, C40.1, D6.P$2, F5.2, F6.2, J4.+24V, J8.+24V, R40.2, TP10.TP, TP14.TP, TP4.TP, U16.IN; no longer C19.1, C22.1, C36.1, C37.1, CR2.P$2, F2.2, U12.IN, U13.IN
- net +3V3: now also R48.2, R49.2, SJ3.2, TP17.TP, TP5.TP, U15.VDD_(A); no longer C25.1, R10.2, R11.2, R36.2, R38.2, U8.VCC2
- net 24V_IN: now also F5.1, F6.1, J10.1, J9.1; no longer F2.1, J4.V+
- net GND: now also C35.2, C36.2(-), C39.2, C40.2, D5.C, D6.P$1, D7.21, D8.C, J10.2, J10.3, J8.GND, J9.2, J9.3, R32.1, R42.2, R46.1, TP13.TP, TP15.TP, TP3.TP, TP6.TP, U15.VSS, U16.GND, U16.SHDN; no longer C19.2, C20.2, C25.2, C36.2, C37.2, CR2.P$1, D2.C, U13.GND, U8.GND2
- net I2C_3V3: no longer C24.1, J2.5, J3.5, R12.2, R13.2, U8.VCC1
- net I2C_GND: no longer C24.2, J2.1, J3.1, U8.GND1
- net N$10: now also D1.A, R11.1; no longer C23.1, F3.1, U13.OUT
- net N$12: now also C23.1, F2.1, U12.OUT; no longer D2.A, R37.1
- net REG_3V3_400MA: now also F2.2, R11.2, SJ3.1; no longer F3.2, R27.2, R38.1
- net SCL: now also R49.1, TP1.TP, U15.SCL; no longer R33.2
- net SCL1: no longer J2.3, J3.3, R12.1, U8.SCL1
- net SCL2: no longer R10.1, R33.1, U8.SCL2
- net SDA: now also R48.1, TP2.TP, U15.SDA; no longer R32.2
- net SDA1: no longer J2.4, J3.4, R13.1, U8.SDA1
- net SDA2: no longer R11.1, R32.1, U8.SDA2
Other:
- note added: "24V Power Conditioning + Fuse"
- note added: "24V to 5V@1A Switching Regulator w/Indicator LED + Enable"
- note added: "3.3V Enable Jumper"
- note added: "5-26V to 3.3V@400mA Regulator w/3v3 Enable, Indicator LED & Fuse"
- note added: "Barrel Jack Connectors"
- note added: "Dual Barrel Jack Connectors with 24V Conditioning + Fuse + Indicator LED"
- note added: "Indicator LED"
- note added: "RJ45 Connector w/dI2C Buffer"
- note added: "RJ45 Connectors"
- note added: "dI2C Buffer"
- note removed: "24V / GND Anderson Powerpole Connector"
- note removed: "24V Power Conditioning"
- note removed: "24V Powerpole Connector"
- note removed: "24V-to-3.3V, 150mA Regulator w/3v3 Enable, Incdicator LED & Fuse"
- note removed: "3.3V Enable Resistor"
- note removed: "3.3V, 150mA Linear Regulator"
- note removed: "5-24V to 3.3V@400mA Regulator w/3v3 Enable, Indicator LED & Fuse"
- note removed: "I2C Connector Pair w/Isolation and Inter-I2C Connection Option"
- note removed: "I2C Isolator"
- note removed: "Inter-I2C Connect Option"
- moved on the sheet: C22, C23, C36, C38, D1, F2, R13, R33

Commit message: added light controller v2.0
Parts:
- removed C30: 0.1uF, openag-capacitors:0.1UF-C0603C104K5RACTU
- removed C34: 4.7uF, openag-capacitors:4.7UF-CL21A475KBQNNNE
- removed R15, R16, R17, R18, R19, R20, R21, R22, R23, R24, R25, R30, R31, R34, R35: 0 OHM, openag-resistors:0OHM-RC0603JR-070RL
- removed SJ_A12, SJ_A13, SJ_A14, SJ_A15: (no value), openag-connectors:SOLDERJUMPERREFLOW_NOPASTE
- removed U11: PHOTONH, openag-microcontrollers:PHOTONHPHOTONH
- added SJ4, SJ6: (no value), openag-connectors:SOLDERJUMPERREFLOW_NOPASTE
- added TP11, TP18, TP19, TP20, TP21, TP22, TP23, TP24, TP25, TP26, TP27, TP28, TP29, TP30, TP31, TP8, TP9: TPTP04R, openag-testpads:TPTP04R
- D1, D5, D8: value APT1608CGCK -> APT1608
- R1: value 0 OHM -> 1K; device openag-resistors:0OHM-RC0603JR-070RL -> openag-resistors:1K-ERJ-PB3D1001V
- R11, R33, R40: value 100 OHM -> 100
Connections:
- removed net I2C_3V3: J7.3V3, SJ_A15.2
- removed net I2C_GND: J7.GND, SJ_A12.2
- removed net N$8: C30.1, C34.1, R17.1, U11.3V3
- removed net P0[6]: R35.1, U9.P0[6]
- removed net P0[7]: R25.1, U9.P0[7]
- removed net P2[6]: R20.1, U9.P2[6]
- removed net P2[7]: R21.1, U9.P2[7]
- removed net PHOTON_A0: R24.1, U11.A0
- removed net PHOTON_A1: R34.1, U11.A1
- removed net PHOTON_D2: R22.1, U11.D2
- removed net PHOTON_D3: R23.1, U11.D3
- removed net PHOTON_D4: U11.D4
- removed net PHOTON_RX: R18.1, U11.RX
- removed net PHOTON_SCL: R5.1, U11.D1
- removed net PHOTON_SDA: R4.1, U11.D0
- removed net PHOTON_TX: R19.1, U11.TX
- removed net SCB0_I2C_SCL: R2.1, U9.P4[0]
- removed net SCB0_I2C_SDA: R1.1, U9.P4[1]
- removed net SCL1: J7.SCL, SJ_A13.2
- removed net SCL2: R31.2
- removed net SDA1: J7.SDA, SJ_A14.2
- removed net SDA2: R30.2
- removed net VDDD: C31.1, C32.1, J1.VTARG, R3.2, U9.VDDD
- new net N/C: J4.+24V, J8.+24V, TP10.TP
- new net SCL_IN: R2.2, R49.1, SJ4.1, TP1.TP, TP26.TP, U15.SCL
- new net SDA_IN: R4.2, R48.1, SJ6.1, TP2.TP, TP25.TP, U15.SDA
- net !LDAC!: now also R1.2, TP23.TP, U9.P0[7]; no longer R34.2, R35.2
- net +24V: no longer J4.+24V, J8.+24V, TP10.TP
- net +3V3: now also C31.1, C32.1, J1.VTARG, J7.3V3, R1.1, TP19.TP, TP27.TP, U9.VDDD; no longer R17.2, R3.1, SJ_A15.1
- net DAC_!CLR!: now also TP8.TP, U9.P0[6]; no longer R24.2, R25.2
- net GND: now also J7.GND, TP9.TP; no longer C30.2, C34.2, SJ_A12.1, U11.GND@2, U11.GND@21
- net SCB1_RX[0]_SCL[0]: now also R2.1, R3.1; no longer R15.1, R31.1
- net SCB1_TX[0]_SDA[0]: now also R4.1, R5.1; no longer R16.1, R30.1
- net SCL: now also J7.SCL, SJ4.2, TP24.TP, U9.P4[0]; no longer R2.2, R49.1, R5.2, SJ_A13.1, TP1.TP, U15.SCL
- net SDA: now also J7.SDA, SJ6.2, TP18.TP, U9.P4[1]; no longer R1.2, R4.2, R48.1, SJ_A14.1, TP2.TP, U15.SDA
- net UART_!RE!: now also TP21.TP, TP30.TP, U9.P2[7]; no longer R21.2, R23.2
- net UART_DE: now also TP22.TP, TP31.TP, U9.P2[6]; no longer R20.2, R22.2
- net UART_RX: now also R3.2, TP20.TP, TP29.TP; no longer R15.2, R18.2
- net UART_TX: now also R5.2, TP11.TP, TP28.TP; no longer R16.2, R19.2
Other:
- note added: "Barrel Jack Connector Pair with 24V Conditioning + Fuse + Indicator LED"
- note added: "Changelog - replaced rj12 connector w/rj45 - added switching reg for 24V to 5V - replaced powerpole with barrel jack - removed photon - added pullup to dac load line - cleaned up modules"
- note added: "Communication Mode Select"
- note added: "I2C Connect"
- note added: "Notes: - P4[0] is SCB0_I2C_SCL - P4[1] is SCB0_I2C_SDA"
- note added: "PSOC4100 Microcontroller w/I2C or RS485 Communication + Programming Header"
- note added: "Testpads"
- note removed: "Changelog - added inductor pass through - added isolator pass through - removed dac reset pushbutton - removed voltage divider for dac reference - exposed ldac to microcontrollers - exposed dac address set - added 400mA 3v3 regulator - set 3v3 regulator led to be on circuit before enable - added fuse to both 3v3 regulator circuits"
- note removed: "Dual Barrel Jack Connectors with 24V Conditioning + Fuse + Indicator LED"
- note removed: "PSOC4100 Microcontroller w/Optional Dual Channel I2C and/or RS485 Connections"
- note removed: "Photon Microcontroller"
- note removed: "Photon w/Optional I2C + RS485 Connections"
- moved on the sheet: C22, C23, C26, C27, C31, C32, C33, C35, C36, C38, C39, C40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

Commit message: added photon rj45 shield
Parts:
- removed SJ_A10, SJ_A11, SJ_A6, SJ_A7, SJ_A8, SJ_A9: (no value), openag-connectors:SOLDERJUMPERREFLOW_NOPASTE
Connections:
- net +24V: no longer SJ_A10.2, SJ_A11.2, SJ_A6.2, SJ_A7.2, SJ_A8.2, SJ_A9.2
- net N$1: no longer SJ_A6.1
- net N$2: no longer SJ_A7.1
- net N$4: no longer SJ_A8.1
- net N$5: no longer SJ_A9.1
- net N$6: no longer SJ_A10.1
- net N$7: no longer SJ_A11.1
Changed lines of the file:
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@@
 <setting verticaltext="up"/>
 </settings>
-<grid distance="1.5" unitdist="inch" unit="inch" style="lines" multiple="1" display="yes" altdistance="0.01" altunitdist="inch" altunit="inch"/>
+<grid distance="0.1" unitdist="inch" unit="inch" style="lines" multiple="1" display="yes" altdistance="0.01" altunitdist="inch" altunit="inch"/>
 <layers>
 <layer number="1" name="Top" color="4" fill="1" visible="no" active="no"/>
@@
 <part name="J6" library="openag-connectors" deviceset="OPENAG-RS485-RJ12" device="" value="OPENAG-RS485-RJ12"/>
 <part name="J7" library="openag-connectors" deviceset="OPENAG-I2C-HEADER" device="" value="OPENAG-I2C-HEADER"/>
-<part name="SJ_A6" library="openag-connectors" deviceset="SOLDERJUMPER" device="REFLOW_NOPASTE"/>
-<part name="SJ_A7" library="openag-connectors" deviceset="SOLDERJUMPER" device="REFLOW_NOPASTE"/>
-<part name="SJ_A8" library="openag-connectors" deviceset="SOLDERJUMPER" device="REFLOW_NOPASTE"/>
-<part name="SJ_A9" library="openag-connectors" deviceset="SOLDERJUMPER" device="REFLOW_NOPASTE"/>
-<part name="SJ_A10" library="openag-connectors" deviceset="SOLDERJUMPER" device="REFLOW_NOPASTE"/>
-<part name="SJ_A11" library="openag-connectors" deviceset="SOLDERJUMPER" device="REFLOW_NOPASTE"/>
 <part name="R28" library="openag-resistors" deviceset="1K-ERJ-PB3D1001V" device="" value="1K"/>
 <part name="R29" library="openag-resistors" deviceset="0OHM-RC0603JR-070RL" device="" value="0 OHM"/>
@@
 <attribute name="VALUE" x="241.3" y="577.596" size="2.54" layer="96"/>
 </instance>
-<instance part="SJ_A6" gate="1" x="-307.34" y="457.2" rot="R180"/>
-<instance part="SJ_A7" gate="1" x="-307.34" y="419.1" rot="R180"/>
-<instance part="SJ_A8" gate="1" x="-307.34" y="381" rot="R180"/>
-<instance part="SJ_A9" gate="1" x="-307.34" y="342.9" rot="R180"/>
-<instance part="SJ_A10" gate="1" x="-307.34" y="304.8" rot="R180"/>
-<instance part="SJ_A11" gate="1" x="-307.34" y="266.7" rot="R180"/>
 <instance part="R28" gate="A" x="-86.36" y="358.14" rot="R270"/>
 <instance part="R29" gate="G$1" x="-157.48" y="396.24"/>
@@
 <net name="+24V" class="0">
 <segment>
-<wire x1="-320.04" y1="454.66" x2="-320.04" y2="457.2" width="0.1524" layer="91"/>
-<wire x1="-320.04" y1="457.2" x2="-320.04" y2="462.28" width="0.1524" layer="91"/>
+<wire x1="-320.04" y1="454.66" x2="-320.04" y2="462.28" width="0.1524" layer="91"/>
 <wire x1="-320.04" y1="462.28" x2="-312.42" y2="462.28" width="0.1524" layer="91"/>
 <wire x1="-320.04" y1="462.28" x2="-322.58" y2="462.28" width="0.1524" layer="91"/>
@@
 <pinref part="C3" gate="G$1" pin="1(+)"/>
 <pinref part="L1" gate="G$1" pin="1"/>
-<pinref part="SJ_A6" gate="1" pin="2"/>
-<wire x1="-312.42" y1="457.2" x2="-320.04" y2="457.2" width="0.1524" layer="91"/>
-<junction x="-320.04" y="457.2"/>
-</segment>
-<segment>
-<wire x1="-320.04" y1="416.56" x2="-320.04" y2="419.1" width="0.1524" layer="91"/>
-<wire x1="-320.04" y1="419.1" x2="-320.04" y2="424.18" width="0.1524" layer="91"/>
+</segment>
+<segment>
+<wire x1="-320.04" y1="416.56" x2="-320.04" y2="424.18" width="0.1524" layer="91"/>
 <wire x1="-320.04" y1="424.18" x2="-312.42" y2="424.18" width="0.1524" layer="91"/>
 <wire x1="-320.04" y1="424.18" x2="-322.58" y2="424.18" width="0.1524" layer="91"/>
@@
 <pinref part="C6" gate="G$1" pin="1(+)"/>
 <pinref part="L2" gate="G$1" pin="1"/>
-<pinref part="SJ_A7" gate="1" pin="2"/>
-<wire x1="-312.42" y1="419.1" x2="-320.04" y2="419.1" width="0.1524" layer="91"/>
-<junction x="-320.04" y="419.1"/>
-</segment>
-<segment>
-<wire x1="-320.04" y1="378.46" x2="-320.04" y2="381" width="0.1524" layer="91"/>
-<wire x1="-320.04" y1="381" x2="-320.04" y2="386.08" width="0.1524" layer="91"/>
+</segment>
+<segment>
+<wire x1="-320.04" y1="378.46" x2="-320.04" y2="386.08" width="0.1524" layer="91"/>
 <wire x1="-320.04" y1="386.08" x2="-312.42" y2="386.08" width="0.1524" layer="91"/>
 <wire x1="-320.04" y1="386.08" x2="-322.58" y2="386.08" width="0.1524" layer="91"/>
@@
 <pinref part="C9" gate="G$1" pin="1(+)"/>
 <pinref part="L3" gate="G$1" pin="1"/>
-<pinref part="SJ_A8" gate="1" pin="2"/>
-<wire x1="-312.42" y1="381" x2="-320.04" y2="381" width="0.1524" layer="91"/>
-<junction x="-320.04" y="381"/>
-</segment>
-<segment>
-<wire x1="-320.04" y1="340.36" x2="-320.04" y2="342.9" width="0.1524" layer="91"/>
-<wire x1="-320.04" y1="342.9" x2="-320.04" y2="347.98" width="0.1524" layer="91"/>
+</segment>
+<segment>
+<wire x1="-320.04" y1="340.36" x2="-320.04" y2="347.98" width="0.1524" layer="91"/>
 <wire x1="-320.04" y1="347.98" x2="-312.42" y2="347.98" width="0.1524" layer="91"/>
 <wire x1="-320.04" y1="347.98" x2="-322.58" y2="347.98" width="0.1524" layer="91"/>
@@
 <pinref part="C12" gate="G$1" pin="1(+)"/>
 <pinref part="L4" gate="G$1" pin="1"/>
-<pinref part="SJ_A9" gate="1" pin="2"/>
-<wire x1="-312.42" y1="342.9" x2="-320.04" y2="342.9" width="0.1524" layer="91"/>
-<junction x="-320.04" y="342.9"/>
-</segment>
-<segment>
-<wire x1="-320.04" y1="302.26" x2="-320.04" y2="304.8" width="0.1524" layer="91"/>
-<wire x1="-320.04" y1="304.8" x2="-320.04" y2="309.88" width="0.1524" layer="91"/>
+</segment>
+<segment>
+<wire x1="-320.04" y1="302.26" x2="-320.04" y2="309.88" width="0.1524" layer="91"/>
 <wire x1="-320.04" y1="309.88" x2="-312.42" y2="309.88" width="0.1524" layer="91"/>
 <wire x1="-320.04" y1="309.88" x2="-322.58" y2="309.88" width="0.1524" layer="91"/>
@@
 <pinref part="C15" gate="G$1" pin="1(+)"/>
 <pinref part="L5" gate="G$1" pin="1"/>
-<pinref part="SJ_A10" gate="1" pin="2"/>
-<wire x1="-312.42" y1="304.8" x2="-320.04" y2="304.8" width="0.1524" layer="91"/>
-<junction x="-320.04" y="304.8"/>
-</segment>
-<segment>
-<wire x1="-320.04" y1="264.16" x2="-320.04" y2="266.7" width="0.1524" layer="91"/>
-<wire x1="-320.04" y1="266.7" x2="-320.04" y2="271.78" width="0.1524" layer="91"/>
+</segment>
+<segment>
+<wire x1="-320.04" y1="264.16" x2="-320.04" y2="271.78" width="0.1524" layer="91"/>
 <wire x1="-320.04" y1="271.78" x2="-312.42" y2="271.78" width="0.1524" layer="91"/>
 <wire x1="-320.04" y1="271.78" x2="-322.58" y2="271.78" width="0.1524" layer="91"/>
@@
 <pinref part="C18" gate="G$1" pin="1(+)"/>
 <pinref part="L6" gate="G$1" pin="1"/>
-<pinref part="SJ_A11" gate="1" pin="2"/>
-<wire x1="-312.42" y1="266.7" x2="-320.04" y2="266.7" width="0.1524" layer="91"/>
-<junction x="-320.04" y="266.7"/>
 </segment>
 <segment>
@@
 <pinref part="C1" gate="G$1" pin="1"/>
 <pinref part="L1" gate="G$1" pin="2"/>
-<pinref part="SJ_A6" gate="1" pin="1"/>
-<wire x1="-302.26" y1="457.2" x2="-297.18" y2="457.2" width="0.1524" layer="91"/>
 <wire x1="-297.18" y1="457.2" x2="-297.18" y2="456.946" width="0.1524" layer="91"/>
 <junction x="-297.18" y="456.946"/>
@@
 <pinref part="C4" gate="G$1" pin="1"/>
 <pinref part="L2" gate="G$1" pin="2"/>
-<pinref part="SJ_A7" gate="1" pin="1"/>
-<wire x1="-302.26" y1="419.1" x2="-297.18" y2="419.1" width="0.1524" layer="91"/>
 <wire x1="-297.18" y1="419.1" x2="-297.18" y2="418.846" width="0.1524" layer="91"/>
 <junction x="-297.18" y="418.846"/>
@@
 <pinref part="C7" gate="G$1" pin="1"/>
 <pinref part="L3" gate="G$1" pin="2"/>
-<pinref part="SJ_A8" gate="1" pin="1"/>
-<wire x1="-302.26" y1="381" x2="-297.18" y2="381" width="0.1524" layer="91"/>
 <wire x1="-297.18" y1="381" x2="-297.18" y2="380.746" width="0.1524" layer="91"/>
 <junction x="-297.18" y="380.746"/>
@@
 <pinref part="C10" gate="G$1" pin="1"/>
 <pinref part="L4" gate="G$1" pin="2"/>
-<pinref part="SJ_A9" gate="1" pin="1"/>
-<wire x1="-302.26" y1="342.9" x2="-297.18" y2="342.9" width="0.1524" layer="91"/>
 <wire x1="-297.18" y1="342.9" x2="-297.18" y2="342.646" width="0.1524" layer="91"/>
 <junction x="-297.18" y="342.646"/>
@@
 <pinref part="C13" gate="G$1" pin="1"/>
 <pinref part="L5" gate="G$1" pin="2"/>
-<pinref part="SJ_A10" gate="1" pin="1"/>
-<wire x1="-302.26" y1="304.8" x2="-297.18" y2="304.8" width="0.1524" layer="91"/>
 <wire x1="-297.18" y1="304.8" x2="-297.18" y2="304.546" width="0.1524" layer="91"/>
 <junction x="-297.18" y="304.546"/>
@@
 <pinref part="C16" gate="G$1" pin="1"/>
 <pinref part="L6" gate="G$1" pin="2"/>
-<pinref part="SJ_A11" gate="1" pin="1"/>
-<wire x1="-302.26" y1="266.7" x2="-297.18" y2="266.7" width="0.1524" layer="91"/>
 <wire x1="-297.18" y1="266.7" x2="-297.18" y2="266.446" width="0.1524" layer="91"/>
 <junction x="-297.18" y="266.446"/>

Commit message: swapped inductor on light panel v2.0
Parts:
- L1, L2, L3, L4, L5, L6: device openag-inductors:120UH-74404064121 -> openag-inductors:120UH-ASPI-6045S-121M-TCT-ND
Changed lines of the file:
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@@
 <part name="C2" library="openag-capacitors" deviceset="10NF-C0603C103K5RACTU" device="" value="10nF"/>
 <part name="C3" library="openag-capacitors" deviceset="100UF-EEE-1HA101UP" device="" value="100uF"/>
-<part name="L1" library="openag-inductors" deviceset="120UH-74404064121" device="" value="120uH"/>
+<part name="L1" library="openag-inductors" deviceset="120UH-ASPI-6045S-121M-TCT-ND" device="" value="120uH"/>
 <part name="GND2" library="openag-supply" deviceset="GND" device=""/>
 <part name="CH1+" library="openag-wirepads" deviceset="3,17/1,3" device=""/>
@@
 <part name="C5" library="openag-capacitors" deviceset="10NF-C0603C103K5RACTU" device="" value="10nF"/>
 <part name="C6" library="openag-capacitors" deviceset="100UF-EEE-1HA101UP" device="" value="100uF"/>
-<part name="L2" library="openag-inductors" deviceset="120UH-74404064121" device="" value="120uH"/>
+<part name="L2" library="openag-inductors" deviceset="120UH-ASPI-6045S-121M-TCT-ND" device="" value="120uH"/>
 <part name="GND3" library="openag-supply" deviceset="GND" device=""/>
 <part name="CH2+" library="openag-wirepads" deviceset="3,17/1,3" device=""/>
@@
 <part name="C8" library="openag-capacitors" deviceset="10NF-C0603C103K5RACTU" device="" value="10nF"/>
 <part name="C9" library="openag-capacitors" deviceset="100UF-EEE-1HA101UP" device="" value="100uF"/>
-<part name="L3" library="openag-inductors" deviceset="120UH-74404064121" device="" value="120uH"/>
+<part name="L3" library="openag-inductors" deviceset="120UH-ASPI-6045S-121M-TCT-ND" device="" value="120uH"/>
 <part name="GND4" library="openag-supply" deviceset="GND" device=""/>
 <part name="CH3+" library="openag-wirepads" deviceset="3,17/1,3" device=""/>
@@
 <part name="C11" library="openag-capacitors" deviceset="10NF-C0603C103K5RACTU" device="" value="10nF"/>
 <part name="C12" library="openag-capacitors" deviceset="100UF-EEE-1HA101UP" device="" value="100uF"/>
-<part name="L4" library="openag-inductors" deviceset="120UH-74404064121" device="" value="120uH"/>
+<part name="L4" library="openag-inductors" deviceset="120UH-ASPI-6045S-121M-TCT-ND" device="" value="120uH"/>
 <part name="GND5" library="openag-supply" deviceset="GND" device=""/>
 <part name="CH4+" library="openag-wirepads" deviceset="3,17/1,3" device=""/>
@@
 <part name="C14" library="openag-capacitors" deviceset="10NF-C0603C103K5RACTU" device="" value="10nF"/>
 <part name="C15" library="openag-capacitors" deviceset="100UF-EEE-1HA101UP" device="" value="100uF"/>
-<part name="L5" library="openag-inductors" deviceset="120UH-74404064121" device="" value="120uH"/>
+<part name="L5" library="openag-inductors" deviceset="120UH-ASPI-6045S-121M-TCT-ND" device="" value="120uH"/>
 <part name="GND6" library="openag-supply" deviceset="GND" device=""/>
 <part name="CH5+" library="openag-wirepads" deviceset="3,17/1,3" device=""/>
@@
 <part name="C17" library="openag-capacitors" deviceset="10NF-C0603C103K5RACTU" device="" value="10nF"/>
 <part name="C18" library="openag-capacitors" deviceset="100UF-EEE-1HA101UP" device="" value="100uF"/>
-<part name="L6" library="openag-inductors" deviceset="120UH-74404064121" device="" value="120uH"/>
+<part name="L6" library="openag-inductors" deviceset="120UH-ASPI-6045S-121M-TCT-ND" device="" value="120uH"/>
 <part name="GND7" library="openag-supply" deviceset="GND" device=""/>
 <part name="CH6+" library="openag-wirepads" deviceset="3,17/1,3" device=""/>
