File: proj/sensor-nodes/air/v1.0/air.sch (EAGLE design)
At the start: 67 parts, among them J1 54602-908LF, J2 54602-908LF, U2 PCA9615DPJ, U3 MIC4680YM-TR, U4 LM2937IMP3.3NOPB, U5 SHT25, U6 CCS811, U7 T6713-5K, U8 HPP845E034R5

Commit message: added easy bom generator
Parts:
- D1, D5: value APT1608CGCK -> APT1608
Other:
- moved on the sheet: TP13, TP14, TP15, TP16, TP17, TP18, TP19, TP20, TP21, TP22, TP23, TP24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
Changed lines of the file:
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@@
 <attribute name="URL" value="github.com/OpenAgInitiative/openag_eagle/proj/sensor-nodes"/>
 </part>
-<part name="D1" library="openag-diodes" deviceset="APT1608CGCK" device="" value="APT1608CGCK"/>
+<part name="D1" library="openag-diodes" deviceset="APT1608CGCK" device="" value="APT1608"/>
 <part name="R2" library="openag-resistors" deviceset="100OHM-RC0603JR-07100RL" device="" value="100"/>
 <part name="GND5" library="openag-supply" deviceset="GND" device=""/>
@@
 <part name="P+5" library="openag-supply" deviceset="+5V" device=""/>
 <part name="R7" library="openag-resistors" deviceset="100OHM-RC0603JR-07100RL" device="" value="100"/>
-<part name="D5" library="openag-diodes" deviceset="APT1608CGCK" device="" value="APT1608CGCK"/>
+<part name="D5" library="openag-diodes" deviceset="APT1608CGCK" device="" value="APT1608"/>
 <part name="TP5" library="openag-testpads" deviceset="TP" device="TP06R"/>
 <part name="TP6" library="openag-testpads" deviceset="TP" device="TP06R"/>
@@
 <instance part="+3V8" gate="G$1" x="55.88" y="137.16"/>
 <instance part="C8" gate="G$1" x="55.88" y="101.6"/>
-<instance part="TP13" gate="G$1" x="50.8" y="121.92"/>
-<instance part="TP14" gate="G$1" x="50.8" y="111.76" rot="R180"/>
+<instance part="TP13" gate="G$1" x="50.8" y="119.38" rot="R270"/>
+<instance part="TP14" gate="G$1" x="50.8" y="114.3" rot="R90"/>
 <instance part="TP15" gate="G$1" x="106.68" y="93.98" rot="R270"/>
-<instance part="TP16" gate="G$1" x="106.68" y="119.38" rot="R270"/>
+<instance part="TP16" gate="G$1" x="104.14" y="119.38" rot="R180"/>
 <instance part="U8" gate="G$1" x="76.2" y="20.32"/>
 <instance part="+3V10" gate="G$1" x="53.34" y="30.48" smashed="yes">
@@
 <instance part="GND16" gate="1" x="53.34" y="15.24"/>
 <instance part="C10" gate="G$1" x="55.88" y="22.86"/>
-<instance part="TP21" gate="G$1" x="93.98" y="27.94"/>
-<instance part="TP22" gate="G$1" x="93.98" y="20.32"/>
-<instance part="TP23" gate="G$1" x="50.8" y="25.4" rot="R90"/>
+<instance part="TP21" gate="G$1" x="93.98" y="25.4" rot="R270"/>
+<instance part="TP22" gate="G$1" x="93.98" y="17.78" rot="R270"/>
+<instance part="TP23" gate="G$1" x="53.34" y="25.4"/>
 <instance part="TP24" gate="G$1" x="50.8" y="17.78" rot="R90"/>
 <instance part="U5" gate="G$1" x="187.96" y="17.78"/>
@@
 </instance>
 <instance part="C2" gate="G$1" x="172.72" y="20.32"/>
-<instance part="TP17" gate="G$1" x="203.2" y="25.4"/>
-<instance part="TP18" gate="G$1" x="203.2" y="15.24"/>
-<instance part="TP19" gate="G$1" x="170.18" y="12.7" rot="R90"/>
-<instance part="TP20" gate="G$1" x="170.18" y="22.86" rot="R90"/>
+<instance part="TP17" gate="G$1" x="203.2" y="22.86" rot="R270"/>
+<instance part="TP18" gate="G$1" x="203.2" y="12.7" rot="R270"/>
+<instance part="TP19" gate="G$1" x="172.72" y="12.7"/>
+<instance part="TP20" gate="G$1" x="172.72" y="22.86"/>
 <instance part="U7" gate="G$1" x="160.02" y="119.38"/>
 <instance part="GND11" gate="1" x="180.34" y="96.52"/>
 <instance part="C7" gate="G$1" x="180.34" y="119.38"/>
 <instance part="+3V6" gate="G$1" x="198.12" y="129.54"/>
-<instance part="TP25" gate="G$1" x="185.42" y="139.7"/>
-<instance part="TP26" gate="G$1" x="185.42" y="132.08"/>
-<instance part="TP27" gate="G$1" x="200.66" y="121.92" rot="R270"/>
-<instance part="TP28" gate="G$1" x="182.88" y="99.06" rot="R270"/>
+<instance part="TP25" gate="G$1" x="185.42" y="137.16" rot="R270"/>
+<instance part="TP26" gate="G$1" x="185.42" y="129.54" rot="R270"/>
+<instance part="TP27" gate="G$1" x="198.12" y="121.92" rot="R180"/>
+<instance part="TP28" gate="G$1" x="180.34" y="99.06" rot="R180"/>
 <instance part="FRAME1" gate="G$1" x="190.5" y="-114.3"/>
 <instance part="D1" gate="G$1" x="-55.88" y="-63.5" rot="R270"/>
@@
 <instance part="F2" gate="A" x="-40.64" y="-22.86"/>
 <instance part="+3V3" gate="G$1" x="-104.14" y="-55.88"/>
-<instance part="TP4" gate="G$1" x="-116.84" y="-30.48" rot="R90"/>
-<instance part="TP29" gate="G$1" x="-114.3" y="-17.78"/>
-<instance part="TP30" gate="G$1" x="-101.6" y="-63.5" rot="R270"/>
+<instance part="TP4" gate="G$1" x="-114.3" y="-30.48"/>
+<instance part="TP29" gate="G$1" x="-114.3" y="-20.32" rot="R270"/>
+<instance part="TP30" gate="G$1" x="-104.14" y="-63.5" rot="R180"/>
 <instance part="P+1" gate="1" x="-121.92" y="-12.7"/>
 <instance part="U2" gate="G$1" x="-88.9" y="78.74"/>
@@
 <instance part="P+13" gate="1" x="-63.5" y="142.24"/>
 <instance part="GND18" gate="1" x="-58.42" y="116.84"/>
-<instance part="TP8" gate="G$1" x="-134.62" y="73.66" rot="R180"/>
-<instance part="TP9" gate="G$1" x="-121.92" y="78.74" rot="R180"/>
-<instance part="TP32" gate="G$1" x="-114.3" y="83.82" rot="R90"/>
-<instance part="TP33" gate="G$1" x="-116.84" y="68.58" rot="R90"/>
-<instance part="TP34" gate="G$1" x="-38.1" y="91.44" rot="R270"/>
-<instance part="TP35" gate="G$1" x="-134.62" y="134.62" rot="R180"/>
+<instance part="TP8" gate="G$1" x="-134.62" y="76.2" rot="R90"/>
+<instance part="TP9" gate="G$1" x="-121.92" y="81.28" rot="R90"/>
+<instance part="TP32" gate="G$1" x="-111.76" y="83.82"/>
+<instance part="TP33" gate="G$1" x="-114.3" y="68.58"/>
+<instance part="TP34" gate="G$1" x="-40.64" y="91.44" rot="R180"/>
+<instance part="TP35" gate="G$1" x="-134.62" y="137.16" rot="R90"/>
 <instance part="J1" gate="G$1" x="-116.84" y="127"/>
 <instance part="C4" gate="G$1" x="43.18" y="-50.8"/>
@@
 <attribute name="VALUE" x="135.255" y="-70.612" size="1.27" layer="96" rot="R90"/>
 </instance>
-<instance part="TP5" gate="G$1" x="144.78" y="-50.8" rot="R180"/>
-<instance part="TP6" gate="G$1" x="40.64" y="-63.5" smashed="yes" rot="R90">
-<attribute name="NAME" x="39.37" y="-64.77" size="1.778" layer="95" rot="R270"/>
-<attribute name="TP_SIGNAL_NAME" x="41.91" y="-62.23" size="1.778" layer="97" rot="R90"/>
-</instance>
-<instance part="TP7" gate="G$1" x="40.64" y="-48.26" smashed="yes" rot="R90">
+<instance part="TP5" gate="G$1" x="144.78" y="-48.26" rot="R90"/>
+<instance part="TP6" gate="G$1" x="43.18" y="-63.5" smashed="yes">
+<attribute name="NAME" x="41.91" y="-62.23" size="1.778" layer="95" rot="R180"/>
+<attribute name="TP_SIGNAL_NAME" x="44.45" y="-64.77" size="1.778" layer="97"/>
+</instance>
+<instance part="TP7" gate="G$1" x="43.18" y="-48.26" smashed="yes">
 <attribute name="NAME" x="41.91" y="-46.99" size="1.778" layer="95" rot="R90"/>
-<attribute name="TP_SIGNAL_NAME" x="41.91" y="-46.99" size="1.778" layer="97" rot="R90"/>
+<attribute name="TP_SIGNAL_NAME" x="44.45" y="-49.53" size="1.778" layer="97"/>
 </instance>
 <instance part="SJ2" gate="1" x="137.16" y="-48.26"/>
@@
 <wire x1="101.6" y1="93.98" x2="101.6" y2="109.22" width="0.1524" layer="91"/>
 <pinref part="GND13" gate="1" pin="GND"/>
-<wire x1="101.6" y1="93.98" x2="104.14" y2="93.98" width="0.1524" layer="91"/>
+<wire x1="101.6" y1="93.98" x2="106.68" y2="93.98" width="0.1524" layer="91"/>
 <junction x="101.6" y="93.98"/>
 <pinref part="TP15" gate="G$1" pin="TP"/>
-<junction x="104.14" y="93.98"/>
+<junction x="106.68" y="93.98"/>
+<wire x1="104.14" y1="93.98" x2="106.68" y2="93.98" width="0.1524" layer="91"/>
 </segment>
 <segment>
@@
 <pinref part="GND16" gate="1" pin="GND"/>
 <pinref part="C10" gate="G$1" pin="2"/>
-<wire x1="55.88" y1="17.78" x2="53.34" y2="17.78" width="0.1524" layer="91"/>
+<wire x1="55.88" y1="17.78" x2="50.8" y2="17.78" width="0.1524" layer="91"/>
 <junction x="55.88" y="17.78"/>
 <pinref part="TP24" gate="G$1" pin="TP"/>
-<junction x="53.34" y="17.78"/>
+<junction x="50.8" y="17.78"/>
+<wire x1="53.34" y1="17.78" x2="50.8" y2="17.78" width="0.1524" layer="91"/>
 </segment>
 <segment>
