File: proj/rj12-adapter/v1.1/rj12_adapter.sch (EAGLE design)
At the start: 64 parts, among them J1 54602-908LF, J2 A-2004-1-4-LP-N-R, J3 54602-908LF, J4 A-2004-1-4-LP-N-R, U1 R-78E5.0-1.0, U2 PCA9615, U4 LM2937-3.3V, U5 PCA9615

Commit message: finalized rj12 adapter v1.1
Other:
- note added: "Changelog - changed 24v-to-5v regulator to R78E5 - changed rj45 pair to use x2 dI2C buffers - updated to latest style & naming conventions"
Changed lines of the file:
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@@
 <text x="248.92" y="224.155" size="3.048" layer="97">RJ12 Connectors</text>
 <text x="314.96" y="220.98" size="3.048" layer="103">Testpads</text>
+<text x="381" y="76.2" size="3.048" layer="97">Changelog
+ - changed 24v-to-5v regulator to R78E5
+ - changed rj45 pair to use x2 dI2C buffers
+ - updated to latest style &amp; naming conventions</text>
 </plain>
 <instances>

Commit message: fixed name issue on rj12 adapter v1.1
Parts:
- U$7: TITLE RJ45 to RJ12 Adapter -> RJ12 to RJ45 Adapter; URL https://github.com/openaginitiative/openag_eagle/proj/rj45-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 -> https://github.com/openaginitiative/openag_eagle/proj/rj12-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
Changed lines of the file:
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@@
 </part>
 <part name="U$7" library="openag-frames" deviceset="TITLE" device="">
-<attribute name="TITLE" value="RJ45 to RJ12 Adapter"/>
-<attribute name="URL" value="https://github.com/openaginitiative/openag_eagle/proj/rj45-adapter"/>
+<attribute name="TITLE" value="RJ12 to RJ45 Adapter"/>
+<attribute name="URL" value="https://github.com/openaginitiative/openag_eagle/proj/rj12-adapter"/>
 <attribute name="VER" value="1.1"/>
 </part>

Commit message: progress on light controller v2.1
Other:
- moved on the sheet: C1, C2, C3, C6, C9, D2, D4, J2, J4, L1, R1, R4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
