File: proj/rj12-adapter/v1.1/rj12_adapter.brd (EAGLE design)
At the start: 85.1 x 57.1 mm, 70 parts, among them J1 54602-908LF, J2 A-2004-1-4-LP-N-R, J3 54602-908LF, J4 A-2004-1-4-LP-N-R, U1 R-78E5.0-1.0, U2 PCA9615, U4 LM2937-3.3V, U5 PCA9615

Commit message: finalized rj12 adapter v1.1
Parts:
- U$9: device openag-frames:CAMBRIDGE-MAP-RJ45-ADAPTER-V-1-1 -> openag-frames:CAMBRIDGE-MAP-RJ12-ADAPTER-V-1-1
Changed lines of the file:
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@@
 <grid distance="50" unitdist="mil" unit="mil" style="lines" multiple="1" display="yes" altdistance="5" altunitdist="mil" altunit="mil"/>
 <layers>
-<layer number="1" name="Top" color="4" fill="1" visible="no" active="yes"/>
+<layer number="1" name="Top" color="4" fill="1" visible="yes" active="yes"/>
 <layer number="2" name="Route2" color="1" fill="3" visible="no" active="no"/>
 <layer number="3" name="Route3" color="4" fill="3" visible="no" active="no"/>
@@
 <layer number="14" name="Route14" color="1" fill="6" visible="no" active="no"/>
 <layer number="15" name="Route15" color="4" fill="6" visible="no" active="no"/>
-<layer number="16" name="Bottom" color="1" fill="1" visible="yes" active="yes"/>
+<layer number="16" name="Bottom" color="1" fill="1" visible="no" active="yes"/>
 <layer number="17" name="Pads" color="2" fill="1" visible="yes" active="yes"/>
 <layer number="18" name="Vias" color="2" fill="1" visible="yes" active="yes"/>
 <layer number="19" name="Unrouted" color="6" fill="1" visible="yes" active="yes"/>
 <layer number="20" name="Dimension" color="24" fill="1" visible="yes" active="yes"/>
-<layer number="21" name="tPlace" color="7" fill="1" visible="no" active="yes"/>
-<layer number="22" name="bPlace" color="7" fill="1" visible="yes" active="yes"/>
-<layer number="23" name="tOrigins" color="15" fill="1" visible="no" active="yes"/>
-<layer number="24" name="bOrigins" color="15" fill="1" visible="yes" active="yes"/>
-<layer number="25" name="tNames" color="7" fill="1" visible="no" active="yes"/>
-<layer number="26" name="bNames" color="7" fill="1" visible="yes" active="yes"/>
+<layer number="21" name="tPlace" color="7" fill="1" visible="yes" active="yes"/>
+<layer number="22" name="bPlace" color="7" fill="1" visible="no" active="yes"/>
+<layer number="23" name="tOrigins" color="15" fill="1" visible="yes" active="yes"/>
+<layer number="24" name="bOrigins" color="15" fill="1" visible="no" active="yes"/>
+<layer number="25" name="tNames" color="7" fill="1" visible="yes" active="yes"/>
+<layer number="26" name="bNames" color="7" fill="1" visible="no" active="yes"/>
 <layer number="27" name="tValues" color="7" fill="1" visible="no" active="yes"/>
 <layer number="28" name="bValues" color="7" fill="1" visible="no" active="yes"/>
@@
 <layer number="37" name="tTest" color="7" fill="1" visible="no" active="yes"/>
 <layer number="38" name="bTest" color="7" fill="1" visible="no" active="yes"/>
-<layer number="39" name="tKeepout" color="4" fill="11" visible="no" active="yes"/>
-<layer number="40" name="bKeepout" color="1" fill="11" visible="yes" active="yes"/>
-<layer number="41" name="tRestrict" color="4" fill="10" visible="no" active="yes"/>
-<layer number="42" name="bRestrict" color="1" fill="10" visible="yes" active="yes"/>
+<layer number="39" name="tKeepout" color="4" fill="11" visible="yes" active="yes"/>
+<layer number="40" name="bKeepout" color="1" fill="11" visible="no" active="yes"/>
+<layer number="41" name="tRestrict" color="4" fill="10" visible="yes" active="yes"/>
+<layer number="42" name="bRestrict" color="1" fill="10" visible="no" active="yes"/>
 <layer number="43" name="vRestrict" color="2" fill="10" visible="no" active="yes"/>
 <layer number="44" name="Drills" color="7" fill="1" visible="no" active="yes"/>
@@
 <layer number="49" name="Reference" color="7" fill="1" visible="no" active="yes"/>
 <layer number="50" name="dxf" color="7" fill="1" visible="no" active="no"/>
-<layer number="51" name="tDocu" color="7" fill="1" visible="no" active="yes"/>
-<layer number="52" name="bDocu" color="7" fill="1" visible="yes" active="yes"/>
+<layer number="51" name="tDocu" color="7" fill="1" visible="yes" active="yes"/>
+<layer number="52" name="bDocu" color="7" fill="1" visible="no" active="yes"/>
 <layer number="53" name="tGND_GNDA" color="7" fill="1" visible="no" active="no"/>
 <layer number="54" name="bGND_GNDA" color="7" fill="1" visible="no" active="no"/>
@@
 <wire x1="23.8125" y1="10.795" x2="26.3525" y2="10.795" width="0.1524" layer="21" style="shortdash"/>
 <wire x1="28.8925" y1="10.795" x2="31.4325" y2="10.795" width="0.1524" layer="21" style="shortdash"/>
-<text x="45.974" y="14.224" size="0.762" layer="22" rot="MR90">  EMI
+<text x="46.228" y="14.224" size="0.762" layer="22" rot="MR90">  EMI
 Bypass</text>
 <wire x1="81.28" y1="11.43" x2="81.28" y2="10.16" width="0.1524" layer="21"/>
@@
 <attribute name="MPN" value="R-78E5.0-1.0" x="46.99" y="25.4" size="0.762" layer="27" display="off"/>
 <attribute name="NAME" x="41.275" y="32.004" size="0.762" layer="25"/>
+<attribute name="VALUE" x="44.45" y="28.956" size="0.762" layer="27"/>
 <attribute name="VALUE" x="44.45" y="28.956" size="0.762" layer="21"/>
-<attribute name="VALUE" x="44.45" y="28.956" size="0.762" layer="27"/>
 <attribute name="VENDOR" value="Digikey" x="46.99" y="25.4" size="0.762" layer="27" display="off"/>
 <attribute name="VLINK" value="https://www.digikey.com/product-detail/en/recom-power/R-78E5.0-1.0/945-2201-ND/4930585" x="46.99" y="25.4" size="0.762" layer="27" display="off"/>
@@
 <attribute name="VPN" value="AE10383-ND" x="73.66" y="20.32" size="1.778" layer="27" display="off"/>
 </element>
-<element name="U$9" library="openag-frames" package="CAMBRIDGE-MAP-RJ45-ADAPTER-V-1-1" value="" x="1.27" y="1.27"/>
 <element name="U$1" library="openag-frames" package="CORNER" value="" x="5.08" y="5.08"/>
 <element name="U$2" library="openag-frames" package="CORNER" value="" x="5.08" y="52.07" rot="R270"/>
 <element name="U$3" library="openag-frames" package="CORNER" value="" x="80.01" y="52.07" rot="R180"/>
 <element name="U$4" library="openag-frames" package="CORNER" value="" x="80.01" y="5.08" rot="R90"/>
+<element name="U$9" library="openag-frames" package="CAMBRIDGE-MAP-RJ12-ADAPTER-V-1-1" value="" x="1.27" y="1.27"/>
 </elements>
 <signals>
@@
 <wire x1="25.4158" y1="33.274" x2="25.4" y2="33.2898" width="0.3048" layer="1"/>
 </signal>
-<signal name="N$4">
-<via x="-16.51" y="63.5" extent="1-16" drill="0.35"/>
-</signal>
 </signals>
