File: proj/atlas-port/double/v1.0/atlas_double.brd (EAGLE design)
At the start: 123.2 x 21.6 mm, 30 parts, among them J1 Atlas Stamp, J2 5227161-9, J3 I2C-HEADER, J4 5227161-9, J5 Atlas Stamp, J6 I2C-HEADER, U1 ISO1540, U2 RM-3.33.3S, U3 ISO1540, U4 RM-3.33.3S

Commit message: added atlas port double v1.0
Parts:
- removed FRAME1: (no value), openag-frames:DOCFIELD
- removed J3, J6: I2C-HEADER, openag-connectors:OPENAG-I2C-HEADER
- removed U$5: (no value), openag-frames:OPENAG-LOGO-750-MIL
- added J7: ATLAS-DOUBLE-CONN, openag-connectors:ATLAS-DOUBLE
- added U$1: (no value), openag-frames:HOLE-150
- J2, J4: device openag-connectors:BNC -> openag-connectors:BNC-5227161
- U$2: device openag-frames:OPENAG-CORNER-MOUNTING-HOLE -> openag-frames:HOLE-150
- U$3: device openag-frames:OPENAG-CORNER-MOUNTING-HOLE -> openag-frames:CAMBRIDGE-MAP-X1-ATLAS-DOUBLE-V-1-0
- U2, U4: device openag-isolators:SIP4 -> openag-isolators:RM3.33.3S-SIP4
- moved U$3 107.2 mm to (0.00, 0.00), turned to 0 degrees
- moved U$2 87.6 mm to (104.1, 10.8)
- moved J4 3.81 mm to (115.6, 10.8)
- moved C1 2.54 mm to (28.2, 6.10)
- moved C2 2.54 mm to (28.2, 15.0)
- moved J1 2.54 mm to (30.5, 10.8)
- moved C3 2.54 mm to (43.2, 9.14)
- moved C4 2.54 mm to (43.2, 14.2)
- moved R1 2.54 mm to (27.7, 9.91)
- moved R2 2.54 mm to (27.7, 8.64)
- moved R3 2.54 mm to (27.7, 12.4)
- moved R4 2.54 mm to (27.7, 11.2)
- moved U1 2.54 mm to (33.3, 11.2)
- moved U2 2.54 mm to (48.3, 6.99)
- moved U3 1.27 mm to (86.1, 10.4)
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Connections:
- net +3V3: now also J7.3V3@1, J7.3V3@2; no longer J3.3V3, J6.3V3
- net GND: now also J7.GND@1, J7.GND@2; no longer J3.GND, J6.GND
- net SCL: now also J7.SCL@1, J7.SCL@2; no longer J3.SCL, J6.SCL
- net SDA: now also J7.SDA@1, J7.SDA@2; no longer J3.SDA, J6.SDA
Routing:
- net PRB_2: track 20.1 -> 15.5 mm
- net PRB_1: track 20.1 -> 15.8 mm
- net PGND_2: track 16.5 -> 13.6 mm
- net PGND_1: track 16.5 -> 13.6 mm
- net ISO_GND_2: track 27.8 -> 30.2 mm
- net SDA: track 101.6 -> 103.9 mm
- net +3V3: track 96.6 -> 98.4 mm
- net SCL: track 89.6 -> 90.9 mm
- net GND: vias 12 -> 23
Other:
- board size 123.2 x 21.6 mm -> 119.4 x 21.6 mm
