File: proj/atlas-port/quad/v1.0/atlas_quad.sch (EAGLE design)
At the start: 105 parts, among them J11 PJ-036AH, J12 PJ-036AH, J13 5227161-9, J14 Atlas Stamp, J15 I2C-HEADER, J16 54602-908LF, J17 54602-908LF, J19 5227161-9, J20 Atlas Stamp, J21 I2C-HEADER, J4 5227161-9, J5 Atlas Stamp, J6 I2C-HEADER, J7 5227161-9, J8 Atlas Stamp, J9 I2C-HEADER, U10 ISO1540, U11 MIC4680YM-TR, U12 PCA9615DPJ, U13 RM-3.33.3S, U14 ISO1540, U3 RM-3.33.3S, U4 ISO1540, U5 RM-3.33.3S, U6 ISO1540, U8 LM2937IMP3.3NOPB, U9 RM-3.33.3S

Commit message: updated atlas port quad v1.0 manufacturing files
Parts:
- F5: value SST 7 -> SST7
- F6: device fuse:GSH15 -> openag-fuses:GSH15
- J16, J17: device openag_connector:OPENAG-V1-RJ45PTH -> openag-connectors:OPENAG-V1-RJ45PTH
- U11: value MIC4680YM-TR -> MIC4680
- U12: value PCA9615DPJ -> PCA9615
- U8: value LM2937IMP3.3NOPB -> LM2937
Changed lines of the file:
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@@
 <setting verticaltext="up"/>
 </settings>
-<grid distance="1.5" unitdist="inch" unit="inch" style="lines" multiple="1" display="yes" altdistance="0.01" altunitdist="inch" altunit="inch"/>
+<grid distance="0.1" unitdist="inch" unit="inch" style="lines" multiple="1" display="yes" altdistance="0.01" altunitdist="inch" altunit="inch"/>
 <layers>
 <layer number="1" name="Top" color="4" fill="1" visible="no" active="no"/>
@@
 <part name="FRAME1" library="openag-frames" deviceset="DOCFIELD" device="">
 <attribute name="AUTHOR" value="JR"/>
-<attribute name="DESCRIPTION" value=""/>
 <attribute name="TITLE" value="Atlas Port Quad"/>
 <attribute name="URL" value="https://github.com/OpenAgInitiative/openag_eagle/proj/atlas-port"/>
@@
 <part name="R30" library="openag-resistors" deviceset="100OHM-RC0603JR-07100RL" device="" value="100"/>
 <part name="GND26" library="openag-supply" deviceset="GND" device=""/>
-<part name="U8" library="openag-regulators" deviceset="LM2937IMP-3.3/NOPB" device="" value="LM2937IMP3.3NOPB"/>
+<part name="U8" library="openag-regulators" deviceset="LM2937IMP-3.3/NOPB" device="" value="LM2937"/>
 <part name="C16" library="openag-capacitors" deviceset="0.1UF-C0603C104K5RACTU" device="" value="0.1uF"/>
 <part name="GND27" library="openag-supply" deviceset="GND" device=""/>
@@
 <part name="C22" library="openag-capacitors" deviceset="15UF-C2012X5R1V156M125AC" device="" value="15uF"/>
 <part name="C23" library="openag-capacitors" deviceset="220UF-TPSY227K010R0100" device="" value="220uF"/>
-<part name="U11" library="openag-regulators" deviceset="MIC4680YM-TR" device="" value="MIC4680YM-TR"/>
+<part name="U11" library="openag-regulators" deviceset="MIC4680YM-TR" device="" value="MIC4680"/>
 <part name="L2" library="openag-inductors" deviceset="68UH-UP2B-680-R" device="" value="68uH"/>
 <part name="D6" library="openag-diodes" deviceset="SBR2A40P1-7" device="" value="SBR2A40P1-7"/>
@@
 <part name="SJ4" library="openag-connectors" deviceset="SOLDERJUMPER" device="REFLOW_NOPASTE"/>
 <part name="GND29" library="openag-supply" deviceset="GND" device=""/>
-<part name="F5" library="openag-fuses" deviceset="SST_7" device="" value="SST 7"/>
+<part name="F5" library="openag-fuses" deviceset="SST_7" device="" value="SST7"/>
 <part name="P+14" library="openag-supply" deviceset="+24V" device=""/>
-<part name="F6" library="fuse" library_urn="urn:adsk.eagle:library:233" deviceset="GSH15" device="" package3d_urn="urn:adsk.eagle:package:14065/1"/>
+<part name="F6" library="openag-fuses" deviceset="GSH15" device=""/>
 <part name="GND30" library="openag-supply" deviceset="GND" device=""/>
 <part name="GND31" library="openag-supply" deviceset="GND" device=""/>
@@
 <part name="TP12" library="openag-testpads" deviceset="TP" device="TP06R"/>
 <part name="D10" library="openag-diodes" deviceset="SMAJ26A-13-F" device="" value="SMAJ26A"/>
-<part name="U12" library="openag-buffers" deviceset="PCA9615DPJ" device="" value="PCA9615DPJ"/>
+<part name="U12" library="openag-buffers" deviceset="PCA9615DPJ" device="" value="PCA9615"/>
 <part name="R35" library="openag-resistors" deviceset="600OHM-RC0603FR-07604RL" device="" value="600"/>
 <part name="R36" library="openag-resistors" deviceset="120OHM-RC0603FR-07120RL" device="" value="120"/>
@@
 <part name="P+17" library="openag-supply" deviceset="+5V" device=""/>
 <part name="P+18" library="openag-supply" deviceset="+5V" device=""/>
-<part name="J16" library="openag_connector" deviceset="OPENAG-V1-RJ45" device="PTH" value="54602-908LF"/>
+<part name="J16" library="openag-connectors" deviceset="OPENAG-V1-RJ45" device="PTH" value="54602-908LF"/>
 <part name="GND38" library="openag-supply" deviceset="GND" device=""/>
 <part name="TP13" library="openag-testpads" deviceset="TP" device="TP06R"/>
@@
 <part name="TP17" library="openag-testpads" deviceset="TP" device="TP06R"/>
 <part name="TP18" library="openag-testpads" deviceset="TP" device="TP06R"/>
-<part name="J17" library="openag_connector" deviceset="OPENAG-V1-RJ45" device="PTH" value="54602-908LF"/>
+<part name="J17" library="openag-connectors" deviceset="OPENAG-V1-RJ45" device="PTH" value="54602-908LF"/>
 <part name="P+19" library="openag-supply" deviceset="+24V" device=""/>
 <part name="P+20" library="openag-supply" deviceset="+24V" device=""/>
@@
 <instance part="TP9" gate="G$1" x="271.78" y="-139.7" smashed="yes">
 <attribute name="NAME" x="267.97" y="-140.97" size="1.778" layer="95" rot="R270"/>
-<attribute name="TP_SIGNAL_NAME" x="273.05" y="-140.97" size="1.778" layer="97"/>
 </instance>
 <instance part="TP10" gate="G$1" x="271.78" y="-124.46" smashed="yes">
 <attribute name="NAME" x="270.51" y="-123.19" size="1.778" layer="95" rot="R90"/>
-<attribute name="TP_SIGNAL_NAME" x="273.05" y="-125.73" size="1.778" layer="97"/>
 </instance>
 <instance part="SJ4" gate="1" x="365.76" y="-124.46"/>
@@
 which will not be processed correctly with this version.
 </note>
-<note version="8.2" severity="warning">
-Since Version 8.2, EAGLE supports online libraries. The ids
-of those online libraries will not be understood (or retained)
-with this version.
-</note>
-<note version="8.3" severity="warning">
-Since Version 8.3, EAGLE supports URNs for individual library
-assets (packages, symbols, and devices). The URNs of those assets
-will not be understood (or retained) with this version.
-</note>
-<note version="8.3" severity="warning">
-Since Version 8.3, EAGLE supports the association of 3D packages
-with devices in libraries, schematics, and board files. Those 3D
-packages will not be understood (or retained) with this version.
-</note>
 </compatibility>

Commit message: added photon quad v1.0 at 90%
Parts:
- removed C29: 4.7uF, openag-capacitors:4.7UF-CL21A475KBQNNNE
- removed C30, C8: 0.1uF, openag-capacitors:0.1UF-C0603C104K5RACTU
- removed D10: SMAJ26A, openag-diodes:SMAJ26A-13-F
- removed D8, D9: APT1608, openag-diodes:APT1608CGCK
- removed F4: 0448.400MR, openag-fuses:0438.375WR
- removed F5: SST7, openag-fuses:SST_7
- removed F6: (no value), openag-fuses:GSH15
- removed FRAME1: (no value), openag-frames:DOCFIELD
- removed J11, J12: PJ-036AH, openag-connectors:PJ-036AH-SMT-TR
- removed J16, J17: 54602-908LF, openag-connectors:OPENAG-V1-RJ45PTH
- removed R20: 1K, openag-resistors:1K-ERJ-PB3D1001V
- removed R30, R33, R34: 100, openag-resistors:100OHM-RC0603JR-07100RL
- removed R31: 3.01K, openag-resistors:3.01K-RC0603FR-073K01L
- removed R32: 976 Ohm, openag-resistors:982OHM-RC0603FR-07976RL
- removed R35, R37, R38, R39: 600, openag-resistors:600OHM-RC0603FR-07604RL
- removed R36, R40: 120, openag-resistors:120OHM-RC0603FR-07120RL
- removed R41, R42: 10K, openag-resistors:10K-ERJ-3EKF1002V
- removed SJ4: (no value), openag-connectors:SOLDERJUMPERREFLOW_NOPASTE
- removed TP16: TPTP06R, openag-testpads:TPTP06R
- removed U11: MIC4680, openag-regulators:MIC4680YM-TR
- added C1, C14, C2, C3, C4: 0.1uF, openag-capacitors:0.1UF-C0603C104K5RACTU
- added C15: 10uF, openag-capacitors:10UF-GMK212BBJ106KG-T
- added D1, D4: APT1608, openag-diodes:APT1608CGCK
- added D3: SMAJ26A, openag-diodes:SMAJ26A-13-F
- added F1, F2: SSQ5, openag-fuses:SSQ5
- added J1: 5227161-9, openag-connectors:BNC-5227161-9PTH
- added J10: 54602-908LF, openag-connectors:RJ45-DI2C-USB-54602-908LFPTH
- added J2: I2C-HEADER, openag-connectors:HEADER-I2C
- added J3: ATLAS-STAMP, openag-connectors:ATLAS-STAMP
- added R1, R2, R23, R24: 2.2k, openag-resistors:2.2K-RC0603JR-072K2L
- added R13: 1K, openag-resistors:1K-ERJ-PB3D1001V
- added R14, R15, R16, R3: 600, openag-resistors:600OHM-RC0603FR-07604RL
- added R21, R22: 100, openag-resistors:100OHM-RC0603JR-07100RL
- added R4: 120, openag-resistors:120OHM-RC0603FR-07120RL
- added TP19, TP20, TP28, TP29, TP30, TP31, TP32, TP4, TP5, TP58, TP6, TP7, TP71, TP72, TP73: TPTP04R, openag-testpads:TPTP04R
- added TP23, TP24, TP25: TPTP06R, openag-testpads:TPTP06R
- added U$5: AUTHOR, openag-frames:AUTHOR
- added U$6: TITLE, openag-frames:TITLE
- added U1: ISO1540, openag-isolators:ISO1540DR
- added U2: RM-3.33.3S, openag-isolators:RM3.33.3S
- added U7: LM2937-3.3V, openag-regulators:LM2937IMP-3.3/NOPB
- C20, C5: value 0.1uF -> 10uF; device openag-capacitors:0.1UF-C0603C104K5RACTU -> openag-capacitors:10UF-GMK212BBJ106KG-T
- C22: value 15uF -> 10uF; device openag-capacitors:15UF-C2012X5R1V156M125AC -> openag-capacitors:10UF-GMK212BBJ106KG-T
- C23: value 220uF -> 0.1uF; device openag-capacitors:220UF-TPSY227K010R0100 -> openag-capacitors:0.1UF-C0603C104K5RACTU
- C24: value 10uF -> 0.1uF; device openag-capacitors:10UF-GMK212BBJ106KG-T -> openag-capacitors:0.1UF-C0603C104K5RACTU
- C28, C6: value 0.1uF -> 4.7uF; device openag-capacitors:0.1UF-C0603C104K5RACTU -> openag-capacitors:4.7UF-CL21A475KBQNNNE
- D6: value SBR2A40P1-7 -> APT1608; device openag-diodes:SBR2A40P1-7 -> openag-diodes:APT1608CGCK
- J13, J19, J7: value 5227161-9 -> ATLAS-STAMP; device openag-connectors:BNC-5227161-9PTH -> openag-connectors:ATLAS-STAMP
- J14, J20, J8: value Atlas Stamp -> I2C-HEADER; device openag-connectors:ATLAS-STAMP -> openag-connectors:HEADER-I2C
- J15, J21, J9: value I2C-HEADER -> 5227161-9; device openag-connectors:OPENAG-I2C-HEADER -> openag-connectors:BNC-5227161-9PTH
- J4: value 5227161-9 -> PJ-036AH; device openag-connectors:BNC-5227161-9PTH -> openag-connectors:BARREL-JACK-PJ-036AH-SMT-TR
- J5: value Atlas Stamp -> PJ-036AH; device openag-connectors:ATLAS-STAMP -> openag-connectors:BARREL-JACK-PJ-036AH-SMT-TR
- J6: value I2C-HEADER -> 54602-908LF; device openag-connectors:OPENAG-I2C-HEADER -> openag-connectors:RJ45-DI2C-USB-54602-908LFPTH
- L2: value 68uH -> 33uH; device openag-inductors:68UH-UP2B-680-R -> openag-inductors:33UH-29333C
- R10, R18, R19: value 1K -> 120; device openag-resistors:1K-ERJ-PB3D1001V -> openag-resistors:120OHM-RC0603FR-07120RL
- R11, R12: value 1K -> 10K; device openag-resistors:1K-ERJ-PB3D1001V -> openag-resistors:10K-ERJ-3EKF1002V
- R17, R7, R8, R9: value 1K -> 600; device openag-resistors:1K-ERJ-PB3D1001V -> openag-resistors:600OHM-RC0603FR-07604RL
- R25: value 1K -> 0 OHM; device openag-resistors:1K-ERJ-PB3D1001V -> openag-resistors:0OHM-RC0603JR-070RL
- R26: value 1K -> 100; device openag-resistors:1K-ERJ-PB3D1001V -> openag-resistors:100OHM-RC0603JR-07100RL
- R27, R28, R5, R6: value 1K -> 2.2k; device openag-resistors:1K-ERJ-PB3D1001V -> openag-resistors:2.2K-RC0603JR-072K2L
- SJ1: device openag-connectors:SOLDERJUMPERREFLOW_NOPASTE -> openag-connectors:EMI-BYPASS
- TP1, TP10, TP11, TP12, TP13, TP14, TP15, TP17, TP18, TP2, TP3, TP8, TP9: value TPTP06R -> TPTP04R; device openag-testpads:TPTP06R -> openag-testpads:TPTP04R
- U12: value PCA9615 -> PHOTONH; device openag-buffers:PCA9615DPJ -> openag-microcontrollers:PHOTONHPHOTONH
- U3: value RM-3.33.3S -> PCA9615; device openag-isolators:RM3.33.3S -> openag-buffers:PCA9615DPJ
- U4: value ISO1540 -> PCA9615; device openag-isolators:ISO1540DR -> openag-buffers:PCA9615DPJ
- U8: value LM2937 -> R-78E5.0-1.0; device openag-regulators:LM2937IMP-3.3/NOPB -> openag-regulators:R-78E5.0-1.0
Connections:
- removed net 24V_IN: F5.1, F6.1, J11.1, J12.1
- removed net DSCLM: J16.DSCLM, J17.DSCLM, R39.2, R40.1, U12.DSCLM
- removed net DSCLP: J16.DSCLP, J17.DSCLP, R38.1, R40.2, U12.DSCLP
- removed net DSDAM: J16.DSDAM, J17.DSDAM, R35.1, R36.2, U12.DSDAM
- removed net DSDAP: J16.DSDAP, J17.DSDAP, R36.1, R37.2, U12.DSDAP
- removed net N$27: D8.A, R33.1
- removed net N$45: C23.1(+), L2.2, R31.2, R33.2, SJ4.1
- removed net N$46: D9.A, R34.1
- removed net REG_3V3_400MA: F4.2, R30.2, SJ1.1
- new net 24V_EMI: C15.1, L2.2, SJ1.2, U8.VIN
- new net 24V_IN1: F2.1, J5.1
- new net 24V_IN2: F1.1, J4.1
- new net DSCLM_1: J6.DSCLM, R10.1, R9.2, U3.DSCLM
- new net DSCLM_2: J10.DSCLM, R16.2, R18.1, U4.DSCLM
- new net DSCLP_1: J6.DSCLP, R10.2, R8.1, U3.DSCLP
- new net DSCLP_2: J10.DSCLP, R17.1, R18.2, U4.DSCLP
- new net DSDAM_1: J6.DSDAM, R3.1, R4.2, U3.DSDAM
- new net DSDAM_2: J10.DSDAM, R14.1, R19.2, U4.DSDAM
- new net DSDAP_1: J6.DSDAP, R4.1, R7.2, U3.DSDAP
- new net DSDAP_3: J10.DSDAP, R15.2, R19.1, U4.DSDAP
- new net N$4: R25.2, U12.VIN
- new net N$5: D1.A, R13.1
- net +24V: now also C21.1, C5.1, C6.1, C7.1, D3.P$2, F1.2, F2.2, J10.+24V, J6.+24V, L2.1, R13.2, R21.2, SJ1.1, TP11.TP, TP17.TP, TP20.TP, TP24.TP, TP4.TP; no longer C22.1, C24.1, C29.1, C30.1, D10.P$2, F5.2, F6.2, J16.+24V, J17.+24V, R34.2, TP10.TP, TP12.TP, TP18.TP, U11.IN
- net +3V3: now also C1.1, C16.1, C18.1, C22.1, C23.1, C24.1, C26.1, C28.1, C3.1, J14.3V3, J2.3V3, J20.3V3, J8.3V3, R11.2, R12.2, TP1.TP, TP28.TP, TP31.TP, TP71.TP, TP9.TP, U1.VCC, U10.VCC, U12.3V3, U14.VCC, U2.+VIN, U3.VDD_(A), U4.VDD_(A), U6.VCC, U7.OUT; no longer C17.1, C19.1, C25.1, C27.1, C5.1, C7.1, J15.3V3, J21.3V3, J6.3V3, J9.3V3, R10.2, R17.2, R18.2, R25.2, R41.2, R42.2, R5.2, R6.2, R9.2, SJ1.2, TP15.TP, TP3.TP, U10.VCC1, U12.VDD_(A), U14.VCC1, U3.+VIN, U4.VCC1, U6.VCC1
- net +5V: now also C14.1, C20.1, R15.1, R17.2, R22.2, R25.1, R7.1, R8.2, TP10.TP, TP23.TP, TP29.TP, U3.VDD_(B), U4.VDD_(B), U7.IN, U8.VOUT; no longer C16.1, R37.1, R38.2, SJ4.2, TP17.TP, TP8.TP, U12.VDD_(B), U8.IN
- net GND: now also C1.2, C14.2, C15.2, C18.2, C20.2, C23.2, C26.2, C28.2, C3.2, C6.2, D1.C, D3.P$1, D4.C, D6.C, J10.GND, J14.GND, J2.GND, J20.GND, J4.2, J4.3, J5.2, J5.3, J8.GND, R14.2, R16.1, R3.2, R9.1, TP12.TP, TP15.TP, TP18.TP, TP19.TP, TP25.TP, TP3.TP, TP30.TP, TP32.TP, TP72.TP, U1.GND, U10.GND, U12.GND@2, U14.GND, U2.-VIN, U3.VSS, U4.VSS, U6.GND, U7.GND, U7.TAB; no longer C17.2, C19.2, C23.2(-), C25.2, C27.2, C29.2, C30.2, D10.P$1, D6.21, D8.C, D9.C, J11.2, J11.3, J12.2, J12.3, J15.GND, J16.GND, J17.GND, J21.GND, J9.GND, R32.1, R35.2, R39.1, TP1.TP, TP11.TP, TP16.TP, TP9.TP, U10.GND1, U11.GND, U11.SHDN, U12.VSS, U14.GND1, U3.-VIN, U4.GND1, U6.GND1, U8.TAB
- net ISO_3V3_1: now also C2.1, C4.1, J3.VCC, R1.2, R2.2, U1.ISO_VCC, U2.+VOUT; no longer C6.1, C8.1, J5.VCC, R7.2, R8.2, U3.+VOUT, U4.VCC2
- net ISO_3V3_2: now also J7.VCC, R5.2, R6.2, U6.ISO_VCC; no longer J8.VCC, R11.2, R12.2, U6.VCC2
- net ISO_3V3_3: now also C17.1, C19.1, J13.VCC, R23.2, R24.2, U10.ISO_VCC; no longer C18.1, C20.1, J14.VCC, R19.2, R20.2, U10.VCC2
- net ISO_3V3_4: now also C25.1, C27.1, J19.VCC, U14.ISO_VCC; no longer C26.1, C28.1, J20.VCC, U14.VCC2
- net ISO_GND_1: now also C2.2, C4.2, J3.GND, U1.ISO_GND, U2.-VOUT; no longer C6.2, C8.2, J5.GND, U3.-VOUT, U4.GND2
- net ISO_GND_2: now also J7.GND, U6.ISO_GND; no longer J8.GND, U6.GND2
- net ISO_GND_3: now also C17.2, C19.2, J13.GND, U10.ISO_GND; no longer C18.2, C20.2, J14.GND, U10.GND2
- net ISO_GND_4: now also C25.2, C27.2, J19.GND, U14.ISO_GND; no longer C26.2, C28.2, J20.GND, U14.GND2
- net ISO_SCL_1: now also J3.RX/SCL, R2.1, U1.ISO_SCL; no longer J5.RX/SCL, R8.1, U4.SCL2
- net ISO_SCL_2: now also J7.RX/SCL, R5.1, U6.ISO_SCL; no longer J8.RX/SCL, R12.1, U6.SCL2
- net ISO_SCL_3: now also J13.RX/SCL, R23.1, U10.ISO_SCL; no longer J14.RX/SCL, R20.1, U10.SCL2
- net ISO_SCL_4: now also J19.RX/SCL, R27.1, U14.ISO_SCL; no longer J20.RX/SCL, R28.1, U14.SCL2
- net ISO_SDA_1: now also J3.TX/SDA, R1.1, U1.ISO_SDA; no longer J5.TX/SDA, R7.1, U4.SDA2
- net ISO_SDA_2: now also J7.TX/SDA, R6.1, U6.ISO_SDA; no longer J8.TX/SDA, R11.1, U6.SDA2
- net ISO_SDA_3: now also J13.TX/SDA, R24.1, U10.ISO_SDA; no longer J14.TX/SDA, R19.1, U10.SDA2
- net ISO_SDA_4: now also J19.TX/SDA, R28.1, U14.ISO_SDA; no longer J20.TX/SDA, R27.1, U14.SDA2
- net N$11: now also D6.A, R26.1; no longer D6.12, L2.1, R31.1, R32.2, U11.FB, U11.SW
- net N$6: now also R21.1; no longer R30.1
- net N$8: now also D4.A, R22.1; no longer C21.1, F4.1, U8.OUT
- net PGND_1: now also J1.GND, J3.PGND; no longer J4.GND, J5.PGND
- net PGND_2: now also J7.PGND, J9.GND; no longer J7.GND, J8.PGND
- net PGND_3: now also J13.PGND, J15.GND; no longer J13.GND, J14.PGND
- net PGND_4: now also J19.PGND, J21.GND; no longer J19.GND, J20.PGND
- net PRB_1: now also J1.OUT, J3.PBR; no longer J4.OUT, J5.PBR
- net PRB_2: now also J7.PBR, J9.OUT; no longer J7.OUT, J8.PBR
- net PRB_3: now also J13.PBR, J15.OUT; no longer J13.OUT, J14.PBR
- net PRB_4: now also J19.PBR, J21.OUT; no longer J19.OUT, J20.PBR
- net SCL: now also J14.SCL, J2.SCL, J20.SCL, J8.SCL, R12.1, TP58.TP, TP6.TP, U1.SCL, U10.SCL, U12.D1, U14.SCL, U3.SCL, U4.SCL, U6.SCL; no longer J15.SCL, J21.SCL, J6.SCL, J9.SCL, R17.1, R25.1, R42.1, R5.1, R9.1, U10.SCL1, U12.SCL, U14.SCL1, U4.SCL1, U6.SCL1
- net SDA: now also J14.SDA, J2.SDA, J20.SDA, J8.SDA, R11.1, TP5.TP, TP73.TP, U1.SDA, U10.SDA, U12.D0, U14.SDA, U3.SDA, U4.SDA, U6.SDA; no longer J15.SDA, J21.SDA, J6.SDA, J9.SDA, R10.1, R18.1, R26.1, R41.1, R6.1, U10.SDA1, U12.SDA, U14.SDA1, U4.SDA1, U6.SDA1
- net USBM: now also J10.USBM, J6.USBM, TP8.TP; no longer J16.USBM, J17.USBM
- net USBP: now also J10.USBP, J6.USBP, TP7.TP; no longer J16.USBP, J17.USBP
Other:
- note added: "24V Power Conditioning"
- note added: "24V to 5V@1A Switching Regulator w/Optional EMI Filter + Indicator LED"
- note added: "5V to 3.3V@400mA Linear Regulator w/Indicator LED"
- note added: "Atlas Sensor Port w/Header"
- note added: "Barrel Jack Connector Pair w/24V Conditioning + Fuse + LED"
- note added: "I2C Header"
- note added: "I2C Pullup"
- note added: "Linear Regulator"
- note added: "Note: - Barrel jack rated for 5A"
- note added: "Optional EMI Filter (Class B)"
- note added: "Particle Photon"
- note added: "RJ45 Connector Pair w/dI2C Buffer"
- note added: "Switching Regulator"
- note added: "Testpads"
- note added: "dI2C Buffer Channel 1"
- note added: "dI2C Buffer Channel 2"
- note removed: "24V Power Conditioning + Fuse"
- note removed: "24V to 5V@1A Switching Regulator w/Indicator LED + Enable"
- note removed: "3.3V Enable Jumper"
- note removed: "3.3V Indicator LED"
- note removed: "3.3V@400mA Regulator"
- note removed: "5-26V to 3.3V@400mA Regulator w/3v3 Enable, Indicator LED & Fuse"
- note removed: "Atlas Sensor Port Quad"
- note removed: "Atlas Sensor Port w/Mount"
- note removed: "Barrel Jack Connector Pair with 24V Conditioning + Fuse + Indicator LED"
- note removed: "RJ45 Connector w/dI2C Buffer"
- note removed: "dI2C Buffer"
