File: proj/light-controller/v2.1/light_controller.brd (EAGLE design)
At the start: 132.1 x 116.8 mm, 152 parts, among them J1 0022232051, J10 PJ-036AH, J5 OPENAG-RS485-RJ12, J6 OPENAG-RS485-RJ12, J7 I2C-HEADER, J9 PJ-036AH, U1 RCD-24-0.70/VREF, U10 ADM2481BRWZ-RL7, U12 LM2937, U14 PCA9685, U16 MIC4680, U2 RCD-24-0.70/VREF, U3 RCD-24-0.70/VREF, U4 RCD-24-0.70/VREF, U5 RCD-24-0.70/VREF, U6 RCD-24-0.70/VREF, U7 DAC5578, U9 CY8C4124PVI-432

Commit message: experimenting with back cambridge map artwork
Parts:
- added C19, C20, C24, C25, C30, C34: 2.2uF, openag-capacitors:C0603
Connections:
- net GND: now also C19.2, C20.2, C24.2, C25.2, C30.2, C34.2
- net VIN1: now also C34.1
- net VIN2: now also C30.1
- net VIN3: now also C25.1
- net VIN4: now also C24.1
- net VIN5: now also C20.1
- net VIN6: now also C19.1
Changed lines of the file:
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@@
 <attribute name="NAME" x="19.685" y="81.153" size="1.016" layer="25" ratio="10" rot="R270"/>
 <attribute name="POPULATE" value="YES" x="15.875" y="74.803" size="1.778" layer="27" rot="R270" display="off"/>
+<attribute name="VALUE" x="14.097" y="71.501" size="1.016" layer="27" ratio="10" rot="R90"/>
 <attribute name="VALUE" value="0022232051" x="15.875" y="74.803" size="1.778" layer="27" rot="R270" display="off"/>
-<attribute name="VALUE" x="14.097" y="71.501" size="1.016" layer="27" ratio="10" rot="R90"/>
 <attribute name="VERIFIED" value="NO" x="15.875" y="74.803" size="1.778" layer="27" rot="R270" display="off"/>
 </element>
@@
 <attribute name="TITLE" value="Light Controller" x="77.724" y="60.6425" size="1.27" layer="22" rot="MR0"/>
 <attribute name="URL" value="github.com/OpenAgInitiative/openag_eagle/proj/light_controller" x="78.359" y="57.3405" size="0.7112" layer="22" rot="MR0"/>
-<attribute name="VER" value="2.0" x="51.054" y="60.6425" size="1.27" layer="22" rot="MR0"/>
+<attribute name="VER" value="2.1" x="51.054" y="60.6425" size="1.27" layer="22" rot="MR0"/>
 </element>
 <element name="R6" library="openag-resistors" package="RC0603N" value="1K" x="99.314" y="54.61" smashed="yes" rot="R270">
@@
 <attribute name="MPN" value="N/A" x="117.348" y="34.29" size="1.778" layer="28" rot="MR90" display="off"/>
 </element>
+<element name="C19" library="openag-capacitors" package="C0603" value="2.2uF" x="2.54" y="-12.7"/>
+<element name="C20" library="openag-capacitors" package="C0603" value="2.2uF" x="2.54" y="-17.78"/>
+<element name="C24" library="openag-capacitors" package="C0603" value="2.2uF" x="2.54" y="-22.86"/>
+<element name="C25" library="openag-capacitors" package="C0603" value="2.2uF" x="2.54" y="-27.94"/>
+<element name="C30" library="openag-capacitors" package="C0603" value="2.2uF" x="2.54" y="-33.02"/>
+<element name="C34" library="openag-capacitors" package="C0603" value="2.2uF" x="2.54" y="-38.1"/>
 </elements>
 <signals>
@@
 <via x="28.702" y="35.052" extent="1-16" drill="0.35"/>
 <wire x1="28.702" y1="38.608" x2="28.702" y2="35.052" width="0.5588" layer="16"/>
+<contactref element="C34" pad="1"/>
+<wire x1="28.575" y1="26.25" x2="1.69" y2="-38.1" width="0" layer="19" extent="1-1"/>
 </signal>
 <signal name="DIM1">
@@
 <via x="58.928" y="71.628" extent="1-16" drill="0.35"/>
 <via x="58.928" y="79.248" extent="1-16" drill="0.35"/>
+<contactref element="C19" pad="2"/>
+<contactref element="C20" pad="2"/>
+<contactref element="C24" pad="2"/>
+<contactref element="C25" pad="2"/>
+<contactref element="C30" pad="2"/>
+<contactref element="C34" pad="2"/>
 <wire x1="107.8865" y1="68.834" x2="102.9035" y2="67.691" width="0" layer="19" extent="1-1"/>
+<wire x1="3.39" y1="-12.7" x2="31.75" y2="0.762" width="0" layer="19" extent="1-1"/>
+<wire x1="3.39" y1="-17.78" x2="3.39" y2="-12.7" width="0" layer="19" extent="1-1"/>
+<wire x1="3.39" y1="-22.86" x2="3.39" y2="-17.78" width="0" layer="19" extent="1-1"/>
+<wire x1="3.39" y1="-27.94" x2="3.39" y2="-22.86" width="0" layer="19" extent="1-1"/>
+<wire x1="3.39" y1="-33.02" x2="3.39" y2="-27.94" width="0" layer="19" extent="1-1"/>
+<wire x1="3.39" y1="-38.1" x2="3.39" y2="-33.02" width="0" layer="19" extent="1-1"/>
 </signal>
 <signal name="VIN2">
@@
 <via x="44.958" y="35.052" extent="1-16" drill="0.35"/>
 <wire x1="44.958" y1="38.608" x2="44.958" y2="35.052" width="0.5588" layer="16"/>
+<contactref element="C30" pad="1"/>
+<wire x1="45.085" y1="26.25" x2="1.69" y2="-33.02" width="0" layer="19" extent="1-1"/>
 </signal>
 <signal name="DIM2">
@@
 <via x="61.468" y="35.052" extent="1-16" drill="0.35"/>
 <wire x1="61.468" y1="38.608" x2="61.468" y2="35.052" width="0.5588" layer="16"/>
+<contactref element="C25" pad="1"/>
+<wire x1="61.595" y1="26.25" x2="1.69" y2="-27.94" width="0" layer="19" extent="1-1"/>
 </signal>
 <signal name="DIM3">
@@
 <via x="77.978" y="35.052" extent="1-16" drill="0.35"/>
 <wire x1="77.978" y1="38.862" x2="77.978" y2="35.052" width="0.5588" layer="16"/>
+<contactref element="C24" pad="1"/>
+<wire x1="78.105" y1="26.25" x2="1.69" y2="-22.86" width="0" layer="19" extent="1-1"/>
 </signal>
 <signal name="DIM4">
@@
 <signal name="VIN5">
 <contactref element="U5" pad="1"/>
-<contactref element="C13" pad="1"/>
 <contactref element="L5" pad="2"/>
 <polygon width="0.3048" layer="1" isolate="0.4064">
@@
 <via x="94.488" y="35.052" extent="1-16" drill="0.35"/>
 <wire x1="94.488" y1="35.052" x2="94.488" y2="38.608" width="0.5588" layer="16"/>
+<contactref element="C20" pad="1"/>
+<contactref element="C13" pad="1"/>
+<wire x1="94.615" y1="26.25" x2="1.69" y2="-17.78" width="0" layer="19" extent="1-1"/>
 </signal>
 <signal name="DIM5">
@@
 <via x="110.998" y="35.052" extent="1-16" drill="0.35"/>
 <wire x1="110.998" y1="35.052" x2="110.998" y2="38.608" width="0.5588" layer="16"/>
+<contactref element="C19" pad="1"/>
+<wire x1="111.125" y1="26.25" x2="1.69" y2="-12.7" width="0" layer="19" extent="1-1"/>
 </signal>
 <signal name="DIM6">

Commit message: progress on light controller v2.1
Parts:
- removed C22: 0.1uF, openag-capacitors:C0603
- removed C23: 10uF, openag-capacitors:C0805
- removed C35: 15uF, openag-capacitors:C0805
- removed D8: APT1608, openag-diodes:CHIPLED_0603
- removed F5: 7A, openag-fuses:SS
- removed F6: (no value), fuse:GSH15
- removed FRAME1: (no value), openag-frames:DOCFIELD
- removed J10, J9: PJ-036AH, openag-connectors:PJ-036AH
- removed R13: 3.01K, openag-resistors:RC0603N
- removed SJ1, SJ4, SJ6: (no value), openag-connectors:SOLDERJUMPER_REFLOW_NOPASTE
- removed TP12, TP13, TP14, TP15, TP16, TP17: TPTP06R, openag-testpads:TP06R
- removed U$5: (no value), openag-frames:OPENAG-LOGO-1000-MIL
- removed U12: LM2937, openag-regulators:MP04A
- added C37: 4.7uF, openag-capacitors:C0805
- added C41, C42: 10uF, openag-capacitors:C0805
- added C43: 0.1uF, openag-capacitors:C0603
- added D4: APT1608, openag-diodes:CHIPLED_0603
- added F1: 7A, openag-fuses:SS
- added J2, J3: PJ-036AH, openag-connectors:PJ-036AH
- added J4, J8: 54602-908LF, openag-connectors:RJ45-DI2C-USB-54602-908LF
- added R10, R12: 0 OHM, openag-resistors:RC0603N
- added R31, R34, R35, R42, R43, R44, R45: 600, openag-resistors:RC0603N
- added R36, R46, R47: 120, openag-resistors:RC0603N
- added R37, R38: 10K, openag-resistors:RC0603N
- added R39, R41: 100, openag-resistors:RC0603N
- added TP1, TP2, TP54, TP55, TP56: TPTP06R, openag-testpads:TP06R
- added TP40, TP41, TP42, TP43, TP44, TP45, TP46, TP47, TP48, TP49, TP5, TP50, TP51, TP52, TP53, TP57, TP58, TP59, TP6, TP60, TP61: TPTP04R, openag-testpads:TP04R
- added U$6: AUTHOR, openag-frames:AUTHOR
- added U$7: TITLE, openag-frames:TITLE
- added U$8: (no value), openag-frames:LOGO
- added U15: LM2937-3.3V, openag-regulators:MP04A
- added U17: R-78E5.0-1.0, openag-regulators:R-78E5.0-1.0
- added U18: PCA9615, openag-buffers:SOP50P490X110-10N
- C36: value 220uF -> 10uF; device openag-capacitors:CT7343 -> openag-capacitors:C0805
- C38: value 10uF -> 0.1uF; device openag-capacitors:C0805 -> openag-capacitors:C0603
- C39: value 4.7uF -> 10uF
- C40: value 0.1uF -> 10uF; device openag-capacitors:C0603 -> openag-capacitors:C0805
- D6: value SMAJ26A -> APT1608; device openag-diodes:SMA -> openag-diodes:CHIPLED_0603
- D7: value SBR2A40P1-7 -> SMAJ26A; device openag-diodes:POWERDI123 -> openag-diodes:SMA
- F2: value 400mA -> (none); device openag-fuses:0603 -> fuse:GSH15
- J7: device openag-connectors:OPENAG-I2C-HEADER -> openag-connectors:HEADER-I2C
- L8: value 68uH -> 33uH; device openag-inductors:UP2B -> openag-inductors:29333C
- R32: value 976 Ohm -> 120
- R33: value 100 -> 600
- R40: value 100 -> 1K
- R56, R57, R58, R59, R60, R61: value 10K -> 1K
- SJ10, SJ2, SJ3, SJ5, SJ7, SJ8, SJ9, SJ_A0, SJ_A1, SJ_A16, SJ_A17, SJ_A2, SJ_A3, SJ_A4, SJ_A5: device openag-connectors:SOLDERJUMPER_REFLOW_NOPASTE -> openag-connectors:SJ1
- TP3, TP4: value TPTP06R -> TPTP04R; device openag-testpads:TP06R -> openag-testpads:TP04R
- U$1, U$2, U$3, U$4: device openag-frames:OPENAG-CORNER-MOUNTING-HOLE -> openag-frames:CORNER
- U16: value MIC4680 -> PCA9615; device openag-regulators:SOIC8 -> openag-buffers:SOP50P490X110-10N
- moved U$3 123.2 mm to (5.08, 113.0), turned to 270 degrees
- moved U$4 123.2 mm to (127.0, 113.0), turned to 180 degrees
- moved C19 112.2 mm to (108.2, 25.1), turned to 270 degrees
- moved C20 98.9 mm to (91.7, 25.1), turned to 270 degrees
- moved C24 87.1 mm to (75.2, 25.1), turned to 270 degrees
- moved C25 77.3 mm to (58.7, 25.1), turned to 270 degrees
- moved C30 70.4 mm to (42.2, 25.1), turned to 270 degrees
- moved C34 67.3 mm to (25.7, 25.1), turned to 270 degrees
- moved U16 63.6 mm to (57.4, 95.4), turned to 180 degrees
- moved R32 62.4 mm to (52.3, 92.5), turned to 270 degrees
- moved R33 59.2 mm to (50.8, 92.5), turned to 90 degrees
- moved R11 56.0 mm to (116.8, 100.8), turned to 180 degrees
- moved R40 55.9 mm to (61.0, 98.0)
- moved TP4 54.8 mm to (56.4, 72.1), turned to 0 degrees
- moved D5 54.5 mm to (64.0, 98.0)
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Connections:
- removed net LIN_REG_VIN: C22.1, TP16.TP, U12.1
- removed net N$10: D1.A, R11.1
- removed net N$11: D7.-, L8.1, R13.1, R32.2, U16.3, U16.4
- removed net N$12: C23.1, F2.1, U12.3
- removed net N$22: D8.A, R33.1
- removed net N$24: C36.+, L8.2, R13.2, R33.2, SJ1.1
- removed net REG_3V3_400MA: F2.2, R11.2, SJ3.1
- removed net TAB: U12.4
- new net 24V_EMI: C40.1, L8.2, SJ3.2, U17.1
- new net DSCLM_1: J4.DSCLM(5), R35.2, R36.1, U16.6
- new net DSCLM_2: J8.DSCLM(5), R44.2, R46.1, U18.6
- new net DSCLP_1: J4.DSCLP(4), R34.1, R36.2, U16.7
- new net DSCLP_2: J8.DSCLP(4), R45.1, R46.2, U18.7
- new net DSDAM_1: J4.DSDAM(2), R31.1, R32.2, U16.9
- new net DSDAM_2: J8.DSDAM(2), R42.1, R47.2, U18.9
- new net DSDAP_1: J4.DSDAP(1), R32.1, R33.2, U16.8
- new net DSDAP_3: J8.DSDAP(1), R43.2, R47.1, U18.8
- new net N$1: D1.A, R39.1
- new net N$3: D6.A, R41.1
- new net N$4: D4.A, R11.1
- new net USBM: J4.USBM(8), J8.USBM(8), TP47.1
- new net USBP: J4.USBP(7), J8.USBP(7), TP46.1
- net +24V: now also C36.1, C37.1, C42.1, C43.1, D7.1, F1.2, F2.2, J4.24V(6), J8.24V(6), L8.1, R11.2, SJ3.1, TP2.TP, TP43.1, TP50.1, TP55.TP; no longer C35.1, C38.1, C39.1, C40.1, D6.1, F5.2, F6.2, TP14.TP, TP4.TP, U16.2
- net +3V3: now also C39.1, R37.2, R38.2, R41.2, TP40.1, TP48.1, TP57.1, TP60.1, U15.3, U16.1, U18.1; no longer SJ3.2, TP17.TP
- net +5V: now also C38.1, C41.1, R33.1, R34.2, R39.2, R43.1, R45.2, TP41.1, TP49.1, TP54.TP, TP58.1, U15.1, U16.10, U17.3, U18.10; no longer SJ1.2, TP12.TP
- net 24V_IN: now also F1.1, F2.1, J2.1, J3.1; no longer F5.1, F6.1, J10.1, J9.1
- net GND: now also C36.2, C37.2, C41.2, C42.2, C43.2, D4.C, D6.C, D7.2, J2.2, J2.3, J3.2, J3.3, R31.2, R35.1, R42.2, R44.1, TP1.TP, TP42.1, TP51.1, TP56.TP, TP59.1, TP61.1, U15.2, U15.4, U17.2, U18.5; no longer C22.2, C23.2, C35.2, C36.-, D6.2, D7.+, D8.C, J10.2, J10.3, J9.2, J9.3, R32.1, TP13.TP, TP15.TP, TP3.TP, U12.2, U16.1, U16.6, U16.7, U16.8
- net SCL: now also R10.2, R38.1, TP3.1, TP45.1, TP52.1, U16.4, U18.4; no longer SJ4.2
- net SCL_IN: now also R10.1, TP5.1; no longer SJ4.1
- net SDA: now also R12.2, R37.1, TP4.1, TP44.1, TP53.1, U16.2, U18.2; no longer SJ6.2
- net SDA_IN: now also R12.1, TP6.1; no longer SJ6.1
Routing:
- net +5V: track 6.89 -> 131.7 mm, vias 2 -> 6
- net +24V: track 40.1 -> 99.3 mm, vias 6 -> 9
- net USBM: track 0.00 -> 40.0 mm
- net SCL_IN: track 44.7 -> 5.51 mm, vias 2 -> 0
- net USBP: track 0.00 -> 38.8 mm, vias 0 -> 1
- net SDA_IN: track 42.5 -> 5.72 mm, vias 2 -> 0
- net UART_DE: track 48.9 -> 27.0 mm
- net UART_!RE!: track 49.3 -> 28.3 mm
- net UART_RX: track 29.2 -> 8.44 mm
- net UART_TX: track 30.4 -> 9.71 mm, vias 2 -> 0
- net DSDAP_3: track 0.00 -> 16.9 mm
- net DSDAP_1: track 0.00 -> 16.7 mm
- net 24V_EMI: track 0.00 -> 16.4 mm
- net N$11: track 16.2 -> 0.00 mm, vias 2 -> 0
- net DSDAM_2: track 0.00 -> 14.7 mm
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- removed copper zone on layer 1, net LIN_REG_VIN
- removed copper zone on layer 1, net N$11
- removed copper zone on layer 16, net N$11
- removed copper zone on layer 1, net N$24
- removed copper zone on layer 16, net N$24
Other:
- board size 132.1 x 116.8 mm -> 132.1 x 118.1 mm
- board text added: "24V to 5V@1A Switching Regulator w/Optional EMI Filter + Indicator LED"
- board text added: "5V to 3.3V@400mA Linear Regulator w/ LED"
- board text added: "Barrel Jack Connector Pair w/24V Conditioning + Fuse + LED"
- board text added: "EMI Bypass"
- board text added: "PSOC4100 Microcontroller w/I2C or RS485 Comm"
- board text added: "RJ45 Connector Pair w/dI2C Buffer + Indicator LED"
- board text added: "SCL-IN"
- board text added: "SDA-IN"
- board text added: "USBM"
- board text added: "USBP"
- board text removed: "24V-to-5V@1A Switching Regulator w/Indicator LED + Enable"
- board text removed: "5-26V to 3.3V@400mA Regulator w/3v3 Enable, Indicator LED & Fuse"
- board text removed: "Barrel Jack Connector Pair w/24V Conditioning + Fuse + Indicator LED"
- board text removed: "Enable"
- board text removed: "Fuse"
- board text removed: "Light Controller v2.1"
- board text removed: "PSOC4100 Microcontroller w/I2C or RS485 Communication"
- board text removed: "VIN"

Commit message: light controller v2.1 90% done
Parts:
- removed C32: 1uF, openag-capacitors:C0603
- removed R26: 1K, openag-resistors:RC0603N
- removed R62: 10K, openag-resistors:RC0603N
- removed SJ3: (no value), openag-connectors:SJ1
- removed U14: PCA9685, openag-pwm:TSSOP28
- removed U16, U18: PCA9615, openag-buffers:SOP50P490X110-10N
- added C23: 1uF, openag-capacitors:C0603
- added R13, R15: 1K, openag-resistors:RC0603N
- added SJ1: (no value), openag-connectors:EMI-BYPASS
- added TP10, TP12, TP13, TP14, TP15, TP16, TP17, TP32, TP33, TP34, TP7: TPTP04R, openag-testpads:TP04R
- added U11, U12: PCA9615, openag-buffers:SOP50P490X110-10N
- added U8: CY8C4124PVI-432, openag-microcontrollers:SSOP-28
- F2: value (none) -> GSH15; device fuse:GSH15 -> openag-fuses:GSH15
- J1: device openag-connectors:22-23-2051 -> openag-connectors:PSOC-PROGRAMMER-22-23-2051
- J2, J3: device openag-connectors:PJ-036AH -> openag-connectors:BARREL-JACK-PJ-036AH
- J5, J6: value OPENAG-RS485-RJ12 -> A-2004-1-4-LP-N-R; device openag-connectors:OPENAG-RS485-RJ12 -> openag-connectors:RJ12-RS485--A-2004-1-4-LP-N-R
- SJ10, SJ2, SJ5, SJ7, SJ8, SJ9: device openag-connectors:SJ1 -> openag-connectors:EMI-BYPASS
- U10: value ADM2481BRWZ-RL7 -> PCA9685; device openag-isolators:SOIC16LWB -> openag-pwm:TSSOP28
- U9: value CY8C4124PVI-432 -> ADM2481; device openag-microcontrollers:SSOP-28 -> openag-isolators:SOIC16LWB
- moved U10 44.7 mm to (54.1, 54.4)
- moved TP27 23.2 mm to (43.7, 107.4)
- moved U9 22.3 mm to (35.1, 95.5), turned to 0 degrees
- moved J7 8.89 mm to (72.4, 76.2), turned to 180 degrees
- moved R12 3.78 mm to (54.9, 74.9)
- moved TP4 3.78 mm to (58.9, 74.9)
- moved TP6 3.78 mm to (52.8, 74.9)
- moved R10 3.42 mm to (54.9, 76.2)
- moved TP3 3.42 mm to (58.9, 76.2)
- moved TP5 3.42 mm to (52.8, 76.2)
- moved C26 2.69 mm to (25.9, 99.3)
- moved R14 2.54 mm to (86.6, 54.6), turned to 90 degrees
- moved TP28 2.29 mm to (37.1, 87.1)
- moved TP29 2.29 mm to (34.8, 87.1)
- moved TP30 2.29 mm to (35.6, 87.1)
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- renumbered C33 to C22, U15 to U13
Connections:
- net !LDAC!: now also TP17.1, TP8.1, U8.24; no longer TP23.1, U9.24
- net +24V: now also SJ1.1, TP12.1; no longer SJ3.1
- net +3V3: now also C23.1, R13.2, R14.2, R6.2, R7.2, R8.2, R9.2, TP13.1, U10.28, U11.1, U12.1, U8.27, U9.1; no longer C32.1, R14.1, R26.1, R6.1, R7.1, R8.1, R9.1, U10.1, U14.28, U16.1, U18.1, U9.27
- net +5V: now also U11.10, U12.10; no longer U16.10, U18.10
- net 24V_EMI: now also SJ1.2; no longer SJ3.2
- net 485_5V: now also U9.16; no longer U10.16
- net 485_A: now also U9.12; no longer U10.12
- net 485_B: now also U9.13; no longer U10.13
- net 485_GND: now also U9.10, U9.15, U9.9; no longer J5.1, J6.1, U10.10, U10.15, U10.9
- net A0: now also U10.1; no longer U14.1
- net A1: now also U10.2; no longer U14.2
- net A2: now also U10.3; no longer U14.3
- net A3: now also U10.4; no longer U14.4
- net A4: now also U10.5; no longer U14.5
- net A5: now also U10.24; no longer U14.24
- net DAC_!CLR!: now also TP23.1, TP32.1, U8.23; no longer TP8.1, U9.23
- net DIM1: now also R6.1; no longer R6.2
- net DIM2: now also R7.1; no longer R7.2
- net DIM3: now also R8.1; no longer R8.2
- net DIM4: now also R9.1; no longer R9.2
- net DIM5: now also R13.1; no longer R14.2
- net DIM6: now also R14.1; no longer R26.2
- net DSCLM_1: now also U11.6; no longer U16.6
- net DSCLM_2: now also U12.6; no longer U18.6
- net DSCLP_1: now also U11.7; no longer U16.7
- net DSCLP_2: now also U12.7; no longer U18.7
- net DSDAM_1: now also U11.9; no longer U16.9
- net DSDAM_2: now also U12.9; no longer U18.9
- net DSDAP_1: now also U11.8; no longer U16.8
- net DSDAP_3: now also U12.8; no longer U18.8
- net GND: now also C23.2, J4.GND(3), J8.GND(3), R15.2, TP10.1, TP14.1, TP33.1, TP34.1, TP7.1, U10.14, U10.25, U11.5, U12.5, U8.28, U9.2, U9.7, U9.8; no longer C32.2, R62.2, U10.2, U10.7, U10.8, U14.14, U14.25, U16.5, U18.5, U9.28
- net N$23: now also U8.26; no longer U9.26
- net OE: now also R15.1, U10.23; no longer R62.1, U14.23
- net PWM1: now also U10.12; no longer U14.12
- net PWM2: now also U10.11; no longer U14.11
- net PWM3: now also U10.10; no longer U14.10
- net PWM4: now also U10.9; no longer U14.9
- net PWM5: now also U10.8; no longer U14.8
- net PWM6: now also U10.7; no longer U14.7
- net SCB1_RX[0]_SCL[0]: now also U8.11; no longer U9.11
- net SCB1_TX[0]_SDA[0]: now also U8.12; no longer U9.12
- net SCL: now also TP16.1, U10.26, U8.15; no longer R38.1, TP45.1, TP52.1, U14.26, U16.4, U18.4, U9.15
- net SCL_IN: now also R38.1, TP45.1, TP52.1, U11.4, U12.4
- net SDA: now also TP15.1, U10.27, U8.16; no longer R37.1, TP44.1, TP53.1, U14.27, U16.2, U18.2, U9.16
- net SDA_IN: now also R37.1, TP44.1, TP53.1, U11.2, U12.2
- net SWD_CLK[0]: now also U8.14; no longer U9.14
- net SWD_IO[0]: now also U8.13; no longer U9.13
- net UART_!RE!: now also U8.10, U9.4; no longer U10.4, U9.10
- net UART_DE: now also U8.9, U9.5; no longer U10.5, U9.9
- net UART_RX: now also U9.3; no longer U10.3
- net UART_TX: now also U9.6; no longer U10.6
- net XRES: now also U8.25; no longer U9.25
Routing:
- net +3V3: track 240.6 -> 353.5 mm, vias 10 -> 14
- net SCL_IN: track 5.51 -> 76.9 mm, vias 0 -> 2
- net SDA_IN: track 5.72 -> 72.2 mm, vias 0 -> 2
- net +24V: track 99.3 -> 134.5 mm, vias 9 -> 12
- net UART_DE: track 27.0 -> 48.5 mm
- net UART_!RE!: track 28.3 -> 49.0 mm
- net UART_RX: track 8.44 -> 27.9 mm
- net UART_TX: track 9.71 -> 28.2 mm, vias 0 -> 2
- net 485_GND: track 55.8 -> 38.8 mm
- net N$23: track 16.6 -> 5.64 mm
- net 485_B: track 32.6 -> 22.8 mm
- net DAC_!CLR!: track 74.1 -> 80.8 mm
- net !LDAC!: track 67.1 -> 73.0 mm
- net SDA: track 117.0 -> 121.8 mm, vias 0 -> 3
- net GND: track 10.9 -> 15.0 mm, vias 96 -> 99
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- removed copper zone on layer 1, net !LDAC!
- removed copper zone on layer 1, net DAC_!CLR!
- removed copper zone on layer 1, net SCL
- removed copper zone on layer 1, net SDA
Other:
- board text added: "6-Channel 24V@700mA (per channel) Current Regulator Module w/I2C Controlled Dimming via PWM or Analog Signaling"
- board text added: "Description goes here."
- board text added: "Something goes here"
- board text removed: "6-Channel 24V, 700mA (per channel) Current Regulator Module w/I2C Controlled Dimming via PWM or Analog Signaling"
- board text removed: "EMI Bypass"

Commit message: added light controller v2.1
Parts:
- removed F1: 7A, openag-fuses:SS
- removed F2: GSH15, openag-fuses:GSH15
- removed J3: PJ-036AH, openag-connectors:BARREL-JACK-PJ-036AH
- added F3: GSH15, openag-fuses:GSH15
- added TP35, TP36: TPTP04R, openag-testpads:TP04R
- added U$9: (no value), openag-frames:CAMBRIDGE-MAP-LIGHT-CONTROLLER-V-2-1
- TP1, TP2: value TPTP06R -> TPTP04R; device openag-testpads:TP06R -> openag-testpads:TP04R
- moved D4 26.7 mm to (95.0, 90.9), turned to 0 degrees
- moved TP1 26.4 mm to (116.1, 88.4), turned to 0 degrees
- moved R11 21.5 mm to (98.3, 90.9), turned to 90 degrees
- moved C37 15.9 mm to (102.1, 91.2), turned to 270 degrees
- moved J2 12.7 mm to (106.7, 107.0)
- moved C36 11.1 mm to (106.4, 91.2), turned to 270 degrees
- moved C43 10.7 mm to (110.2, 91.2), turned to 270 degrees
- moved TP2 5.85 mm to (103.4, 88.4), turned to 0 degrees
- moved D5 3.84 mm to (67.8, 98.6)
- moved J8 3.84 mm to (76.2, 109.8)
- moved R31 3.84 mm to (59.2, 92.3)
- moved R32 3.84 mm to (56.1, 93.0)
- moved R33 3.84 mm to (54.6, 93.0)
- moved R34 3.84 mm to (54.6, 96.1)
- moved R35 3.84 mm to (55.4, 98.3)
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Connections:
- net +24V: now also F3.2, TP1.1, TP36.1; no longer F1.2, F2.2, TP2.TP
- net 24V_IN: now also F3.1; no longer F1.1, F2.1, J3.1
- net GND: now also TP2.1, TP35.1; no longer J3.2, J3.3, TP1.TP
Routing:
- net +24V: track 134.5 -> 113.6 mm, vias 12 -> 13
- net +3V3: track 353.5 -> 347.1 mm
- net +5V: track 132.6 -> 137.4 mm
- net SDA_IN: track 72.2 -> 76.1 mm
- net SCL_IN: track 76.9 -> 80.8 mm
- net N$4: track 2.04 -> 3.31 mm
- net GND: track 15.0 -> 16.0 mm, vias 99 -> 153
Other:
- board size 132.1 x 118.1 mm -> 132.1 x 119.4 mm
- board text added: "Barrel Jack Connector w/24V Conditioning + Fuse + LED"
- board text added: "Changelog - replaced 24v-to-5v regulator with R78E5 - added dual i2c buffers - updated to style conventions v1.0"
- board text added: "Drives x6 channels of LEDs by regulating the current up to 700mA (per channel) at 24V. Communicates via differential-I2C (dI2C) or RS485 (See enables on PSOC module). To communicate directly with the board ICs and avoid programming the PSOC, enable I2C Connect. Current regulators can be driven by either dimming or PWM control. Allows for daisy chaining comms between multiple boards."
- board text added: "Use 5A Fuse"
- board text removed: "Barrel Jack Connector Pair w/24V Conditioning + Fuse + LED"
- board text removed: "Description goes here."
- board text removed: "Something goes here"
