File: proj/light-controller/v2.1/light_controller.brd (EAGLE design)
At the start: 132.1 x 119.4 mm, 207 parts, among them J1 0022232051, J2 PJ-036AH, J4 54602-908LF, J5 A-2004-1-4-LP-N-R, J6 A-2004-1-4-LP-N-R, J7 I2C-HEADER, J8 54602-908LF, U1 RCD-24-0.70/VREF, U10 PCA9685, U11 PCA9615, U12 PCA9615, U13 LM2937-3.3V, U17 R-78E5.0-1.0, U2 RCD-24-0.70/VREF, U3 RCD-24-0.70/VREF, U4 RCD-24-0.70/VREF, U5 RCD-24-0.70/VREF, U6 RCD-24-0.70/VREF, U7 DAC5578, U8 CY8C4124PVI-432, U9 ADM2481

Commit message: added photon quad v1.0 at 90%
Changed lines of the file:
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@@
 <attribute name="MPN" value="R-78E5.0-1.0" x="106.68" y="76.2" size="0.762" layer="27" rot="R90" display="off"/>
 <attribute name="NAME" x="100.076" y="70.485" size="0.762" layer="25" rot="R90"/>
+<attribute name="VALUE" x="103.124" y="73.66" size="0.762" layer="27" rot="R90"/>
 <attribute name="VALUE" x="103.124" y="73.66" size="0.762" layer="21" rot="R90"/>
-<attribute name="VALUE" x="103.124" y="73.66" size="0.762" layer="27" rot="R90"/>
 <attribute name="VENDOR" value="Digikey" x="106.68" y="76.2" size="0.762" layer="27" rot="R90" display="off"/>
 <attribute name="VLINK" value="https://www.digikey.com/product-detail/en/recom-power/R-78E5.0-1.0/945-2201-ND/4930585" x="106.68" y="76.2" size="0.762" layer="27" rot="R90" display="off"/>
@@
 <attribute name="MPN" value="A-2004-1-4-LP-N-R" x="35.052" y="112.3188" size="0.762" layer="27" rot="R90" display="off"/>
 <attribute name="NAME" x="41.148" y="100.5078" size="0.762" layer="25"/>
+<attribute name="VALUE" x="40.132" y="115.2398" size="0.762" layer="21" rot="R180"/>
 <attribute name="VALUE" x="40.132" y="115.2398" size="0.762" layer="27" rot="R180"/>
-<attribute name="VALUE" x="40.132" y="115.2398" size="0.762" layer="21" rot="R180"/>
 <attribute name="VENDOR" value="Digikey" x="35.052" y="112.3188" size="0.762" layer="27" rot="R90" display="off"/>
 <attribute name="VLINK" value="https://www.digikey.com/product-detail/en/assmann-wsw-components/A-2004-1-4-LP-N-R/AE10383-ND/2183634" x="35.052" y="112.3188" size="0.762" layer="27" rot="R90" display="off"/>
@@
 <attribute name="MPN" value="A-2004-1-4-LP-N-R" x="16.764" y="112.3188" size="0.762" layer="27" rot="R90" display="off"/>
 <attribute name="NAME" x="12.7" y="100.5078" size="0.762" layer="25"/>
+<attribute name="VALUE" x="24.892" y="115.2398" size="0.762" layer="21" rot="R180"/>
 <attribute name="VALUE" x="24.892" y="115.2398" size="0.762" layer="27" rot="R180"/>
-<attribute name="VALUE" x="24.892" y="115.2398" size="0.762" layer="21" rot="R180"/>
 <attribute name="VENDOR" value="Digikey" x="16.764" y="112.3188" size="0.762" layer="27" rot="R90" display="off"/>
 <attribute name="VLINK" value="https://www.digikey.com/product-detail/en/assmann-wsw-components/A-2004-1-4-LP-N-R/AE10383-ND/2183634" x="16.764" y="112.3188" size="0.762" layer="27" rot="R90" display="off"/>
@@
 <attribute name="MPN" value="54602-908LF" x="59.69" y="109.7788" size="0.762" layer="27" rot="R180" display="off"/>
 <attribute name="NAME" x="52.07" y="98.6663" size="0.762" layer="25"/>
+<attribute name="VALUE" x="63.373" y="112.8268" size="0.762" layer="21" rot="R180"/>
 <attribute name="VALUE" x="63.373" y="112.8268" size="0.762" layer="27" rot="R180"/>
-<attribute name="VALUE" x="63.373" y="112.8268" size="0.762" layer="21" rot="R180"/>
 <attribute name="VENDOR" value="Digikey" x="59.69" y="109.7788" size="0.762" layer="27" rot="R180" display="off"/>
 <attribute name="VLINK" value="https://www.digikey.com/product-detail/en/amphenol-fci/54602-908LF/609-1046-ND/1001360" x="59.69" y="109.7788" size="0.762" layer="27" rot="R180" display="off"/>
@@
 <attribute name="MPN" value="54602-908LF" x="76.2" y="109.7788" size="0.762" layer="27" rot="R180" display="off"/>
 <attribute name="NAME" x="83.82" y="99.3013" size="0.762" layer="25" rot="R180"/>
+<attribute name="VALUE" x="79.883" y="112.8268" size="0.762" layer="21" rot="R180"/>
 <attribute name="VALUE" x="79.883" y="112.8268" size="0.762" layer="27" rot="R180"/>
-<attribute name="VALUE" x="79.883" y="112.8268" size="0.762" layer="21" rot="R180"/>
 <attribute name="VENDOR" value="Digikey" x="76.2" y="109.7788" size="0.762" layer="27" rot="R180" display="off"/>
 <attribute name="VLINK" value="https://www.digikey.com/product-detail/en/amphenol-fci/54602-908LF/609-1046-ND/1001360" x="76.2" y="109.7788" size="0.762" layer="27" rot="R180" display="off"/>
@@
 <attribute name="MPN" value="64900001039" x="106.68" y="97.79" size="0.762" layer="27" display="off"/>
 <attribute name="NAME" x="94.1324" y="91.9988" size="0.762" layer="25" ratio="10"/>
+<attribute name="VALUE" x="105.0544" y="101.219" size="0.762" layer="27" ratio="10"/>
 <attribute name="VALUE" x="105.0544" y="101.219" size="0.762" layer="21" ratio="10"/>
-<attribute name="VALUE" x="105.0544" y="101.219" size="0.762" layer="27" ratio="10"/>
 <attribute name="VENDOR" value="Digikey" x="106.68" y="97.79" size="0.762" layer="27" display="off"/>
 <attribute name="VLINK" value="https://www.digikey.com/product-detail/en/littelfuse-inc/64900001039/WK0011-ND/245470" x="106.68" y="97.79" size="0.762" layer="27" display="off"/>
