File: proj/plc/v1.0/plc-accessory.brd (EAGLE design)
At the start: 132.1 x 116.8 mm, 163 parts, among them J1 0022232051, J10 PJ-036AH, J4 54602-908LF, J5 OPENAG-RS485-RJ12, J6 OPENAG-RS485-RJ12, J7 OPENAG-I2C-HEADER, J8 54602-908LF, J9 PJ-036AH, U1 RCD-24-0.70/VREF, U10 ADM2481BRWZ-RL7, U12 LM2937IMP3.3NOPB, U14 PCA9685, U15 PCA9615DPJ, U16 MIC4680YM-TR, U2 RCD-24-0.70/VREF, U3 RCD-24-0.70/VREF, U4 RCD-24-0.70/VREF, U5 RCD-24-0.70/VREF, U6 RCD-24-0.70/VREF, U7 DAC5578SPW, U9 CY8C4124PVI-432

Commit message: plc
Parts:
- removed C1, C10, C11, C13, C14, C16, C17, C2, C4, C5, C7, C8: 10nF, openag-capacitors:C0603
- removed C12, C15, C18, C3, C6, C9: 100uF, openag-capacitors:EEE-1HA101UP
- removed C21: 10uF, openag-capacitors:C0805
- removed C26, C27, C28, C31: 0.1uF, openag-capacitors:C0603
- removed C29: 4.7uF, openag-capacitors:C0805
- removed C32, C33: 1uF, openag-capacitors:C0603
- removed CH1+, CH1-, CH2+, CH2-, CH3+, CH3-, CH4+, CH4-, CH5+, CH5-, CH6+, CH6-: (no value), openag-wirepads:3,17/1,3
- removed J1: 0022232051, openag-connectors:22-23-2051
- removed J5, J6: OPENAG-RS485-RJ12, openag-connectors:OPENAG-RS485-RJ12
- removed L1, L2, L3, L4, L5, L6: 120uH, openag-inductors:74404064121
- removed R1, R14, R26, R28, R6, R7, R8, R9: 1K, openag-resistors:RC0603N
- removed R2, R29, R3, R4, R5: 0 OHM, openag-resistors:RC0603N
- removed R56, R57, R58, R59, R60, R61, R62: 10K, openag-resistors:RC0603N
- removed SJ_A0, SJ_A1, SJ_A16, SJ_A17, SJ_A2, SJ_A3, SJ_A4, SJ_A5: (no value), openag-connectors:SOLDERJUMPER_REFLOW_NOPASTE
- removed TP11, TP18, TP19, TP20, TP21, TP22, TP23, TP24, TP25, TP26, TP27, TP28, TP29, TP30, TP31, TP8, TP9: TPTP04R, openag-testpads:TP04R
- removed U1, U2, U3, U4, U5, U6: RCD-24-0.70/VREF, openag-regulators:RCD-24-PINNED
- removed U10: ADM2481BRWZ-RL7, openag-isolators:SOIC16LWB
- removed U14: PCA9685, openag-pwm:TSSOP28
- removed U7: DAC5578SPW, openag-dacs:TSSOP16
- removed U9: CY8C4124PVI-432, openag-microcontrollers:SSOP-28
- moved FRAME1 92.7 mm to (178.8, 50.2)
Connections:
- removed net !LDAC!: R1.2, R29.2, TP23.1, U7.1, U9.24
- removed net 485_5V: C26.1, J5.2, J6.2, U10.16
- removed net 485_A: J5.3, J6.3, U10.12
- removed net 485_B: J5.4, J6.4, U10.13
- removed net 485_GND: C26.2, J5.1, J5.6, J6.1, J6.6, U10.10, U10.15, U10.9
- removed net A0: R61.2, SJ_A0.2, U14.1
- removed net A1: R60.2, SJ_A1.2, U14.2
- removed net A2: R59.2, SJ_A2.2, U14.3
- removed net A3: R58.2, SJ_A3.2, U14.4
- removed net A4: R57.2, SJ_A4.2, U14.5
- removed net A5: R56.2, SJ_A5.2, U14.24
- removed net ADDR0: SJ_A16.2, SJ_A17.2, U7.2
- removed net CH1+: CH1+.1, U1.6
- removed net CH1-: C2.1, CH1-.1, U1.5
- removed net CH2+: CH2+.1, U2.6
- removed net CH2-: C5.1, CH2-.1, U2.5
- removed net CH3+: CH3+.1, U3.6
- removed net CH3-: C8.1, CH3-.1, U3.5
- removed net CH4+: CH4+.1, U4.6
- removed net CH4-: C11.1, CH4-.1, U4.5
- removed net CH5+: CH5+.1, U5.6
- removed net CH5-: C14.1, CH5-.1, U5.5
- removed net CH6+: CH6+.1, U6.6
- removed net CH6-: C17.1, CH6-.1, U6.5
- removed net DAC_!CLR!: R28.2, TP8.1, U7.9, U9.23
- removed net DIM1: R6.2, U1.2, U7.7
- removed net DIM2: R7.2, U2.2, U7.6
- removed net DIM3: R8.2, U3.2, U7.5
- removed net DIM4: R9.2, U4.2, U7.4
- removed net DIM5: R14.2, U5.2, U7.10
- removed net DIM6: R26.2, U6.2, U7.11
- removed net N$1: C1.1, L1.2, U1.1
- removed net N$2: C4.1, L2.2, U2.1
- removed net N$23: C33.1, U9.26
- removed net N$4: C7.1, L3.2, U3.1
- removed net N$5: C10.1, L4.2, U4.1
- removed net N$6: C13.1, L5.2, U5.1
- removed net N$7: C16.1, L6.2, U6.1
- removed net OE: R62.1, U14.23
- removed net PWM1: U1.3, U14.12
- removed net PWM2: U14.11, U2.3
- removed net PWM3: U14.10, U3.3
- removed net PWM4: U14.9, U4.3
- removed net PWM5: U14.8, U5.3
- removed net PWM6: U14.7, U6.3
- removed net SCB1_RX[0]_SCL[0]: R2.1, R3.1, U9.11
- removed net SCB1_TX[0]_SDA[0]: R4.1, R5.1, U9.12
- removed net SWD_CLK[0]: J1.2, U9.14
- removed net SWD_IO[0]: J1.1, U9.13
- removed net UART_!RE!: TP21.1, TP30.1, U10.4, U9.10
- removed net UART_DE: TP22.1, TP31.1, U10.5, U9.9
- removed net UART_RX: R3.2, TP20.1, TP29.1, U10.3
- removed net UART_TX: R5.2, TP11.1, TP28.1, U10.6
- removed net XRES: J1.3, U9.25
- net +24V: no longer C12.+, C15.+, C18.+, C3.+, C6.+, C9.+, L1.1, L2.1, L3.1, L4.1, L5.1, L6.1
- net +3V3: no longer C21.1, C27.1, C28.1, C29.1, C31.1, C32.1, J1.5, R1.1, R14.1, R26.1, R28.1, R6.1, R7.1, R8.1, R9.1, SJ_A0.1, SJ_A1.1, SJ_A16.1, SJ_A2.1, SJ_A3.1, SJ_A4.1, SJ_A5.1, TP19.1, TP27.1, U10.1, U14.28, U7.3, U7.8, U9.27
- net GND: no longer C1.2, C10.2, C11.2, C12.-, C13.2, C14.2, C15.-, C16.2, C17.2, C18.-, C2.2, C21.2, C27.2, C28.2, C29.2, C3.-, C31.2, C32.2, C33.2, C4.2, C5.2, C6.-, C7.2, C8.2, C9.-, J1.4, R29.1, R56.1, R57.1, R58.1, R59.1, R60.1, R61.1, R62.2, SJ_A17.1, TP9.1, U1.4, U10.2, U10.7, U10.8, U14.14, U14.25, U2.4, U3.4, U4.4, U5.4, U6.4, U7.14, U9.28
- net SCL: no longer TP24.1, U14.26, U7.16, U9.15
- net SCL_IN: no longer R2.2, TP26.1
- net SDA: no longer TP18.1, U14.27, U7.15, U9.16
- net SDA_IN: no longer R4.2, TP25.1
Routing:
- net DIM1: track 175.5 -> 0.00 mm, vias 1 -> 0
- net PWM6: track 166.3 -> 0.00 mm
- net DIM2: track 156.6 -> 0.00 mm, vias 1 -> 0
- net PWM5: track 148.3 -> 0.00 mm
- net DIM3: track 137.9 -> 0.00 mm, vias 1 -> 0
- net PWM4: track 130.2 -> 0.00 mm
- net DIM4: track 118.9 -> 0.00 mm, vias 1 -> 0
- net PWM3: track 112.2 -> 0.00 mm
- net +3V3: track 267.0 -> 163.4 mm, vias 10 -> 8
- net PWM2: track 94.1 -> 0.00 mm
- net DIM5: track 91.5 -> 0.00 mm, vias 1 -> 0
- net DAC_!CLR!: track 82.2 -> 0.00 mm, vias 2 -> 0
- net PWM1: track 79.8 -> 0.00 mm
- net DIM6: track 75.9 -> 0.00 mm, vias 1 -> 0
- net !LDAC!: track 76.3 -> 0.51 mm, vias 5 -> 0
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