File: proj/plc/v1.0/plc-accessory.sch (EAGLE design)
At the start: 158 parts, among them J1 0022232051, J10 PJ-036AH, J4 54602-908LF, J5 OPENAG-RS485-RJ12, J6 OPENAG-RS485-RJ12, J7 OPENAG-I2C-HEADER, J8 54602-908LF, J9 PJ-036AH, U1 RCD-24-0.70/VREF, U10 ADM2481BRWZ-RL7, U12 LM2937IMP3.3NOPB, U14 PCA9685, U15 PCA9615DPJ, U16 MIC4680YM-TR, U2 RCD-24-0.70/VREF, U3 RCD-24-0.70/VREF, U4 RCD-24-0.70/VREF, U5 RCD-24-0.70/VREF, U6 RCD-24-0.70/VREF, U7 DAC5578SPW, U9 CY8C4124PVI-432

Commit message: plc
Parts:
- removed C1, C10, C11, C13, C14, C16, C17, C2, C4, C5, C7, C8: 10nF, openag-capacitors:10NF-C0603C103K5RACTU
- removed C12, C15, C18, C3, C6, C9: 100uF, openag-capacitors:100UF-EEE-1HA101UP
- removed C21: 10uF, openag-capacitors:10UF-GMK212BBJ106KG-T
- removed C26, C27, C28, C31: 0.1uF, openag-capacitors:0.1UF-C0603C104K5RACTU
- removed C29: 4.7uF, openag-capacitors:4.7UF-CL21A475KBQNNNE
- removed C32, C33: 1uF, openag-capacitors:1UF-CL10A105KB8NNNC
- removed CH1+, CH1-, CH2+, CH2-, CH3+, CH3-, CH4+, CH4-, CH5+, CH5-, CH6+, CH6-: (no value), openag-wirepads:3,17/1,3
- removed J1: 0022232051, openag-connectors:MINI-PROG3-5POS-MATING-CONNECTOR
- removed J5, J6: OPENAG-RS485-RJ12, openag-connectors:OPENAG-RS485-RJ12
- removed L1, L2, L3, L4, L5, L6: 120uH, openag-inductors:120UH-ASPI-6045S-121M-TCT-ND
- removed R1, R14, R26, R28, R6, R7, R8, R9: 1K, openag-resistors:1K-ERJ-PB3D1001V
- removed R2, R29, R3, R4, R5: 0 OHM, openag-resistors:0OHM-RC0603JR-070RL
- removed R56, R57, R58, R59, R60, R61, R62: 10K, openag-resistors:10K-ERJ-3EKF1002V
- removed SJ_A0, SJ_A1, SJ_A16, SJ_A17, SJ_A2, SJ_A3, SJ_A4, SJ_A5: (no value), openag-connectors:SOLDERJUMPERREFLOW_NOPASTE
- removed TP11, TP18, TP19, TP20, TP21, TP22, TP23, TP24, TP25, TP26, TP27, TP28, TP29, TP30, TP31, TP8, TP9: TPTP04R, openag-testpads:TPTP04R
- removed U1, U2, U3, U4, U5, U6: RCD-24-0.70/VREF, openag-regulators:RCD-24-0.70/VREF
- removed U10: ADM2481BRWZ-RL7, openag-isolators:ADM2481BRWZ-RL7
- removed U14: PCA9685, openag-pwm:PCA9685PW/Q900,118
- removed U7: DAC5578SPW, openag-dacs:DAC5578SPW
- removed U9: CY8C4124PVI-432, openag-microcontrollers:CY8C4124PVI-432
- FRAME1: AUTHOR JR -> DP; DESCRIPTION Controls 6 channels of 24V, 700mA for LED strings that can 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 -> PLC; TITLE Light Controller -> PLC; VER 2.0 -> (none)
Connections:
- removed net !LDAC!: R1.2, R29.2, TP23.TP, U7.!LDAC!, U9.P0[7]
- removed net 485_5V: C26.1, J5.2, J6.2, U10.VDD2
- removed net 485_A: J5.3, J6.3, U10.A
- removed net 485_B: J5.4, J6.4, U10.B
- removed net 485_GND: C26.2, J5.1, J5.6, J6.1, J6.6, U10.GND2
- removed net A0: R61.2, SJ_A0.2, U14.A0
- removed net A1: R60.2, SJ_A1.2, U14.A1
- removed net A2: R59.2, SJ_A2.2, U14.A2
- removed net A3: R58.2, SJ_A3.2, U14.A3
- removed net A4: R57.2, SJ_A4.2, U14.A4
- removed net A5: R56.2, SJ_A5.2, U14.A5
- removed net ADDR0: SJ_A16.2, SJ_A17.2, U7.ADDR0
- removed net CH1+: CH1+.P, U1.+VOUT
- removed net CH1-: C2.1, CH1-.P, U1.-VOUT
- removed net CH2+: CH2+.P, U2.+VOUT
- removed net CH2-: C5.1, CH2-.P, U2.-VOUT
- removed net CH3+: CH3+.P, U3.+VOUT
- removed net CH3-: C8.1, CH3-.P, U3.-VOUT
- removed net CH4+: CH4+.P, U4.+VOUT
- removed net CH4-: C11.1, CH4-.P, U4.-VOUT
- removed net CH5+: CH5+.P, U5.+VOUT
- removed net CH5-: C14.1, CH5-.P, U5.-VOUT
- removed net CH6+: CH6+.P, U6.+VOUT
- removed net CH6-: C17.1, CH6-.P, U6.-VOUT
- removed net DAC_!CLR!: R28.2, TP8.TP, U7.!CLR!, U9.P0[6]
- removed net DIM1: R6.2, U1.ANALOGUE_DIM, U7.VOUT_G
- removed net DIM2: R7.2, U2.ANALOGUE_DIM, U7.VOUT_E
- removed net DIM3: R8.2, U3.ANALOGUE_DIM, U7.VOUT_C
- removed net DIM4: R9.2, U4.ANALOGUE_DIM, U7.VOUT_A
- removed net DIM5: R14.2, U5.ANALOGUE_DIM, U7.VOUT_H
- removed net DIM6: R26.2, U6.ANALOGUE_DIM, U7.VOUT_F
- removed net N$1: C1.1, L1.2, U1.+VIN
- removed net N$2: C4.1, L2.2, U2.+VIN
- removed net N$23: C33.1, U9.VCCD
- removed net N$4: C7.1, L3.2, U3.+VIN
- removed net N$5: C10.1, L4.2, U4.+VIN
- removed net N$6: C13.1, L5.2, U5.+VIN
- removed net N$7: C16.1, L6.2, U6.+VIN
- removed net OE: R62.1, U14.#OE
- removed net PWM1: U1.PWM/ON/OFF, U14.PWM6
- removed net PWM2: U14.PWM5, U2.PWM/ON/OFF
- removed net PWM3: U14.PWM4, U3.PWM/ON/OFF
- removed net PWM4: U14.PWM3, U4.PWM/ON/OFF
- removed net PWM5: U14.PWM2, U5.PWM/ON/OFF
- removed net PWM6: U14.PWM1, U6.PWM/ON/OFF
- removed net SCB1_RX[0]_SCL[0]: R2.1, R3.1, U9.P3[0]
- removed net SCB1_TX[0]_SDA[0]: R4.1, R5.1, U9.P3[1]
- removed net SWD_CLK[0]: J1.SCLK, U9.P3[3]
- removed net SWD_IO[0]: J1.SDAT, U9.P3[2]
- removed net UART_!RE!: TP21.TP, TP30.TP, U10.!RE!, U9.P2[7]
- removed net UART_DE: TP22.TP, TP31.TP, U10.DE, U9.P2[6]
- removed net UART_RX: R3.2, TP20.TP, TP29.TP, U10.RXD
- removed net UART_TX: R5.2, TP11.TP, TP28.TP, U10.TXD
- removed net XRES: J1.XRES, U9.XRES
- net +24V: no longer C12.1(+), C15.1(+), C18.1(+), C3.1(+), C6.1(+), C9.1(+), L1.1, L2.1, L3.1, L4.1, L5.1, L6.1
- net +3V3: no longer C21.1, C27.1, C28.1, C29.1, C31.1, C32.1, J1.VTARG, R1.1, R14.1, R26.1, R28.1, R6.1, R7.1, R8.1, R9.1, SJ_A0.1, SJ_A1.1, SJ_A16.1, SJ_A2.1, SJ_A3.1, SJ_A4.1, SJ_A5.1, TP19.TP, TP27.TP, U10.VDD1, U14.VDD, U7.AVDD, U7.VREF_IN, U9.VDDD
- net GND: no longer C1.2, C10.2, C11.2, C12.2(-), C13.2, C14.2, C15.2(-), C16.2, C17.2, C18.2(-), C2.2, C21.2, C27.2, C28.2, C29.2, C3.2(-), C31.2, C32.2, C33.2, C4.2, C5.2, C6.2(-), C7.2, C8.2, C9.2(-), J1.GND, R29.1, R56.1, R57.1, R58.1, R59.1, R60.1, R61.1, R62.2, SJ_A17.1, TP9.TP, U1.GND, U10.GND1, U14.EXTCLK, U14.GND, U2.GND, U3.GND, U4.GND, U5.GND, U6.GND, U7.GND, U9.VSS
- net SCL: no longer TP24.TP, U14.SCL, U7.SCL, U9.P4[0]
- net SCL_IN: no longer R2.2, TP26.TP
- net SDA: no longer TP18.TP, U14.SDA, U7.SDA, U9.P4[1]
- net SDA_IN: no longer R4.2, TP25.TP
Other:
- note removed: "1 + A5 + A4 + A3 + A2 + A1 +A1 + RW"
- note removed: "24V-0.7A Current Regulators"
- note removed: "6-Channel 24V, 700mA (per channel) Current Regulator Module w/I2C Controlled Dimming via PWM or Analog Signaling"
- note removed: "Communication Mode Select"
- note removed: "I2C Address ="
- note removed: "I2C to 8-Channel 8-Bit DAC"
- note removed: "Notes: - GND !LDAC! for syncronous mode - Broadcast I2C Addr = 0x47 - ADDR0=Low, I2C Addr=0x48 - ADDR0=High, I2C Addr=0x4A - ADDR0=Float, I2C Addr=0x4C"
- note removed: "Notes: - P4[0] is SCB0_I2C_SCL - P4[1] is SCB0_I2C_SDA"
- note removed: "Open = 0 / Closed = 1"
- note removed: "PCA9685 16-Channel I2C PWM Driver"
- note removed: "PSOC 4100 Microcontroller"
- note removed: "PSOC 4100 Programming Header"
- note removed: "PSOC4100 Microcontroller w/I2C or RS485 Communication + Programming Header"
- note removed: "RJ12 Connectors"
- note removed: "RS485 Connection Pair w/UART Transceiver"
- note removed: "RS485 Isolator"
- note removed: "Testpads"
- moved on the sheet: C35, C36, D7, D8, J4, J7, J8, L8, R13, R32, R33, R42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
