File: proj/light-controller/v2.2/light_controller.brd (EAGLE design)
At the start: 123.2 x 125.7 mm, 219 parts, among them J1 0022232051, J2 PJ-036AH, J4 54602-908LF, J5 A-2004-1-4-LP-N-R, J6 A-2004-1-4-LP-N-R, J7 I2C-HEADER, J8 54602-908LF, U1 RCD-24-0.70/VREF, U10 PCA9685, U11 PCA9615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

Commit message: added BOM for light controlled v2.2
Parts:
- added F1: Use 5A Fuse, openag-fuses:FUSE-CARTRIDGE
Other:
- board text removed: "5A Fuse"
