File: prj/photon-rj45/v2.0/photon_rj45.brd (EAGLE design)
At the start: 120.7 x 54.6 mm, 2 parts

Commit message: added photon rj45 board v2.0
Parts:
- removed U$2: TITLE, openag-frames:TITLE
- added C1, C5: 0.1uF, openag-capacitors:C0603
- added C2, C4: 4.7uF, openag-capacitors:C0805
- added C3, C7: 10uF, openag-capacitors:C0805
- added D1, D2: APT1608, openag-diodes:CHIPLED_0603
- added D3: SMAJ26A, openag-diodes:SMA
- added F1: SSQ5, openag-fuses:SS
- added J1: 54602-908LF, openag-connectors:RJ45-DI2C-USB-54602-908LF
- added J3: PJ-036AH, openag-connectors:BARREL-JACK-PJ-036AH
- added R1: 100, openag-resistors:RC0603N
- added R16, R18, R19, R20: 600, openag-resistors:RC0603N
- added R17, R21: 120, openag-resistors:RC0603N
- added R22, R23: 10K, openag-resistors:RC0603N
- added R24: 1K, openag-resistors:RC0603N
- added U1: PHOTONH, openag-microcontrollers:PHOTON-NO-BOTTOM-LABELS
- added U3: R-78E5.0-1.0, openag-regulators:R-78E5.0-1.0
- added U4: PCA9615, openag-buffers:SOP50P490X110-10N
- U$1: value AUTHOR -> (none); device openag-frames:AUTHOR -> openag-frames:LOGO-BARE-750
- moved U$1 11.2 mm to (3.56, 1.78), flipped to the bottom, turned to 90 degrees
Connections:
- new net +24V: C3.1, C4.1, C5.1, D3.1, F1.2, J1.24V(6), R1.2, R24.2, U3.1
- new net +3V3: C1.1, C2.1, R22.2, R23.2, U1.24, U4.1
- new net +5V: C7.1, R18.1, R19.2, U1.1, U3.3, U4.10
- new net 24V_IN1: F1.1, J3.1
- new net DSCLM_1: J1.DSCLM(5), R20.2, R21.1, U4.6
- new net DSCLP_1: J1.DSCLP(4), R19.1, R21.2, U4.7
- new net DSDAM_1: J1.DSDAM(2), R16.1, R17.2, U4.9
- new net DSDAP_1: J1.DSDAP(1), R17.1, R18.2, U4.8
- new net GND: C1.2, C2.2, C3.2, C4.2, C5.2, C7.2, D1.C, D2.C, D3.2, J1.GND(3), J3.2, J3.3, R16.2, R20.1, U1.2, U1.21, U3.2, U4.5
- new net N$5: D2.A, R24.1
- new net N$6: D1.A, R1.1
- new net SCL_IN: R23.1, U4.4
- new net SDA_IN: R22.1, U4.2
- new net USBM: J1.USBM(8)
- new net USBP: J1.USBP(7)
- new net VBAT: U1.22
Routing:
- net +24V: track 0.00 -> 90.9 mm, vias 0 -> 1
- net +5V: track 0.00 -> 53.3 mm, vias 0 -> 3
- net +3V3: track 0.00 -> 48.1 mm, vias 0 -> 2
- net DSDAP_1: track 0.00 -> 19.0 mm
- net DSDAM_1: track 0.00 -> 16.8 mm
- net DSCLM_1: track 0.00 -> 13.2 mm
- net DSCLP_1: track 0.00 -> 12.8 mm
- net SCL_IN: track 0.00 -> 11.4 mm
- net GND: track 0.00 -> 10.1 mm, vias 0 -> 2
- net SDA_IN: track 0.00 -> 6.33 mm
- net 24V_IN1: track 0.00 -> 4.45 mm
- net N$6: track 0.00 -> 2.24 mm
- net N$5: track 0.00 -> 1.89 mm
Other:
- board size 120.7 x 54.6 mm -> 54.6 x 22.9 mm
- board text added: "Photon RJ45 v2.0"

Commit message: updated keyboard shortcuts and fixed i2c resistor values on light controller v2.2
Parts:
- added J2: PJ-036AH, openag-connectors:BARREL-JACK-PJ-036AH
- added J4: PPTC121LFBN-RC, openag-connectors:NAME-VALUE-ONLY
- J3: value PJ-036AH -> PPTC121LFBN-RC; device openag-connectors:BARREL-JACK-PJ-036AH -> openag-connectors:NAME-VALUE-ONLY
- moved J3 36.8 mm to (47.9, 1.78), flipped to the bottom
Connections:
- net 24V_IN1: now also J2.1; no longer J3.1
- net GND: now also J2.2, J2.3; no longer J3.2, J3.3
Changed lines of the file:
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@@
 <setting verticaltext="up"/>
 </settings>
-<grid distance="50" unitdist="mil" unit="mil" style="lines" multiple="1" display="yes" altdistance="5" altunitdist="mil" altunit="mil"/>
+<grid distance="10" unitdist="mil" unit="mil" style="lines" multiple="1" display="yes" altdistance="5" altunitdist="mil" altunit="mil"/>
 <layers>
 <layer number="1" name="Top" color="4" fill="1" visible="yes" active="yes"/>
@@
 <attribute name="VPN" value="SMAJ26A-FDICT-ND" x="14.732" y="3.556" size="1.778" layer="27" rot="R270" display="off"/>
 </element>
-<element name="J3" library="openag-connectors" package="BARREL-JACK-PJ-036AH" value="PJ-036AH" x="12.2428" y="10.795" smashed="yes">
+<element name="J2" library="openag-connectors" package="BARREL-JACK-PJ-036AH" value="PJ-036AH" x="12.2428" y="10.795" smashed="yes">
 <attribute name="MANUFACTURER" value="CUI Inc." x="12.2428" y="10.795" size="1.778" layer="27" display="off"/>
 <attribute name="MPN" value="PJ-036AH-SMT-TR" x="12.2428" y="10.795" size="1.778" layer="27" display="off"/>
@@
 </element>
 <element name="U$1" library="openag-frames" package="LOGO-BARE-750" value="" x="3.556" y="1.778" rot="MR90"/>
+<element name="J3" library="openag-connectors" package="NAME-VALUE-ONLY" value="PPTC121LFBN-RC" x="47.879" y="1.778" smashed="yes" rot="MR0">
+<attribute name="MANUFACTURER" value="Sullins Connector Solutions" x="47.879" y="1.778" size="1.778" layer="28" rot="MR0" display="off"/>
+<attribute name="MPN" value="PPTC121LFBN-RC" x="47.879" y="1.778" size="1.778" layer="28" rot="MR0" display="off"/>
+<attribute name="NAME" x="47.879" y="1.778" size="0.762" layer="26" rot="MR90"/>
+<attribute name="VALUE" x="46.101" y="1.778" size="0.762" layer="28" rot="MR0"/>
+<attribute name="VENDOR" value="Digikey" x="47.879" y="1.778" size="1.778" layer="28" rot="MR0" display="off"/>
+<attribute name="VLINK" value="https://www.digikey.com/product-detail/en/sullins-connector-solutions/PPTC121LFBN-RC/S6100-ND/807231#" x="47.879" y="1.778" size="1.778" layer="28" rot="MR0" display="off"/>
+<attribute name="VPN" value="S6100-ND" x="47.879" y="1.778" size="1.778" layer="28" rot="MR0" display="off"/>
+</element>
+<element name="J4" library="openag-connectors" package="NAME-VALUE-ONLY" value="PPTC121LFBN-RC" x="48.006" y="19.304" smashed="yes" rot="MR0">
+<attribute name="MANUFACTURER" value="Sullins Connector Solutions" x="48.006" y="19.304" size="1.778" layer="28" rot="MR0" display="off"/>
+<attribute name="MPN" value="PPTC121LFBN-RC" x="48.006" y="19.304" size="1.778" layer="28" rot="MR0" display="off"/>
+<attribute name="NAME" x="48.006" y="19.304" size="0.762" layer="26" rot="MR90"/>
+<attribute name="VALUE" x="45.466" y="19.304" size="0.762" layer="28" rot="MR0"/>
+<attribute name="VENDOR" value="Digikey" x="48.006" y="19.304" size="1.778" layer="28" rot="MR0" display="off"/>
+<attribute name="VLINK" value="https://www.digikey.com/product-detail/en/sullins-connector-solutions/PPTC121LFBN-RC/S6100-ND/807231#" x="48.006" y="19.304" size="1.778" layer="28" rot="MR0" display="off"/>
+<attribute name="VPN" value="S6100-ND" x="48.006" y="19.304" size="1.778" layer="28" rot="MR0" display="off"/>
+</element>
 </elements>
 <signals>
@@
 <contactref element="D1" pad="C"/>
 <contactref element="D3" pad="2"/>
-<contactref element="J3" pad="2"/>
-<contactref element="J3" pad="3"/>
+<contactref element="J2" pad="2"/>
+<contactref element="J2" pad="3"/>
 <contactref element="U1" pad="2"/>
 <wire x1="34.6202" y1="5.957" x2="35.294" y2="5.957" width="0.3048" layer="1"/>
@@
 </signal>
 <signal name="24V_IN1">
-<contactref element="J3" pad="1"/>
+<contactref element="J2" pad="1"/>
 <contactref element="F1" pad="1"/>
 <wire x1="15.113" y1="14.0081" x2="15.113" y2="10.2368" width="1.27" layer="1"/>
