File: prj/relay/relay.sch (EAGLE design)
At the start: 16 parts

Commit message: mech
Parts:
- added C1, C2, C4: 10uF, openag-capacitors:10UF-GMK212BBJ106KG-T
- added D4, D6: APT1608, openag-diodes:APT1608CGCK
- added J1, J2: 54602-908LF, openag-connectors:RJ45-DI2C-USB-54602-908LFPTH
- added L1: 33uH, openag-inductors:33UH-29333C
- added R10, R11: 2.2k, openag-resistors:2.2K-RC0603JR-072K2L
- added R12: 1K, openag-resistors:1K-ERJ-PB3D1001V
- added R13, R14, R15, R16, R4, R6, R7, R8: 600, openag-resistors:600OHM-RC0603FR-07604RL
- added R17, R18, R5, R9: 120, openag-resistors:120OHM-RC0603FR-07120RL
- added R19, R3: 100, openag-resistors:100OHM-RC0603JR-07100RL
- added SJ2: (no value), openag-connectors:EMI-BYPASS
- added TP10, TP11, TP13, TP14, TP15, TP16, TP17, TP18, TP19, TP20, TP6, TP7, TP8, TP9: TPTP04R, openag-testpads:TPTP04R
- added TP2, TP4, TP5: TPTP06R, openag-testpads:TPTP06R
- added U1: MCP4725A0T-E/CHSOT-23-6_MC-L, openag-dacs:MCP4725A0T-E/CHSOT-23-6_MC-L
- added U2: R-78E5.0-1.0, openag-regulators:R-78E5.0-1.0
- added U3, U4: PCA9615, openag-buffers:PCA9615DPJ
Connections:
- new net +3V3: R10.2, R11.2, TP15.TP, TP6.TP, U3.VDD_(A), U4.VDD_(A)
- new net DSCLM_1: J1.DSCLM, R8.2, R9.1, U3.DSCLM
- new net DSCLM_2: J2.DSCLM, R15.2, R17.1, U4.DSCLM
- new net DSCLP_1: J1.DSCLP, R7.1, R9.2, U3.DSCLP
- new net DSCLP_2: J2.DSCLP, R16.1, R17.2, U4.DSCLP
- new net DSDAM_1: J1.DSDAM, R4.1, R5.2, U3.DSDAM
- new net DSDAM_2: J2.DSDAM, R13.1, R18.2, U4.DSDAM
- new net DSDAP_1: J1.DSDAP, R5.1, R6.2, U3.DSDAP
- new net DSDAP_3: J2.DSDAP, R14.2, R18.1, U4.DSDAP
- new net N$32: R19.2, U1.A0
- new net N$33: D4.A, R3.1
- new net N$43: D6.A, R12.1
- new net SCL_IN: R11.1, TP11.TP, TP19.TP, U1.SCL, U3.SCL, U4.SCL
- new net SDA_IN: R10.1, TP10.TP, TP20.TP, U1.SDA, U3.SDA, U4.SDA
- new net USBM: J1.USBM, J2.USBM, TP14.TP
- new net USBP: J1.USBP, J2.USBP, TP13.TP
- net +24V: now also C4.1, J1.+24V, J2.+24V, L1.1, R12.2, SJ2.1, TP17.TP, TP4.TP, TP9.TP
- net +5V: now also C2.1, R14.1, R16.2, R3.2, R6.1, R7.2, TP16.TP, TP2.TP, TP7.TP, U1.VDD, U2.VOUT, U3.VDD_(B), U4.VDD_(B)
- net 24V_EMI: now also C1.1, L1.2, SJ2.2, U2.VIN
- net GND: now also C1.2, C2.2, C4.2, D4.C, D6.C, R13.2, R15.1, R19.1, R4.2, R8.1, TP18.TP, TP5.TP, TP8.TP, U1.VSS, U2.GND, U3.VSS, U4.VSS
- net N$31: now also U1.VOUT
Other:
- note added: "I2C Pullup"
- note added: "RJ45 Connector Pair w/dI2C Redriver"
- note added: "RJ45 Connectors"
- note added: "dI2C Buffer Channel 1"
- note added: "dI2C Buffer Channel 2"
- moved on the sheet: D1, F1, R2, RELAY_1
