File: prj/pfc-edu/v2.0/PFCEDU_V2.sch (EAGLE design)
At the start: 235 parts, among them IC2 PCA9615DP, IC3 PCA9615DP, J2 54602-908LF, J3 54602-908LF, Q1 MMBT2222A, Q2 MMBT2222A, Q3 MMBT2222A, Q4 MMBT2222A, Q5 MMBT2222A, T1 R-78E5.0-1.0, T2 R-78E12.0-1.0, U1 TCA9548APWRPW24-M, U10 HPP845E034R5, U11 SHT25, U12 T6713-5K, U17 LM2937IMP3.3NOPB, U2 STD12NF06LT4, U20 RCD-24-0.70/VREF, U21 RCD-24-0.70/VREF, U22 RCD-24-0.70/VREF, U23 RCD-24-0.70/VREF, U24 RCD-24-0.70/VREF, U25 RCD-24-0.70/VREF, U27 DAC5578SPW, U3 STD12NF06LT4, U30 PCA9685, U4 PCF8574APWRPW20-M, U5 STD12NF06LT4, U6 STD12NF06LT4, U7 STD12NF06LT4, U9 CCS811

Commit message: PCB update
Connections:
- net +5V: no longer U$4.SYS5V
Changed lines of the file:
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@@
 <?xml version="1.0" encoding="utf-8"?>
 <!DOCTYPE eagle SYSTEM "eagle.dtd">
-<eagle version="9.0.1">
+<eagle version="9.1.1">
 <drawing>
 <settings>
@@
 <wire x1="-261.62" y1="266.7" x2="-284.48" y2="266.7" width="0.1524" layer="91"/>
 <wire x1="-284.48" y1="266.7" x2="-284.48" y2="281.94" width="0.1524" layer="91"/>
-<pinref part="U$4" gate="G$1" pin="SYS5V"/>
-<wire x1="-261.62" y1="261.62" x2="-284.48" y2="261.62" width="0.1524" layer="91"/>
-<wire x1="-284.48" y1="261.62" x2="-284.48" y2="266.7" width="0.1524" layer="91"/>
-<junction x="-284.48" y="266.7"/>
-</segment>
-<segment>
+</segment>
+<segment>
