File: prj/pfc-edu/v3.0/PFCEDU_V3.brd (EAGLE design)
At the start: 403.9 x 355.1 mm, 269 parts, among them IC2 PCA9615DP, IC3 PCA9615DP, J2 54602-908LF, J3 54602-908LF, Q1 MMBT2222A, Q2 MMBT2222A, Q3 MMBT2222A, Q4 MMBT2222A, Q5 MMBT2222A, T1 R-78E5.0-1.0, T2 R-78E12.0-1.0, U1 TCA9548APWRPW24-M, U10 HPP845E034R5, U11 SHT25, U12 T6713-5K, U17 LM2937-3.3V, U18 DAC5578, U2 STD12NF06LT4, U3 STD12NF06LT4, U4 PCF8574APWRPW20-M, U5 STD12NF06LT4, U6 STD12NF06LT4, U7 STD12NF06LT4, U9 CCS811

Commit message: PCB update
Parts:
- removed C5: .1uF, rcl:C0603@1
- removed PAD1, PAD15, PAD16, PAD17, PAD18, PAD2, PAD3, PAD4, PAD5, PAD6: WIREPAD3,81/1,3, wirepad:3,81/1,3
- removed Q1, Q2, Q3, Q4, Q5: MMBT2222A, transistor-npn:SOT23-BEC
- removed R15, R32: 10K, SparkFun-Resistors:0603-RES
- removed R47, R50, R51, R52: (no value), rcl:R0805W
- removed TP102, TP103: TPTP04R, openag-testpads:TP04R
- removed U3: STD12NF06LT4, OpenAG_I2C:DPAK
- removed U4: PCF8574APWRPW20-M, IO_Expander:PW20-M
- added C10, C12, C17, C18, C19, C2, C20, C23, C24, C25, C27, C4: 0.1uF, openag-capacitors:C0603
- added J1, J5, J6: 5-1634503-1, openag-connectors:CONN5_5-1634503-1
- added J10, J8, J9: ATLAS-STAMP, openag-connectors:ATLAS-STAMP
- added J7: UJ2-AV-1-SMT, UJ2-AV-1-SMT:CUI_UJ2-AV-1-SMT
- added T3, T4: (no value), zetex:SOT-23
- added U$5, U$6: USB_RIGHT, openag-connectors:USB_RIGHT
- added U13: ISO1540, openag-isolators:D8
- added U8: RM-3.33.3S, openag-isolators:RM3.33.3S-SIP4
- F1: value 0448.400MR -> 400mA
- R14: value 10K -> (none); device SparkFun-Resistors:0603-RES -> rcl:R0805W
- R33, R37, R39, R40: value 10K -> 1K; device SparkFun-Resistors:0603-RES -> openag-resistors:RC0603N
- R34, R35, R36, R38, R41, R43, R45, R46: value (none) -> 1K; device rcl:R0805W -> openag-resistors:RC0603N
- U2, U6: value STD12NF06LT4 -> RM-3.33.3S; device OpenAG_I2C:DPAK -> openag-isolators:RM3.33.3S-SIP4
- U5, U7: value STD12NF06LT4 -> ISO1540; device OpenAG_I2C:DPAK -> openag-isolators:D8
- moved R46 305.0 mm to (249.7, 274.8), turned to 0 degrees
- moved R45 289.1 mm to (249.7, 277.4)
- moved R41 285.8 mm to (249.7, 276.1), turned to 0 degrees
- moved R35 262.9 mm to (30.2, 9.14), turned to 180 degrees
- moved R34 261.4 mm to (30.2, 13.0), turned to 180 degrees
- moved R38 248.8 mm to (19.6, 254.3)
- moved U2 247.4 mm to (50.8, 7.49), turned to 90 degrees
- moved R14 242.3 mm to (223.5, 30.7), turned to 0 degrees
- moved U6 240.6 mm to (14.1, 233.7)
- moved U7 237.8 mm to (18.3, 248.7)
- moved R13 209.9 mm to (223.5, 34.0), turned to 0 degrees
- moved R33 198.9 mm to (30.2, 10.4), turned to 180 degrees
- moved R43 119.0 mm to (249.7, 273.6), turned to 0 degrees
- moved U$9 112.5 mm to (140.1, 3.08)
- moved U5 97.0 mm to (35.8, 11.7), turned to 90 degrees
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Connections:
- removed net A0_IO: R14.1, R33.2, U4.6
- removed net A1_IO: R15.1, R32.2, U4.7
- removed net LED+_2: C75.2, LED+7.MP, RS7.1, TP120.TP, U$26.4
- removed net LED+_3: C78.2, LED+9.MP, RS9.1, TP125.TP, U$27.4
- removed net LED+_4: C81.2, LED+10.MP, RS10.1, TP130.TP, U$28.4
- removed net LED+_5: C84.2, LED+11.MP, RS11.1, TP135.TP, U$29.4
- removed net LED+_6: C87.2, LED+12.MP, RS12.1, TP140.TP, U$30.4
- removed net LED-: C72.1, L14.2, LED-2.MP, TP112.TP
- removed net LED-_2: C75.1, L16.2, LED-7.MP, TP117.TP
- removed net LED-_3: C78.1, L17.2, LED-9.MP, TP122.TP
- removed net LED-_4: C81.1, L18.2, LED-10.MP, TP127.TP
- removed net LED-_5: C84.1, L19.2, LED-11.MP, TP132.TP
- removed net LED-_6: C87.1, L20.2, LED-12.MP, TP137.TP
- removed net MOS1: PAD3.1, U3.3
- removed net MOS2: PAD1.1, U2.3
- removed net MOS3: PAD5.1, U5.3
- removed net MOS4: PAD15.1, U6.3
- removed net MOS5: PAD17.1, U7.3
- removed net N$13: R37.1, U4.1
- removed net N$14: Q2.C, R34.1, U2.1
- removed net N$15: Q2.B, R35.1
- removed net N$16: Q3.C, R38.1, U5.1
- removed net N$17: Q3.B, R41.1
- removed net N$6: Q5.C, R50.1, U7.1
- removed net N$7: Q5.B, R51.1
- removed net N$9: Q1.B, R36.1
- removed net P0_IO: R35.2, R43.2, U4.10
- removed net P1_IO: R48.2, R49.2, U4.11
- removed net P2_IO: R51.2, R52.2, U4.12
- removed net P3_IO: U4.14
- removed net P4_IO: U4.16
- removed net P5_IO: U4.17
- removed net P6_IO: R41.2, R45.2, U4.19
- removed net P7_IO: R36.2, R46.2, U4.20
- new net D+: J7.2, U$5.PIN2, U$6.PIN2
- new net D-: J7.3, U$5.PIN3, U$6.PIN3
- new net ISO_3V3_2: C12.1, C4.1, J9.4, R34.2, R36.2, U2.4, U5.8
- new net ISO_3V3_3: C18.1, C20.1, J10.4, R38.2, R40.2, U6.4, U7.8
- new net ISO_3V3_4: C24.1, C27.1, J8.4, R43.2, R46.2, U13.8, U8.4
- new net ISO_GND_2: C12.2, C4.2, J9.3, U2.3, U5.5
- new net ISO_GND_3: C18.2, C20.2, J10.3, U6.3, U7.5
- new net ISO_GND_4: C24.2, C27.2, J8.3, U13.5, U8.3
- new net ISO_SCL_2: J9.1, R36.1, U5.6
- new net ISO_SCL_3: J10.1, R40.1, U7.6
- new net ISO_SCL_4: J8.1, R46.1, U13.6
- new net ISO_SDA_2: J9.2, R34.1, U5.7
- new net ISO_SDA_3: J10.2, R38.1, U7.7
- new net ISO_SDA_4: J8.2, R43.1, U13.7
- new net N$8: T4.1, U$5.PIN4
- new net PGND_2: J1.2, J1.3, J1.4, J1.5, J9.6
- new net PGND_3: J10.6, J6.2, J6.3, J6.4, J6.5
- new net PGND_4: J5.2, J5.3, J5.4, J5.5, J8.6
- new net PRB_2: J1.1, J9.5
- new net PRB_3: J10.5, J6.1
- new net PRB_4: J5.1, J8.5
- new net USB1: R49.2, U18.12
- new net USB2: R14.2, U18.13
- new net V+: J7.1, U$5.PIN1, U$6.PIN1
- net +12V: no longer PAD2.1, PAD4.1, PAD6.1, R13.2, R34.2, R38.2, R43.1, R45.1, R46.1, R47.2, R49.1, R50.2, R52.1
- net +3V3: now also C10.1, C17.1, C19.1, C2.1, C23.1, C25.1, R33.2, R35.2, R41.2, R45.2, U13.1, U2.2, U5.1, U6.2, U7.1, U8.2; no longer C5.1, R14.2, R15.2, R40.2, U4.5
- net +5V: no longer PAD16.1, PAD18.1, U$4.SYS5V, U$4.SYS5V1
- net CH1+: now also LED+2.MP, TP115.TP
- net CH1-: now also C72.1, L14.2, LED-2.MP, TP112.TP
- net CH2+: now also C75.2, LED+7.MP, RS7.1, TP120.TP, U$26.4
- net CH2-: now also C75.1, L16.2, LED-7.MP, TP117.TP
- net CH3+: now also C78.2, LED+9.MP, RS9.1, TP125.TP, U$27.4
- net CH3-: now also C78.1, L17.2, LED-9.MP, TP122.TP
- net CH4+: now also C81.2, LED+10.MP, RS10.1, TP130.TP, U$28.4
- net CH4-: now also C81.1, L18.2, LED-10.MP, TP127.TP
- net CH5+: now also C84.2, LED+11.MP, RS11.1, TP135.TP, U$29.4
- net CH5-: now also C84.1, L19.2, LED-11.MP, TP132.TP
- net CH6+: now also C87.2, LED+12.MP, RS12.1, TP140.TP, U$30.4
- net CH6-: now also C87.1, L20.2, LED-12.MP, TP137.TP
- net GND: now also C10.2, C17.2, C19.2, C2.2, C23.2, C25.2, R13.2, R48.2, T3.2, T4.2, U$5.GND1, U$5.GND2, U$5.GND3, U$5.GND4, U$6.PIN4, U13.4, U2.1, U5.4, U6.1, U7.4, U8.1; no longer C5.2, Q1.E, Q2.E, Q3.E, Q4.E, Q5.E, R32.1, R33.1, U2.2, U3.2, U4.15, U4.9, U5.2, U6.2, U7.2
- net LED+: no longer LED+2.MP, TP115.TP
- net N$1: now also R13.1, R14.1, T4.3; no longer Q4.C, R47.1, U6.1
- net N$3: now also R49.1, T3.3; no longer Q4.B
- net N$5: now also J7.4, T3.1; no longer Q1.C, R13.1, U3.1
- net SC3: now also U18.16
- net SC5: no longer R39.1, U4.2
- net SC6: now also R33.1, R37.1, R41.1, U13.3, U5.3, U7.3
- net SCL: no longer TP103.1, U18.16
- net SD3: now also U18.15
- net SD5: no longer R40.1, U4.4
- net SD6: now also R35.1, R39.1, R45.1, U13.2, U5.2, U7.2
- net SDA: no longer TP102.1, U18.15
Routing:
- net SC6: track 0.00 -> 756.4 mm, vias 0 -> 4
- net SD6: track 0.00 -> 630.9 mm, vias 0 -> 3
- net +12V: track 703.7 -> 366.4 mm, vias 6 -> 0
- net V+: track 0.00 -> 329.3 mm, vias 0 -> 5
- net D+: track 0.00 -> 315.1 mm, vias 0 -> 2
- net D-: track 0.00 -> 314.1 mm
- net P2_IO: track 311.6 -> 0.00 mm, vias 6 -> 0
- net P1_IO: track 277.2 -> 0.00 mm, vias 4 -> 0
- net P6_IO: track 250.3 -> 0.00 mm, vias 2 -> 0
- net +3V3: track 943.9 -> 1137.3 mm, vias 16 -> 21
- net USB2: track 0.00 -> 161.0 mm, vias 0 -> 4
- net P7_IO: track 144.4 -> 0.00 mm, vias 2 -> 0
- net USB1: track 0.00 -> 142.7 mm, vias 0 -> 4
- net P0_IO: track 142.7 -> 0.00 mm, vias 6 -> 0
- net CH2+: track 93.2 -> 151.2 mm
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- added copper zone on layer 1, net CH1+
- added copper zone on layer 1, net CH1-
- added copper zone on layer 1, net CH2+
- added copper zone on layer 1, net CH2-
- added copper zone on layer 1, net CH3+
- added copper zone on layer 1, net CH3-
- added copper zone on layer 1, net CH4+
- added copper zone on layer 1, net CH4-
- added copper zone on layer 1, net CH5+
- added copper zone on layer 1, net CH5-
- added copper zone on layer 1, net CH6+
- added copper zone on layer 1, net CH6-
- removed copper zone on layer 1, net LED+
- removed copper zone on layer 1, net LED+_2
- removed copper zone on layer 1, net LED+_3
- removed copper zone on layer 1, net LED+_4
- removed copper zone on layer 1, net LED+_5
- removed copper zone on layer 1, net LED+_6
- removed copper zone on layer 1, net LED-
- removed copper zone on layer 1, net LED-_2
- removed copper zone on layer 1, net LED-_3
- removed copper zone on layer 1, net LED-_4
- removed copper zone on layer 1, net LED-_5
- removed copper zone on layer 1, net LED-_6
Other:
- outline, holes or cut-outs redrawn
- board text removed: "Changelog - replaced 24v-to-5v regulator with R78E5 - added dual i2c buffers - updated to style conventions v1.0"
- board text removed: "Drives x6 channels of LEDs by regulating the current up to 700mA (per channel) at 24V. Communicates via dI2C or RS485 (See enables on PSOC module). To communicate directly with the board ICs and avoid programming the PSOC, enable I2C Connect. Current regulators can be driven by either dimming or PWM control."
