File: prj/pfc-edu/v3.0/PFCEDU_V3.sch (EAGLE design)
At the start: 266 parts, among them IC2 PCA9615DP, IC3 PCA9615DP, J2 54602-908LF, J3 54602-908LF, Q1 MMBT2222A, Q2 MMBT2222A, Q3 MMBT2222A, Q4 MMBT2222A, Q5 MMBT2222A, T1 R-78E5.0-1.0, T2 R-78E12.0-1.0, U1 TCA9548APWRPW24-M, U10 HPP845E034R5, U11 SHT25, U12 T6713-5K, U17 LM2937-3.3V, U18 DAC5578, U2 STD12NF06LT4, U3 STD12NF06LT4, U4 PCF8574APWRPW20-M, U5 STD12NF06LT4, U6 STD12NF06LT4, U7 STD12NF06LT4, U9 CCS811

Commit message: PCB update
Parts:
- removed C5: .1uF, rcl:C-USC0603
- removed PAD1, PAD15, PAD16, PAD17, PAD18, PAD2, PAD3, PAD4, PAD5, PAD6: WIREPAD3,81/1,3, wirepad:WIREPAD3,81/1,3
- removed Q1, Q2, Q3, Q4, Q5: MMBT2222A, transistor-npn:BCF30SMD
- removed R15, R32: 10K, SparkFun-Resistors:10KOHM-1/10W-1%(0603)0603
- removed R47, R50, R51, R52: (no value), rcl:R-US_R0805W
- removed TP102, TP103: TPTP04R, openag-testpads:TPTP04R
- removed U3: STD12NF06LT4, OpenAG_I2C:STD12NF06LT4
- removed U4: PCF8574APWRPW20-M, IO_Expander:PCF8574APWRPW20-M
- added C10, C12, C17, C18, C19, C2, C20, C23, C24, C25, C27, C4: 0.1uF, openag-capacitors:0.1UF-C0603C104K5RACTU
- added J1, J5, J6: 5-1634503-1, openag-connectors:5-1634503-1
- added J10, J8, J9: ATLAS-STAMP, openag-connectors:ATLAS-STAMP
- added J7: UJ2-AV-1-SMT, UJ2-AV-1-SMT:UJ2-AV-1-SMT
- added T3, T4: (no value), zetex:NMOSSOT23
- added U$5, U$6: USB_RIGHT, openag-connectors:USB_RIGHT
- added U13: ISO1540, openag-isolators:ISO1540DR
- added U8: RM-3.33.3S, openag-isolators:RM3.33.3S
- ATTRIBUTES: DESCRIPTION PFC EDU -> (none)
- F1: value 0448.400MR -> 400mA
- R14: value 10K -> (none); device SparkFun-Resistors:10KOHM-1/10W-1%(0603)0603 -> rcl:R-US_R0805W
- R33, R37, R39, R40: value 10K -> 1K; device SparkFun-Resistors:10KOHM-1/10W-1%(0603)0603 -> openag-resistors:1K-ERJ-PB3D1001V
- R34, R35, R36, R38, R41, R43, R45, R46: value (none) -> 1K; device rcl:R-US_R0805W -> openag-resistors:1K-ERJ-PB3D1001V
- U2, U6: value STD12NF06LT4 -> RM-3.33.3S; device OpenAG_I2C:STD12NF06LT4 -> openag-isolators:RM3.33.3S
- U5, U7: value STD12NF06LT4 -> ISO1540; device OpenAG_I2C:STD12NF06LT4 -> openag-isolators:ISO1540DR
Connections:
- removed net A0_IO: R14.1, R33.2, U4.A0
- removed net A1_IO: R15.1, R32.2, U4.A1
- removed net LED+_2: C75.2, LED+7.MP, RS7.1, TP120.TP, U$26.ISEN
- removed net LED+_3: C78.2, LED+9.MP, RS9.1, TP125.TP, U$27.ISEN
- removed net LED+_4: C81.2, LED+10.MP, RS10.1, TP130.TP, U$28.ISEN
- removed net LED+_5: C84.2, LED+11.MP, RS11.1, TP135.TP, U$29.ISEN
- removed net LED+_6: C87.2, LED+12.MP, RS12.1, TP140.TP, U$30.ISEN
- removed net LED-: C72.1, L14.2, LED-2.MP, TP112.TP
- removed net LED-_2: C75.1, L16.2, LED-7.MP, TP117.TP
- removed net LED-_3: C78.1, L17.2, LED-9.MP, TP122.TP
- removed net LED-_4: C81.1, L18.2, LED-10.MP, TP127.TP
- removed net LED-_5: C84.1, L19.2, LED-11.MP, TP132.TP
- removed net LED-_6: C87.1, L20.2, LED-12.MP, TP137.TP
- removed net MOS1: PAD3.P, U3.2
- removed net MOS2: PAD1.P, U2.2
- removed net MOS3: PAD5.P, U5.2
- removed net MOS4: PAD15.P, U6.2
- removed net MOS5: PAD17.P, U7.2
- removed net N$13: R37.1, U4.!INT
- removed net N$14: Q2.C, R34.1, U2.1
- removed net N$15: Q2.B, R35.1
- removed net N$16: Q3.C, R38.1, U5.1
- removed net N$17: Q3.B, R41.1
- removed net N$6: Q5.C, R50.1, U7.1
- removed net N$7: Q5.B, R51.1
- removed net N$9: Q1.B, R36.1
- removed net P0_IO: R35.2, R43.2, U4.P0
- removed net P1_IO: R48.2, R49.2, U4.P1
- removed net P2_IO: R51.2, R52.2, U4.P2
- removed net P3_IO: U4.P3
- removed net P4_IO: U4.P4
- removed net P5_IO: U4.P5
- removed net P6_IO: R41.2, R45.2, U4.P6
- removed net P7_IO: R36.2, R46.2, U4.P7
- new net D+: J7.2, U$5.PIN2, U$6.PIN2
- new net D-: J7.3, U$5.PIN3, U$6.PIN3
- new net ISO_3V3_2: C12.1, C4.1, J9.VCC, R34.2, R36.2, U2.+VOUT, U5.VCC2
- new net ISO_3V3_3: C18.1, C20.1, J10.VCC, R38.2, R40.2, U6.+VOUT, U7.VCC2
- new net ISO_3V3_4: C24.1, C27.1, J8.VCC, R43.2, R46.2, U13.VCC2, U8.+VOUT
- new net ISO_GND_2: C12.2, C4.2, J9.GND, U2.-VOUT, U5.GND2
- new net ISO_GND_3: C18.2, C20.2, J10.GND, U6.-VOUT, U7.GND2
- new net ISO_GND_4: C24.2, C27.2, J8.GND, U13.GND2, U8.-VOUT
- new net ISO_SCL_2: J9.RX/SCL, R36.1, U5.SCL2
- new net ISO_SCL_3: J10.RX/SCL, R40.1, U7.SCL2
- new net ISO_SCL_4: J8.RX/SCL, R46.1, U13.SCL2
- new net ISO_SDA_2: J9.TX/SDA, R34.1, U5.SDA2
- new net ISO_SDA_3: J10.TX/SDA, R38.1, U7.SDA2
- new net ISO_SDA_4: J8.TX/SDA, R43.1, U13.SDA2
- new net N$8: T4.D, U$5.PIN4
- new net PGND_2: J1.2, J1.3, J1.4, J1.5, J9.PGND
- new net PGND_3: J10.PGND, J6.2, J6.3, J6.4, J6.5
- new net PGND_4: J5.2, J5.3, J5.4, J5.5, J8.PGND
- new net PRB_2: J1.1, J9.PBR
- new net PRB_3: J10.PBR, J6.1
- new net PRB_4: J5.1, J8.PBR
- new net USB1: R49.2, U18.VOUT_D
- new net USB2: R14.2, U18.VOUT_B
- new net V+: J7.1, U$5.PIN1, U$6.PIN1
- net +12V: no longer PAD2.P, PAD4.P, PAD6.P, R13.2, R34.2, R38.2, R43.1, R45.1, R46.1, R47.2, R49.1, R50.2, R52.1
- net +3V3: now also C10.1, C17.1, C19.1, C2.1, C23.1, C25.1, R33.2, R35.2, R41.2, R45.2, U13.VCC1, U2.+VIN, U5.VCC1, U6.+VIN, U7.VCC1, U8.+VIN; no longer C5.1, R14.2, R15.2, R40.2, U4.VCC
- net +5V: no longer PAD16.P, PAD18.P, U$4.SYS5V
- net CH1+: now also LED+2.MP, TP115.TP
- net CH1-: now also C72.1, L14.2, LED-2.MP, TP112.TP
- net CH2+: now also C75.2, LED+7.MP, RS7.1, TP120.TP, U$26.ISEN
- net CH2-: now also C75.1, L16.2, LED-7.MP, TP117.TP
- net CH3+: now also C78.2, LED+9.MP, RS9.1, TP125.TP, U$27.ISEN
- net CH3-: now also C78.1, L17.2, LED-9.MP, TP122.TP
- net CH4+: now also C81.2, LED+10.MP, RS10.1, TP130.TP, U$28.ISEN
- net CH4-: now also C81.1, L18.2, LED-10.MP, TP127.TP
- net CH5+: now also C84.2, LED+11.MP, RS11.1, TP135.TP, U$29.ISEN
- net CH5-: now also C84.1, L19.2, LED-11.MP, TP132.TP
- net CH6+: now also C87.2, LED+12.MP, RS12.1, TP140.TP, U$30.ISEN
- net CH6-: now also C87.1, L20.2, LED-12.MP, TP137.TP
- net GND: now also C10.2, C17.2, C19.2, C2.2, C23.2, C25.2, R13.2, R48.2, T3.S, T4.S, U$5.CHASIS, U$6.PIN4, U13.GND1, U2.-VIN, U5.GND1, U6.-VIN, U7.GND1, U8.-VIN; no longer C5.2, Q1.E, Q2.E, Q3.E, Q4.E, Q5.E, R32.1, R33.1, U2.3, U3.3, U4.A2, U4.GND, U5.3, U6.3, U7.3
- net LED+: no longer LED+2.MP, TP115.TP
- net N$1: now also R13.1, R14.1, T4.G; no longer Q4.C, R47.1, U6.1
- net N$3: now also R49.1, T3.G; no longer Q4.B
- net N$5: now also J7.4, T3.D; no longer Q1.C, R13.1, U3.1
- net SC3: now also U18.SCL
- net SC5: no longer R39.1, U4.SCL
- net SC6: now also R33.1, R37.1, R41.1, U13.SCL1, U5.SCL1, U7.SCL1
- net SCL: no longer TP103.TP, U18.SCL
- net SD3: now also U18.SDA
- net SD5: no longer R40.1, U4.SDA
- net SD6: now also R35.1, R39.1, R45.1, U13.SDA1, U5.SDA1, U7.SDA1
- net SDA: no longer TP102.TP, U18.SDA
Other:
- note added: "3.3V Isolator"
- note added: "Atlas Sensor Port"
- note added: "Atlas Stamp"
- note added: "BNC Connector"
- note added: "I2C Isolator"
- note added: "USB Control"
- note removed: "6-Channel 24V, 700mA (per channel) Current Regulator Module w/I2C Controlled Dimming via PWM or Analog Signaling"
- moved on the sheet: C16, C21, C26, C30, C70, C72, C73, C74, C75, C76, C77, C78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
