File: prj/light-controller/v3.0/light_controller.sch (EAGLE design)
At the start: 197 parts, among them J2 PJ-036AH, J4 54602-908LF, J7 I2C-HEADER, J8 54602-908LF, Q1 MMBT2222A, Q2 MMBT2222A, Q3 MMBT2222A, Q4 MMBT2222A, Q5 MMBT2222A, Q6 MMBT2222A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

Commit message: test
terst
Parts:
- RS1, RS3, RS4, RS5, RS6, RS8: value .06 ohms -> 6.34 ohm
