File: prj/sensor-nodes/air/v1.1/air.sch (EAGLE design)
At the start: 92 parts, among them J1 54602-908LF, J2 54602-908LF, U1 PCA9615, U2 PCA9615, U3 PHOTONH, U4 R-78E5.0-1.0, U5 SHT25, U6 CCS811, U7 T6713-5K, U8 HPP845E034R5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

Commit message: test
terst
Parts:
- U1, U2: device openag-buffers:PCA9615DPJ -> openag-redrivers:PCA9615DPJ
- U3: device openag-microcontrollers:PHOTONHPHOTONH -> openag-microcontrollers:PHOTONH-LABELS
