File: prj/template/v1.0/Eagle_Template.sch (EAGLE design)
At the start: 265 parts, among them IC2 PCA9615DP, IC3 PCA9615DP, J1 5-1634503-1, J10 ATLAS-STAMP, J2 54602-908LF, J3 54602-908LF, J5 5-1634503-1, J6 5-1634503-1, J7 UJ2-AV-1-SMT, J8 ATLAS-STAMP, J9 ATLAS-STAMP, T1 R-78E5.0-1.0, T2 R-78E12.0-1.0, U1 TCA9548APWRPW24-M, U10 HPP845E034R5, U11 SHT25, U12 T6713-5K, U14 ISO1540, U17 LM2937-3.3V, U18 DAC5578, U2 RM-3.33.3S, U3 ISO1540, U4 ISO1540, U6 RM-3.33.3S, U8 RM-3.33.3S, U9 CCS811

Commit message: test
terst
Parts:
- removed C1, C22, C73, C76, C79, C82, C85, C88: 10uF, openag-capacitors:10UF-GMK212BBJ106KG-T
- removed C10, C12, C13, C14, C15, C16, C17, C18, C19, C2, C20, C21, C23, C24, C25, C26, C27, C4, C70, C72, C74, C75, C77, C78, C80, C81, C83, C84, C86, C87: 0.1uF, openag-capacitors:0.1UF-C0603C104K5RACTU
- removed C11: .1uF, rcl:C-USC0603
- removed C2\2, C30, C5: 4.7uF, openag-capacitors:4.7UF-CL21A475KBQNNNE
- removed CH1-6, CH1-7, CH1-8, CH1-9, CH2-6, CH2-7, CH2-8, CH2-9, CH3-6, CH3-7, CH3-8, CH3-9, CH4-6, CH4-7, CH4-8, CH4-9, CH5-6, CH5-7, CH5-8, CH5-9, CH6-6, CH6-7, CH6-8, CH6-9: XP-E, Tomaszewski:LED_W/THERM-XP-E
- removed D1: SMAJ14A, openag-diodes:SMAJ14A
- removed D2, D3, D4, D8: APT1608, openag-diodes:APT1608CGCK
- removed D20, D21, D22, D23, D24, D25: SBR2A40P1-7, openag-diodes:SBR2A40P1-7
- removed F1: 400mA, openag-fuses:0438.375WR
- removed F12: (no value), fuse:GSH15
- removed IC2, IC3: PCA9615DP, PCA9615DP:PCA9615DP
- removed J1, J5, J6: 5-1634503-1, openag-connectors:5-1634503-1
- removed J10, J8, J9: ATLAS-STAMP, openag-connectors:ATLAS-STAMP
- removed J2, J3: 54602-908LF, openag_connector:OPENAG-V1-RJ45PTH
- removed J7: UJ2-AV-1-SMT, UJ2-AV-1-SMT:UJ2-AV-1-SMT
- removed L14, L16, L17, L18, L19, L20: 100UH, openag-inductors:100UH_BOURNES
- removed LED+10, LED+11, LED+12, LED+2, LED+7, LED+9, LED-10, LED-11, LED-12, LED-2, LED-7, LED-9: SE14, solpad:SE14
- removed PAD10, PAD7, PAD8, PAD9: WIREPAD3,81/1,3, wirepad:WIREPAD3,81/1,3
- removed PAD11, PAD12, PAD13, PAD14: (no value), wirepad:SMD2
- removed R10, R11, R12, R44: 100, openag-resistors:100OHM-RC0603JR-07100RL
- removed R117, R118, R119, R120, R121, R122, R33, R34, R35, R36, R37, R38, R39, R40, R41, R43, R45, R46, R88, R90: 1K, openag-resistors:1K-ERJ-PB3D1001V
- removed R13, R14, R48, R49: (no value), rcl:R-US_R0805W
- removed R16, R18, R19, R20, R24, R26, R27, R28: 600, rcl:R-US_R0603
- removed R17, R21, R25, R29: 120, rcl:R-US_R0603
- removed R22, R23, R30, R31: 10K, rcl:R-US_R0603
- removed R42: 4.7K, openag-resistors:4.7K-RC1206JR-074K7L
- removed R89: 0 OHM, openag-resistors:0OHM-RC0603JR-070RL
- removed RS10, RS11, RS12, RS2, RS7, RS9: 6.34 ohm, openag-resistors:6.3OHM-RC0805FR-076R34L
- removed SJ1, SJ_A1, SJ_A2: (no value), openag-connectors:SOLDERJUMPERREFLOW_NOPASTE
- removed T1: R-78E5.0-1.0, R-78E5.0-1.0:R-78E5.0-1.0
- removed T2: R-78E12.0-1.0, R-78E5.0-1.0:R-78E5.0-1.0
- removed T3, T4: (no value), zetex:NMOSSOT23
- removed TP1, TP112, TP113, TP114, TP115, TP116, TP117, TP118, TP119, TP120, TP121, TP122, TP123, TP124, TP125, TP126, TP127, TP128, TP129, TP130, TP131, TP132, TP133, TP134, TP135, TP136, TP137, TP138, TP139, TP140, TP141, TP2, TP3, TP36, TP37, TP38, TP39, TP40, TP41, TP42, TP43, TP44, TP45, TP5, TP6, TP61, TP62, TP63, TP7: TPTP06R, openag-testpads:TPTP06R
- removed TP100, TP101, TP104, TP105, TP106, TP107, TP99: TPTP04R, openag-testpads:TPTP04R
- removed U$25, U$26, U$27, U$28, U$29, U$30: AL8861, openag-driver-IC:AL8861
- removed U$3: PJ-036AH, PJ-036ah:PJ-036AH
- removed U$4: BBB_SMD, openag-connectors:BBB_SMD
- removed U$5, U$6: USB_RIGHT, openag-connectors:USB_RIGHT
- removed U10: HPP845E034R5, openag-sensors:HPP845E034R5
- removed U11: SHT25, openag-sensors:SHT25
- removed U12: T6713-5K, openag-sensors:T6713-5K
- removed U14, U3, U4: ISO1540, openag-isolators:ISO1540DR
- removed U17: LM2937-3.3V, openag-regulators:LM2937IMP-3.3/NOPB
- removed U18: DAC5578, openag-dacs:DAC5578SPW
- removed U2, U6, U8: RM-3.33.3S, openag-isolators:RM3.33.3S
- removed U9: CCS811, openag-sensors:CCS811
- ATTRIBUTES: TITLE PFC EDU -> NAME HERE
Connections:
- removed net !LDAC!: R89.2, R90.2, TP104.TP, U18.!LDAC!
- removed net +12V: PAD7.P, PAD8.P, T2.+VOUT
- removed net +24V: C1.1, C11.1, C5.1, C70.1, C73.1, C74.1, C76.1, C77.1, C79.1, C80.1, C82.1, C83.1, C85.1, C86.1, C88.1, D1.P$2, D20.-, D21.-, D22.-, D23.-, D24.-, D25.-, F12.2, J2.+24V, J3.+24V, R12.2, RS10.2, RS11.2, RS12.2, RS2.2, RS7.2, RS9.2, T1.+VIN, T2.+VIN, TP113.TP, TP118.TP, TP123.TP, TP128.TP, TP133.TP, TP138.TP, TP99.TP, U$25.VIN, U$26.VIN, U$27.VIN, U$28.VIN, U$29.VIN, U$30.VIN
- removed net +5V: C21.1, IC2.VDD_(B), IC3.VDD_(B), PAD11.P, R11.2, R18.1, R19.2, R26.1, R27.2, T1.+VOUT, TP62.TP, U$4.VDD5V, U17.IN
- removed net 24V_IN: F12.1, U$3.1
- removed net ADDR0: SJ_A1.2, SJ_A2.2, U18.ADDR0
- removed net CH1+: CH1-6.A, LED+2.MP, TP115.TP
- removed net CH1-: C72.1, CH1-9.C, L14.2, LED-2.MP, TP112.TP
- removed net CH2+: C75.2, CH2-6.A, LED+7.MP, RS7.1, TP120.TP, U$26.ISEN
- removed net CH2-: C75.1, CH2-9.C, L16.2, LED-7.MP, TP117.TP
- removed net CH3+: C78.2, CH3-6.A, LED+9.MP, RS9.1, TP125.TP, U$27.ISEN
- removed net CH3-: C78.1, CH3-9.C, L17.2, LED-9.MP, TP122.TP
- removed net CH4+: C81.2, CH4-6.A, LED+10.MP, RS10.1, TP130.TP, U$28.ISEN
- removed net CH4-: C81.1, CH4-9.C, L18.2, LED-10.MP, TP127.TP
- removed net CH5+: C84.2, CH5-6.A, LED+11.MP, RS11.1, TP135.TP, U$29.ISEN
- removed net CH5-: C84.1, CH5-9.C, L19.2, LED-11.MP, TP132.TP
- removed net CH6+: C87.2, CH6-6.A, LED+12.MP, RS12.1, TP140.TP, U$30.ISEN
- removed net CH6-: C87.1, CH6-9.C, L20.2, LED-12.MP, TP137.TP
- removed net D+: J7.2, U$5.PIN2, U$6.PIN2
- removed net D-: J7.3, U$5.PIN3, U$6.PIN3
- removed net DAC_!CLR!: R88.2, TP105.TP, U18.!CLR!
- removed net DSCLM0: IC2.DSCLM, J2.DSCLM, R20.2, R21.1
- removed net DSCLM1: IC3.DSCLM, J3.DSCLM, R28.2, R29.1
- removed net DSCLP0: IC2.DSCLP, J2.DSCLP, R19.1, R21.2
- removed net DSCLP1: IC3.DSCLP, J3.DSCLP, R27.1, R29.2
- removed net DSDAM0: IC2.DSDAM, J2.DSDAM, R16.1, R17.2
- removed net DSDAM1: IC3.DSDAM, J3.DSDAM, R24.1, R25.2
- removed net DSDAP0: IC2.DSDAP, J2.DSDAP, R17.1, R18.2
- removed net DSDAP1: IC3.DSDAP, J3.DSDAP, R25.1, R26.2
- removed net ISO_3V3_2: C12.1, C4.1, J9.VCC, R34.2, R36.2, U2.+VOUT, U3.ISO_VCC2
- removed net ISO_3V3_3: C18.1, C20.1, J10.VCC, R38.2, R40.2, U4.ISO_VCC2, U6.+VOUT
- removed net ISO_3V3_4: C24.1, C27.1, J8.VCC, R43.2, R46.2, U14.ISO_VCC2, U8.+VOUT
- removed net ISO_GND_2: C12.2, C4.2, J9.GND, U2.-VOUT, U3.ISO_GND2
- removed net ISO_GND_3: C18.2, C20.2, J10.GND, U4.ISO_GND2, U6.-VOUT
- removed net ISO_GND_4: C24.2, C27.2, J8.GND, U14.ISO_GND2, U8.-VOUT
- removed net ISO_SCL_2: J9.RX/SCL, R36.1, U3.ISO_SCL2
- removed net ISO_SCL_3: J10.RX/SCL, R40.1, U4.ISO_SCL2
- removed net ISO_SCL_4: J8.RX/SCL, R46.1, U14.ISO_SCL2
- removed net ISO_SDA_2: J9.TX/SDA, R34.1, U3.ISO_SDA2
- removed net ISO_SDA_3: J10.TX/SDA, R38.1, U4.ISO_SDA2
- removed net ISO_SDA_4: J8.TX/SDA, R43.1, U14.ISO_SDA2
- removed net LED+: C72.2, RS2.1, U$25.ISEN
- removed net LX: D20.+, L14.1, U$25.LX
- removed net LX_2: D21.+, L16.1, U$26.LX
- removed net LX_3: D22.+, L17.1, U$27.LX
- removed net LX_4: D23.+, L18.1, U$28.LX
- removed net LX_5: D24.+, L19.1, U$29.LX
- removed net LX_6: D25.+, L20.1, U$30.LX
- removed net N$1: R13.1, R14.1, T4.G
- removed net N$12: D2.A, R10.1
- removed net N$159: CH5-7.C, CH5-8.A
- removed net N$160: CH5-6.C, CH5-7.A
- removed net N$179: D8.A, R44.1
- removed net N$180: C22.1, F1.1, U17.OUT
- removed net N$2: D3.A, R11.1
- removed net N$29: CH2-8.C, CH2-9.A
- removed net N$3: R48.1, R49.1, T3.G
- removed net N$31: CH2-7.C, CH2-8.A
- removed net N$32: CH2-6.C, CH2-7.A
- removed net N$33: CH4-8.C, CH4-9.A
- removed net N$34: CH4-7.C, CH4-8.A
- removed net N$35: CH4-6.C, CH4-7.A
- removed net N$36: CH6-8.C, CH6-9.A
- removed net N$37: CH6-7.C, CH6-8.A
- removed net N$4: D4.A, R12.1
- removed net N$42: U9.PWM, U9.SENSE
- removed net N$43: C13.1, R42.1, U9.NRESET
- removed net N$46: CH6-6.C, CH6-7.A
- removed net N$47: CH1-8.C, CH1-9.A
- removed net N$48: CH1-7.C, CH1-8.A
- removed net N$5: J7.4, T3.D
- removed net N$8: T4.D, U$5.PIN4
- removed net N$81: CH1-6.C, CH1-7.A
- removed net N$82: CH3-8.C, CH3-9.A
- removed net N$83: CH3-7.C, CH3-8.A
- removed net N$84: CH3-6.C, CH3-7.A
- removed net N$85: CH5-8.C, CH5-9.A
- removed net PGND_2: J1.2, J1.3, J1.4, J1.5, J9.PGND
- removed net PGND_3: J10.PGND, J6.2, J6.3, J6.4, J6.5
- removed net PGND_4: J5.2, J5.3, J5.4, J5.5, J8.PGND
- removed net PRB_2: J1.1, J9.PBR
- removed net PRB_3: J10.PBR, J6.1
- removed net PRB_4: J5.1, J8.PBR
- removed net REG_3V3_400MA: R44.2, SJ1.1
- removed net T1: CH1-6.THERM, CH1-7.THERM, CH1-8.THERM, CH1-9.THERM, CH2-6.THERM, CH2-7.THERM, CH2-8.THERM, CH2-9.THERM, CH3-6.THERM, CH3-7.THERM, CH3-8.THERM, CH3-9.THERM, CH4-6.THERM, CH4-7.THERM, CH4-8.THERM, CH4-9.THERM, CH5-6.THERM, CH5-7.THERM, CH5-8.THERM, CH5-9.THERM, CH6-6.THERM, CH6-7.THERM, CH6-8.THERM, CH6-9.THERM
- removed net USB1: R49.2, U18.VOUT_D
- removed net USB2: R14.2, U18.VOUT_B
- removed net USBM0: J2.USBM
- removed net USBM1: J3.USBM
- removed net USBP0: J2.USBP
- removed net USBP1: J3.USBP
- removed net V+: J7.1, U$5.PIN1, U$6.PIN1
- removed net VSET: R117.1, TP116.TP, U$25.VSET, U18.VOUT_G
- removed net VSET_2: R118.1, TP121.TP, U$26.VSET, U18.VOUT_E
- removed net VSET_3: R119.1, TP126.TP, U$27.VSET, U18.VOUT_C
- removed net VSET_4: R120.1, TP131.TP, U$28.VSET, U18.VOUT_A
- removed net VSET_5: R121.1, TP136.TP, U$29.VSET, U18.VOUT_H
- removed net VSET_6: R122.1, TP141.TP, U$30.VSET, U18.VOUT_F
- net +3V3: no longer C10.1, C14.1, C15.1, C16.1, C17.1, C19.1, C2.1, C23.1, C25.1, C26.1, C2\2.1, C30.1, F1.2, IC2.VDD_(A), IC3.VDD_(A), R10.2, R117.2, R118.2, R119.2, R120.2, R121.2, R122.2, R22.2, R23.2, R30.2, R31.2, R33.2, R35.2, R37.2, R39.2, R41.2, R42.2, R45.2, R88.1, R90.1, SJ1.2, SJ_A1.1, TP100.TP, TP36.TP, TP41.TP, TP44.TP, TP5.TP, TP63.TP, U$4.VDD3.3, U10.VDD, U11.VDD, U12.V++, U14.VCC1, U18.AVDD, U18.VREF_IN, U2.+VIN, U3.VCC1, U4.VCC1, U6.+VIN, U8.+VIN, U9.VDD
- net GND: no longer C1.2, C10.2, C11.2, C13.2, C14.2, C15.2, C16.2, C17.2, C19.2, C2.2, C21.2, C22.2, C23.2, C25.2, C26.2, C2\2.2, C30.2, C5.2, C70.2, C73.2, C74.2, C76.2, C77.2, C79.2, C80.2, C82.2, C83.2, C85.2, C86.2, C88.2, D1.P$1, D2.C, D3.C, D4.C, D8.C, IC2.VSS, IC3.VSS, J2.GND, J3.GND, PAD10.P, PAD14.P, PAD9.P, R13.2, R16.2, R20.1, R24.2, R28.1, R48.2, R89.1, SJ_A2.1, T1.GND, T2.GND, T3.S, T4.S, TP101.TP, TP106.TP, TP107.TP, TP114.TP, TP119.TP, TP124.TP, TP129.TP, TP134.TP, TP139.TP, TP3.TP, TP37.TP, TP40.TP, TP45.TP, TP61.TP, U$25.GND, U$26.GND, U$27.GND, U$28.GND, U$29.GND, U$3.2, U$3.3, U$30.GND, U$4.DGND, U$5.CHASIS, U$6.PIN4, U10.VSS, U11.VSS, U12.CTRL/TEST, U12.GND, U14.GND1, U17.GND, U17.TAB, U18.GND, U2.-VIN, U3.GND1, U4.GND1, U6.-VIN, U8.-VIN, U9.ADDR, U9.GND, U9.NWAKE
- net SC0: no longer IC2.SCL, R23.1
- net SC1: no longer IC3.SCL, R31.1
- net SC2: no longer TP1.TP, TP39.TP, TP43.TP, TP7.TP, U10.SCL, U11.SCL, U12.RX/SCL, U9.SCL
- net SC3: no longer U18.SCL
- net SC4: no longer PAD13.P
- net SC6: no longer R33.1, R37.1, R41.1, U14.SCL1, U3.SCL1, U4.SCL1
- net SCL: no longer U$4.I2C2_SCL
- net SD0: no longer IC2.SDA, R22.1
- net SD1: no longer IC3.SDA, R30.1
- net SD2: no longer TP2.TP, TP38.TP, TP42.TP, TP6.TP, U10.SDA, U11.SDA, U12.TX/SDA, U9.SDA
- net SD3: no longer U18.SDA
- net SD4: no longer PAD12.P
- net SD6: no longer R35.1, R39.1, R45.1, U14.SDA1, U3.SDA1, U4.SDA1
- net SDA: no longer U$4.I2C_SDA
Other:
- note added: "Example"
- note removed: "24V Indicator LED"
- note removed: "24V Input Power Conditioning"
- note removed: "3.3V Enable Jumper"
- note removed: "3.3V Indicator LED"
- note removed: "3.3V Isolator"
- note removed: "3.3V@400mA Regulator"
- note removed: "5-26V to 3.3V@400mA Regulator w/3v3 Enable, Indicator LED & Fuse"
- note removed: "5V Indicator LED"
- note removed: "6 Channel 4 LED Series"
- note removed: "8-Channel 8-Bit I2C DAC"
- note removed: "Atlas Sensor Port"
- note removed: "Atlas Stamp"
- note removed: "BNC Connector"
- note removed: "CCS811 CO2 Sensor"
- note removed: "Connectors"
- note removed: "Constant Current Regulator"
- note removed: "DAC Address Set"
- note removed: "DAC HW Enable"
- note removed: "DAC Signal Pullups"
- note removed: "HTU20D(F) Temp / Humidity Sensor"
- note removed: "I2C Isolator"
- note removed: "I2C Multiplexer"
- note removed: "Indicator LEDs"
- note removed: "LED Buck Driver up to 1.5A output"
- note removed: "Note - I2C Address is 0x40"
- note removed: "Note: - I2C Addr = 0x5A if ADDR is LOW - I2C Addr = 0x5B if ADDR is HIGH - PWM & Sense must be connected together - Pull-up and decouple nReset to avoid erroneous noise-induced resets"
- note removed: "Notes - I2C Address is 0x40"
- note removed: "Notes - See app note p.6 for i2c details - SDA has internal 4.7k pullup - SCL needs external 4.7k pullup - For I2C Comm, ground Ctrl/Test - I2C address default is 0x15"
- note removed: "Notes: - GND !LDAC! for syncronous mode - Broadcast I2C Addr = 0x47 - ADDR0=Low, I2C Addr=0x48 - ADDR0=High, I2C Addr=0x4A - ADDR0=Float, I2C Addr=0x4C"
- note removed: "Power Features"
- note removed: "RJ45 and Buffer SD0 & SC0"
- note removed: "RJ45 and Buffer SD1 & SC1"
- note removed: "SHT25 Temp / Humidity"
- note removed: "T6713 CO2 Sensor"
- note removed: "Testpads"
- note removed: "USB Control"
