File: prj/gpio/ADC5.sch (EAGLE design)
At the start: 147 parts, among them IC1 PCA9615DP, J1 54602-908LF, J2 PJ-036AH, U1 R-78E5.0-1.0, U2 LM2937-3.3V, U4 DAC5578

Commit message: added fermentaboard, etc
Parts:
- removed 0, 1, 2, 3, 4, 5, 6, 7, LSP1, LSP10, LSP11, LSP12, LSP13, LSP14, LSP15, LSP16, LSP17, LSP18, LSP19, LSP2, LSP20, LSP21, LSP22, LSP23, LSP24, LSP26, LSP27, LSP28, LSP29, LSP3, LSP30, LSP31, LSP32, LSP33, LSP34, LSP35, LSP36, LSP37, LSP38, LSP39, LSP4, LSP40, LSP41, LSP42, LSP43, LSP44, LSP45, LSP46, LSP47, LSP48, LSP49, LSP5, LSP6, LSP7, LSP8, LSP9: LSP13, solpad:LSP13
- added SV2, SV3: (no value), con-lstb:MA08-2
- added SV4, SV5: (no value), con-lstb:MA06-2
Connections:
- net +3V3: now also SV2.1, SV2.11, SV2.13, SV2.15, SV2.3, SV2.5, SV2.7, SV2.9, SV4.1, SV4.11, SV4.3, SV4.5, SV4.7, SV4.9; no longer LSP10.MP, LSP11.MP, LSP12.MP, LSP13.MP, LSP14.MP, LSP15.MP, LSP16.MP, LSP38.MP, LSP39.MP, LSP40.MP, LSP41.MP, LSP42.MP, LSP43.MP, LSP9.MP
- net +5V: now also SV2.10, SV2.12, SV2.14, SV2.16, SV2.2, SV2.4, SV2.6, SV2.8, SV4.10, SV4.12, SV4.2, SV4.4, SV4.6, SV4.8; no longer LSP17.MP, LSP18.MP, LSP19.MP, LSP20.MP, LSP21.MP, LSP22.MP, LSP23.MP, LSP24.MP, LSP44.MP, LSP45.MP, LSP46.MP, LSP47.MP, LSP48.MP, LSP49.MP
- net DIM1: now also SV5.11; no longer LSP31.MP
- net DIM2: now also SV5.9; no longer LSP30.MP
- net DIM3: now also SV5.7; no longer LSP29.MP
- net DIM4: now also SV5.5; no longer LSP28.MP
- net DIM5: now also SV5.3; no longer LSP27.MP
- net DIM6: now also SV5.1; no longer LSP26.MP
- net GND: now also SV3.10, SV3.12, SV3.14, SV3.16, SV3.2, SV3.4, SV3.6, SV3.8, SV5.10, SV5.12, SV5.2, SV5.4, SV5.6, SV5.8; no longer LSP1.MP, LSP2.MP, LSP3.MP, LSP32.MP, LSP33.MP, LSP34.MP, LSP35.MP, LSP36.MP, LSP37.MP, LSP4.MP, LSP5.MP, LSP6.MP, LSP7.MP, LSP8.MP
- net IN0: now also SV3.7; no longer 0.MP
- net IN1: now also SV3.5; no longer 1.MP
- net IN2: now also SV3.3; no longer 2.MP
- net IN3: now also SV3.1; no longer 3.MP
- net IN4: now also SV3.15; no longer 4.MP
- net IN5: now also SV3.13; no longer 5.MP
- net IN6: now also SV3.11; no longer 6.MP
- net IN7: now also SV3.9; no longer 7.MP
