File: prj/light-controller/v4.0/light_controller.brd (EAGLE design)
At the start: 121.2 x 91.4 mm, 204 parts, among them J2 PJ-036AH, J4 54602-908LF, J7 I2C-HEADER, J8 54602-908LF, Q1 MMBT2222A, Q2 MMBT2222A, Q3 MMBT2222A, Q4 MMBT2222A, Q5 MMBT2222A, Q6 MMBT2222A, Q7 MMBT2222A, Q8 MMBT2222A, U11 PCA9615, U13 LM2937-3.3V, U17 R-78E5.0-1.0, U7 DAC5578

Commit message: Added readme to RPI adapter
RPI to BBB socket adapter, v1.0 has incorrect wiring
Parts:
- removed J7: I2C-HEADER, openag-connectors:HEADER-I2C
- removed TP40, TP41: TPTP04R, openag-testpads:TP04R
- added CH1-1, CH1-2, CH1-3, CH1-4, CH1-5, CH1-6, CH2-1, CH2-2, CH2-3, CH2-4, CH2-5, CH2-6, CH3-1, CH3-2, CH3-3, CH3-4, CH3-5, CH3-6, CH4-1, CH4-2, CH4-3, CH4-4, CH4-5, CH4-6, CH4-7, CH4-8, CH5-1, CH5-2, CH5-3, CH5-4, CH5-5, CH5-6, CH6-1, CH6-2, CH6-3, CH6-4: XP-E, Tomaszewski:CREE-XLAMP-XP-E
- added R24, R25: (no value), rcl:R0603
- moved U$1 190.3 mm to (-37.8, -180.3)
- moved U$2 187.9 mm to (147.1, -180.3)
- moved TP52 88.4 mm to (-2.03, 39.3)
- moved J4 88.3 mm to (-28.2, 55.8)
- moved J8 88.3 mm to (-11.7, 55.8)
- moved R31 88.3 mm to (-22.6, 36.2)
- moved R32 88.3 mm to (-25.7, 37.0)
- moved R33 88.3 mm to (-27.2, 37.0)
- moved R34 88.3 mm to (-27.2, 40.1)
- moved R35 88.3 mm to (-26.4, 42.3)
- moved R36 88.3 mm to (-25.7, 40.1)
- moved R37 88.3 mm to (-16.3, 37.6)
- moved R38 88.3 mm to (-16.3, 35.6)
- moved TP42 88.3 mm to (-37.6, 56.6)
- moved TP48 88.3 mm to (-2.29, 53.0)
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Connections:
- new net N$2: CH2-4.C, CH2-4.C@1, CH2-5.A, CH2-5.A@1
- new net N$26: CH2-3.C, CH2-3.C@1, CH2-4.A, CH2-4.A@1
- new net N$30: CH2-2.C, CH2-2.C@1, CH2-3.A, CH2-3.A@1
- new net N$31: CH2-5.C, CH2-5.C@1, CH2-6.A, CH2-6.A@1
- new net N$32: CH4-4.C, CH4-4.C@1, CH4-5.A, CH4-5.A@1
- new net N$33: CH4-5.C, CH4-5.C@1, CH4-6.A, CH4-6.A@1
- new net N$34: CH4-7.A, CH4-7.A@1, CH6-4.C, CH6-4.C@1
- new net N$35: CH4-8.C, CH4-8.C@1, CH6-1.A, CH6-1.A@1
- new net N$36: CH1-4.C, CH1-4.C@1, CH1-5.A, CH1-5.A@1
- new net N$37: CH1-3.C, CH1-3.C@1, CH1-4.A, CH1-4.A@1
- new net N$38: CH2-1.C, CH2-1.C@1, CH2-2.A, CH2-2.A@1
- new net N$39: CH4-3.C, CH4-3.C@1, CH4-4.A, CH4-4.A@1
- new net N$40: CH4-2.C, CH4-2.C@1, CH4-3.A, CH4-3.A@1
- new net N$41: CH4-1.C, CH4-1.C@1, CH4-2.A, CH4-2.A@1
- new net N$42: CH6-3.C, CH6-3.C@1, CH6-4.A, CH6-4.A@1
- new net N$43: CH6-2.C, CH6-2.C@1, CH6-3.A, CH6-3.A@1
- new net N$44: CH6-1.C, CH6-1.C@1, CH6-2.A, CH6-2.A@1
- new net N$45: CH1-2.C, CH1-2.C@1, CH1-3.A, CH1-3.A@1
- new net N$46: CH1-1.C, CH1-1.C@1, CH1-2.A, CH1-2.A@1
- new net N$47: CH1-1.A, CH1-1.A@1, CH1-6.C, CH1-6.C@1
- new net N$48: CH3-4.C, CH3-4.C@1, CH3-6.A, CH3-6.A@1
- new net N$49: CH3-3.C, CH3-3.C@1, CH3-4.A, CH3-4.A@1
- new net N$50: CH3-2.C, CH3-2.C@1, CH3-3.A, CH3-3.A@1
- new net N$51: CH3-1.C, CH3-1.C@1, CH3-2.A, CH3-2.A@1
- new net N$52: CH3-1.A, CH3-1.A@1, CH3-5.C, CH3-5.C@1
- new net N$53: CH5-4.C, CH5-4.C@1, CH5-5.A, CH5-5.A@1
- new net N$54: CH5-3.C, CH5-3.C@1, CH5-4.A, CH5-4.A@1
- new net N$55: CH5-2.C, CH5-2.C@1, CH5-3.A, CH5-3.A@1
- new net N$56: CH5-1.C, CH5-1.C@1, CH5-2.A, CH5-2.A@1
- new net N$57: CH5-1.A, CH5-1.A@1, CH5-6.C, CH5-6.C@1
- new net T2: CH1-1.THERM, CH1-2.THERM, CH1-3.THERM, CH1-4.THERM, CH1-5.THERM, CH1-6.THERM, CH2-1.THERM, CH2-2.THERM, CH2-3.THERM, CH2-4.THERM, CH2-5.THERM, CH2-6.THERM, CH3-1.THERM, CH3-2.THERM, CH3-3.THERM, CH3-4.THERM, CH3-5.THERM, CH3-6.THERM, CH4-1.THERM, CH4-2.THERM, CH4-3.THERM, CH4-4.THERM, CH4-5.THERM, CH4-6.THERM, CH4-7.THERM, CH4-8.THERM, CH5-1.THERM, CH5-2.THERM, CH5-3.THERM, CH5-4.THERM, CH5-5.THERM, CH5-6.THERM, CH6-1.THERM, CH6-2.THERM, CH6-3.THERM, CH6-4.THERM, R24.1, R25.1
- net +3V3: no longer J7.3V3, TP40.1
- net +5V: no longer TP41.1
- net GND: now also R24.2, R25.2; no longer J7.GND
- net LED+: now also CH1-6.A, CH1-6.A@1
- net LED+_2: now also CH2-1.A, CH2-1.A@1
- net LED+_3: now also CH3-5.A, CH3-5.A@1
- net LED+_4: now also CH4-1.A, CH4-1.A@1
- net LED+_5: now also CH5-6.A, CH5-6.A@1
- net LED+_6: now also CH4-8.A, CH4-8.A@1
- net LED-: now also CH1-5.C, CH1-5.C@1
- net LED-_2: now also CH2-6.C, CH2-6.C@1
- net LED-_3: now also CH3-6.C, CH3-6.C@1
- net LED-_4: now also CH4-6.C, CH4-6.C@1
- net LED-_5: now also CH5-5.C, CH5-5.C@1
- net LED-_6: now also CH4-7.C, CH4-7.C@1
- net SCL: no longer J7.SCL
- net SDA: no longer J7.SDA
Routing:
- net N$31: track 0.00 -> 438.0 mm, vias 0 -> 2
- net N$33: track 0.00 -> 348.5 mm, vias 0 -> 2
- net N$42: track 0.00 -> 326.1 mm, vias 0 -> 2
- net LED-_5: track 10.9 -> 302.1 mm
- net LED-_4: track 9.58 -> 298.3 mm
- net LED-_3: track 11.6 -> 275.8 mm
- net LED-_2: track 9.84 -> 264.7 mm
- net LED-_6: track 11.3 -> 247.6 mm
- net N$51: track 0.00 -> 197.4 mm
- net N$36: track 0.00 -> 194.2 mm
- net T2: track 0.00 -> 193.1 mm, vias 0 -> 936
- net N$45: track 0.00 -> 187.7 mm, vias 0 -> 4
- net N$2: track 0.00 -> 171.5 mm
- net N$30: track 0.00 -> 164.7 mm, vias 0 -> 4
- net N$37: track 0.00 -> 161.4 mm, vias 0 -> 2
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- added copper zone on layer 1, net T2
- added copper zone on layer 16, net T2
Other:
- board size 121.2 x 91.4 mm -> 195.6 x 254.5 mm
- board text removed: "I2C Header"

Commit message: Added boards
waterbot board, relay board
Routing:
- net LED+: track 47.5 -> 289.2 mm, vias 0 -> 2
- net LED-_2: track 264.7 -> 331.3 mm, vias 0 -> 2
- net LED-_6: track 247.6 -> 306.9 mm, vias 0 -> 4
- net LED+_2: track 125.6 -> 184.2 mm, vias 0 -> 2
- net LED-_5: track 302.1 -> 344.9 mm, vias 0 -> 2
- net LED+_3: track 181.0 -> 221.9 mm
- net LED-_4: track 298.3 -> 325.0 mm, vias 0 -> 2
- net LED-: track 132.3 -> 144.9 mm, vias 0 -> 4
- net N$36: track 194.2 -> 183.4 mm
- net N$34: track 120.9 -> 116.4 mm
- net N$46: track 77.7 -> 75.5 mm
- net N$40: track 127.8 -> 129.5 mm
- net N$2: track 171.5 -> 170.1 mm
- net DIM2: track 121.6 -> 120.3 mm
- net LED-_3: track 275.8 -> 274.9 mm, vias 0 -> 2
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
Commit message: Added boards (Relay, Display, GPIO, etc)
Changed lines of the file:
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@@
 <attribute name="MPN" value="29333C" x="97.282" y="60.96" size="0.762" layer="27" display="off"/>
 <attribute name="NAME" x="93.472" y="65.024" size="0.762" layer="25"/>
+<attribute name="VALUE" x="97.79" y="59.436" size="0.762" layer="27" rot="R90"/>
 <attribute name="VALUE" x="97.79" y="59.436" size="0.762" layer="21" rot="R90"/>
-<attribute name="VALUE" x="97.79" y="59.436" size="0.762" layer="27" rot="R90"/>
 <attribute name="VENDOR" value="Digikey" x="97.282" y="60.96" size="0.762" layer="27" display="off"/>
 <attribute name="VLINK" value="https://www.digikey.com/product-detail/en/murata-power-solutions-inc/29333C/811-1138-1-ND/1924860" x="97.282" y="60.96" size="0.762" layer="27" display="off"/>
@@
 <attribute name="MPN" value="R-78E5.0-1.0" x="106.68" y="59.69" size="0.762" layer="27" rot="R270" display="off"/>
 <attribute name="NAME" x="113.284" y="65.405" size="0.762" layer="25" rot="R270"/>
+<attribute name="VALUE" x="110.236" y="62.23" size="0.762" layer="21" rot="R270"/>
 <attribute name="VALUE" x="110.236" y="62.23" size="0.762" layer="27" rot="R270"/>
-<attribute name="VALUE" x="110.236" y="62.23" size="0.762" layer="21" rot="R270"/>
 <attribute name="VENDOR" value="Digikey" x="106.68" y="59.69" size="0.762" layer="27" rot="R270" display="off"/>
 <attribute name="VLINK" value="https://www.digikey.com/product-detail/en/recom-power/R-78E5.0-1.0/945-2201-ND/4930585" x="106.68" y="59.69" size="0.762" layer="27" rot="R270" display="off"/>
@@
 <attribute name="MPN" value="54602-908LF" x="-28.194" y="55.8038" size="0.762" layer="27" rot="R180" display="off"/>
 <attribute name="NAME" x="-35.814" y="44.4373" size="0.762" layer="25"/>
+<attribute name="VALUE" x="-24.511" y="58.8518" size="0.762" layer="27" rot="R180"/>
 <attribute name="VALUE" x="-24.511" y="58.8518" size="0.762" layer="21" rot="R180"/>
-<attribute name="VALUE" x="-24.511" y="58.8518" size="0.762" layer="27" rot="R180"/>
 <attribute name="VENDOR" value="Digikey" x="-28.194" y="55.8038" size="0.762" layer="27" rot="R180" display="off"/>
 <attribute name="VLINK" value="https://www.digikey.com/product-detail/en/amphenol-fci/54602-908LF/609-1046-ND/1001360" x="-28.194" y="55.8038" size="0.762" layer="27" rot="R180" display="off"/>
@@
 <attribute name="MPN" value="54602-908LF" x="-11.684" y="55.8038" size="0.762" layer="27" rot="R180" display="off"/>
 <attribute name="NAME" x="-4.064" y="45.3263" size="0.762" layer="25" rot="R180"/>
+<attribute name="VALUE" x="-8.001" y="58.8518" size="0.762" layer="27" rot="R180"/>
 <attribute name="VALUE" x="-8.001" y="58.8518" size="0.762" layer="21" rot="R180"/>
-<attribute name="VALUE" x="-8.001" y="58.8518" size="0.762" layer="27" rot="R180"/>
 <attribute name="VENDOR" value="Digikey" x="-11.684" y="55.8038" size="0.762" layer="27" rot="R180" display="off"/>
 <attribute name="VLINK" value="https://www.digikey.com/product-detail/en/amphenol-fci/54602-908LF/609-1046-ND/1001360" x="-11.684" y="55.8038" size="0.762" layer="27" rot="R180" display="off"/>
@@
 <attribute name="MPN" value="PJ-036AH-SMT-TR" x="131.826" y="49.0982" size="1.778" layer="27" rot="R270" display="off"/>
 <attribute name="NAME" x="134.62" y="47.8282" size="0.762" layer="21"/>
+<attribute name="VALUE" x="129.54" y="55.1942" size="0.762" layer="21"/>
 <attribute name="VALUE" x="129.54" y="55.1942" size="0.762" layer="27"/>
-<attribute name="VALUE" x="129.54" y="55.1942" size="0.762" layer="21"/>
 <attribute name="VENDOR" value="Digikey" x="131.826" y="49.0982" size="1.778" layer="27" rot="R270" display="off"/>
 <attribute name="VLINK" value="https://www.digikey.com/product-detail/en/cui-inc/PJ-036AH-SMT-TR/CP-036AHPJCT-ND/1530994" x="131.826" y="49.0982" size="1.778" layer="27" rot="R270" display="off"/>
@@
 <attribute name="MPN" value="DAC5578SPW" x="64.008" y="59.182" size="1.778" layer="27" rot="R90" display="off"/>
 <attribute name="NAME" x="66.04" y="56.261" size="0.762" layer="25" rot="R180"/>
+<attribute name="VALUE" x="64.423" y="56.948" size="0.762" layer="27" rot="R90"/>
 <attribute name="VALUE" x="64.423" y="56.948" size="0.762" layer="21" rot="R90"/>
-<attribute name="VALUE" x="64.423" y="56.948" size="0.762" layer="27" rot="R90"/>
 <attribute name="VENDOR" value="Digikey" x="64.008" y="59.182" size="1.778" layer="27" rot="R90" display="off"/>
 <attribute name="VLINK" value="https://www.digikey.com/product-detail/en/texas-instruments/DAC5578SPW/296-27736-5-ND/2360827" x="64.008" y="59.182" size="1.778" layer="27" rot="R90" display="off"/>
@@
 <attribute name="MPN" value="LM2937IMP-3.3/NOPB" x="82.296" y="59.944" size="1.778" layer="27" rot="R180" display="off"/>
 <attribute name="NAME" x="84.328" y="56.134" size="0.762" layer="25" ratio="6" rot="R180"/>
+<attribute name="VALUE" x="82.042" y="62.992" size="0.762" layer="27" ratio="6" rot="R270"/>
 <attribute name="VALUE" x="82.042" y="62.992" size="0.762" layer="21" ratio="6" rot="R270"/>
-<attribute name="VALUE" x="82.042" y="62.992" size="0.762" layer="27" ratio="6" rot="R270"/>
 <attribute name="VENDOR" value="Digikey" x="82.296" y="59.944" size="1.778" layer="27" rot="R180" display="off"/>
 <attribute name="VLINK" value="https://www.digikey.com/product-detail/en/texas-instruments/LM2937IMP-3.3-NOPB/LM2937IMP-3.3-NOPBCT-ND/270742#" x="82.296" y="59.944" size="1.778" layer="27" rot="R180" display="off"/>
@@
 <attribute name="MPN" value="64900001039" x="131.826" y="39.878" size="0.762" layer="27" display="off"/>
 <attribute name="NAME" x="119.2784" y="34.0868" size="0.762" layer="25" ratio="10"/>
+<attribute name="VALUE" x="130.2004" y="43.307" size="0.762" layer="21" ratio="10"/>
 <attribute name="VALUE" x="130.2004" y="43.307" size="0.762" layer="27" ratio="10"/>
-<attribute name="VALUE" x="130.2004" y="43.307" size="0.762" layer="21" ratio="10"/>
 <attribute name="VENDOR" value="Digikey" x="131.826" y="39.878" size="0.762" layer="27" display="off"/>
 <attribute name="VLINK" value="https://www.digikey.com/product-detail/en/littelfuse-inc/64900001039/WK0011-ND/245470" x="131.826" y="39.878" size="0.762" layer="27" display="off"/>

Commit message: added fermentaboard, etc
Changed lines of the file:
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@@
 <attribute name="MPN" value="29333C" x="97.282" y="60.96" size="0.762" layer="27" display="off"/>
 <attribute name="NAME" x="93.472" y="65.024" size="0.762" layer="25"/>
+<attribute name="VALUE" x="97.79" y="59.436" size="0.762" layer="21" rot="R90"/>
 <attribute name="VALUE" x="97.79" y="59.436" size="0.762" layer="27" rot="R90"/>
-<attribute name="VALUE" x="97.79" y="59.436" size="0.762" layer="21" rot="R90"/>
 <attribute name="VENDOR" value="Digikey" x="97.282" y="60.96" size="0.762" layer="27" display="off"/>
 <attribute name="VLINK" value="https://www.digikey.com/product-detail/en/murata-power-solutions-inc/29333C/811-1138-1-ND/1924860" x="97.282" y="60.96" size="0.762" layer="27" display="off"/>
@@
 <attribute name="MPN" value="R-78E5.0-1.0" x="106.68" y="59.69" size="0.762" layer="27" rot="R270" display="off"/>
 <attribute name="NAME" x="113.284" y="65.405" size="0.762" layer="25" rot="R270"/>
+<attribute name="VALUE" x="110.236" y="62.23" size="0.762" layer="27" rot="R270"/>
 <attribute name="VALUE" x="110.236" y="62.23" size="0.762" layer="21" rot="R270"/>
-<attribute name="VALUE" x="110.236" y="62.23" size="0.762" layer="27" rot="R270"/>
 <attribute name="VENDOR" value="Digikey" x="106.68" y="59.69" size="0.762" layer="27" rot="R270" display="off"/>
 <attribute name="VLINK" value="https://www.digikey.com/product-detail/en/recom-power/R-78E5.0-1.0/945-2201-ND/4930585" x="106.68" y="59.69" size="0.762" layer="27" rot="R270" display="off"/>
@@
 <attribute name="MPN" value="54602-908LF" x="-28.194" y="55.8038" size="0.762" layer="27" rot="R180" display="off"/>
 <attribute name="NAME" x="-35.814" y="44.4373" size="0.762" layer="25"/>
+<attribute name="VALUE" x="-24.511" y="58.8518" size="0.762" layer="21" rot="R180"/>
 <attribute name="VALUE" x="-24.511" y="58.8518" size="0.762" layer="27" rot="R180"/>
-<attribute name="VALUE" x="-24.511" y="58.8518" size="0.762" layer="21" rot="R180"/>
 <attribute name="VENDOR" value="Digikey" x="-28.194" y="55.8038" size="0.762" layer="27" rot="R180" display="off"/>
 <attribute name="VLINK" value="https://www.digikey.com/product-detail/en/amphenol-fci/54602-908LF/609-1046-ND/1001360" x="-28.194" y="55.8038" size="0.762" layer="27" rot="R180" display="off"/>
@@
 <attribute name="MPN" value="54602-908LF" x="-11.684" y="55.8038" size="0.762" layer="27" rot="R180" display="off"/>
 <attribute name="NAME" x="-4.064" y="45.3263" size="0.762" layer="25" rot="R180"/>
+<attribute name="VALUE" x="-8.001" y="58.8518" size="0.762" layer="21" rot="R180"/>
 <attribute name="VALUE" x="-8.001" y="58.8518" size="0.762" layer="27" rot="R180"/>
-<attribute name="VALUE" x="-8.001" y="58.8518" size="0.762" layer="21" rot="R180"/>
 <attribute name="VENDOR" value="Digikey" x="-11.684" y="55.8038" size="0.762" layer="27" rot="R180" display="off"/>
 <attribute name="VLINK" value="https://www.digikey.com/product-detail/en/amphenol-fci/54602-908LF/609-1046-ND/1001360" x="-11.684" y="55.8038" size="0.762" layer="27" rot="R180" display="off"/>
@@
 <attribute name="MPN" value="PJ-036AH-SMT-TR" x="131.826" y="49.0982" size="1.778" layer="27" rot="R270" display="off"/>
 <attribute name="NAME" x="134.62" y="47.8282" size="0.762" layer="21"/>
+<attribute name="VALUE" x="129.54" y="55.1942" size="0.762" layer="27"/>
 <attribute name="VALUE" x="129.54" y="55.1942" size="0.762" layer="21"/>
-<attribute name="VALUE" x="129.54" y="55.1942" size="0.762" layer="27"/>
 <attribute name="VENDOR" value="Digikey" x="131.826" y="49.0982" size="1.778" layer="27" rot="R270" display="off"/>
 <attribute name="VLINK" value="https://www.digikey.com/product-detail/en/cui-inc/PJ-036AH-SMT-TR/CP-036AHPJCT-ND/1530994" x="131.826" y="49.0982" size="1.778" layer="27" rot="R270" display="off"/>
@@
 <attribute name="MPN" value="DAC5578SPW" x="64.008" y="59.182" size="1.778" layer="27" rot="R90" display="off"/>
 <attribute name="NAME" x="66.04" y="56.261" size="0.762" layer="25" rot="R180"/>
+<attribute name="VALUE" x="64.423" y="56.948" size="0.762" layer="21" rot="R90"/>
 <attribute name="VALUE" x="64.423" y="56.948" size="0.762" layer="27" rot="R90"/>
-<attribute name="VALUE" x="64.423" y="56.948" size="0.762" layer="21" rot="R90"/>
 <attribute name="VENDOR" value="Digikey" x="64.008" y="59.182" size="1.778" layer="27" rot="R90" display="off"/>
 <attribute name="VLINK" value="https://www.digikey.com/product-detail/en/texas-instruments/DAC5578SPW/296-27736-5-ND/2360827" x="64.008" y="59.182" size="1.778" layer="27" rot="R90" display="off"/>
@@
 <attribute name="MPN" value="LM2937IMP-3.3/NOPB" x="82.296" y="59.944" size="1.778" layer="27" rot="R180" display="off"/>
 <attribute name="NAME" x="84.328" y="56.134" size="0.762" layer="25" ratio="6" rot="R180"/>
+<attribute name="VALUE" x="82.042" y="62.992" size="0.762" layer="21" ratio="6" rot="R270"/>
 <attribute name="VALUE" x="82.042" y="62.992" size="0.762" layer="27" ratio="6" rot="R270"/>
-<attribute name="VALUE" x="82.042" y="62.992" size="0.762" layer="21" ratio="6" rot="R270"/>
 <attribute name="VENDOR" value="Digikey" x="82.296" y="59.944" size="1.778" layer="27" rot="R180" display="off"/>
 <attribute name="VLINK" value="https://www.digikey.com/product-detail/en/texas-instruments/LM2937IMP-3.3-NOPB/LM2937IMP-3.3-NOPBCT-ND/270742#" x="82.296" y="59.944" size="1.778" layer="27" rot="R180" display="off"/>
@@
 <attribute name="MPN" value="64900001039" x="131.826" y="39.878" size="0.762" layer="27" display="off"/>
 <attribute name="NAME" x="119.2784" y="34.0868" size="0.762" layer="25" ratio="10"/>
+<attribute name="VALUE" x="130.2004" y="43.307" size="0.762" layer="27" ratio="10"/>
 <attribute name="VALUE" x="130.2004" y="43.307" size="0.762" layer="21" ratio="10"/>
-<attribute name="VALUE" x="130.2004" y="43.307" size="0.762" layer="27" ratio="10"/>
 <attribute name="VENDOR" value="Digikey" x="131.826" y="39.878" size="0.762" layer="27" display="off"/>
 <attribute name="VLINK" value="https://www.digikey.com/product-detail/en/littelfuse-inc/64900001039/WK0011-ND/245470" x="131.826" y="39.878" size="0.762" layer="27" display="off"/>
