File: prj/pfc-edu/v4.0/PFCEDU_V4.brd (EAGLE design)
At the start: 403.9 x 355.1 mm, 268 parts, among them IC2 PCA9615DP, IC3 PCA9615DP, J1 5-1634503-1, J10 ATLAS-STAMP, J2 54602-908LF, J3 54602-908LF, J5 5-1634503-1, J6 5-1634503-1, J7 UJ2-AV-1-SMT, J8 ATLAS-STAMP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

Commit message: PFC EDU
Parts:
- removed T1: R-78E5.0-1.0, R-78E5.0-1.0:R-78E5.0-1.0
- removed T2: R-78E12.0-1.0, R-78E5.0-1.0:R-78E5.0-1.0
- added U5: R-78E12-1.0, openag-regulators:R-78E5.0-1.0
- added U7: R-78E5.0-1.0, openag-regulators:R-78E5.0-1.0
Connections:
- net +12V: now also U5.3; no longer T2.3
- net +24V: now also U5.1, U7.1; no longer T1.1, T2.1
- net +5V: now also U7.3; no longer T1.3
- net GND: now also U5.2, U7.2; no longer T1.2, T2.2
Routing:
- net +24V: track 859.6 -> 874.7 mm

Commit message: PFC EDU
Airwire, LED+ connection ch1
Parts:
- U$3: device PJ-036ah:PJ-036AH -> openag-connectors:BARREL-JACK-PJ-036AH
Routing:
- net LED+: track 4.38 -> 11.4 mm
- net ISO_SCL_2: track 18.6 -> 19.8 mm
Changed lines of the file:
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@@
 </layers>
 <board>
-<fusionsync huburn="a.cGVyc29uYWw6dWUyZDQ5ZWNm" projecturn="a.cGVyc29uYWw6dWUyZDQ5ZWNmIzIwMTgwODI3MTQ1NzkzNzAx" f3durn="urn:adsk.wipprod:dm.lineage:A54xREN7THWxmwrWM6qwpw" pcbguid="4216efb9-2f54-44b7-b09a-7bcfc6d0badd" lastpulledtime="2018-02-02T18:34:31Z" lastsyncedchangeguid="78ec3fee-b9e6-7f76-2271-f597d7512f37"/>
+<fusionsync huburn="a.cGVyc29uYWw6dWUyZDQ5ZWNm" projecturn="a.cGVyc29uYWw6dWUyZDQ5ZWNmIzIwMTgwODI3MTQ1NzkzNzAx" f3durn="urn:adsk.wipprod:dm.lineage:A54xREN7THWxmwrWM6qwpw" pcbguid="4216efb9-2f54-44b7-b09a-7bcfc6d0badd" lastpulledtime="2018-02-02T18:34:31Z" lastsyncedchangeguid="64e18597-f7a9-e501-604d-8baf1b858176"/>
 <plain>
 <wire x1="151.6226875" y1="284.734" x2="0" y2="284.734" width="0" layer="109"/>
@@
 <attribute name="VPN" value="311-100GRCT-ND" x="34.0461625" y="246.64161875" size="1.778" layer="27" rot="R90" display="off"/>
 </element>
-<element name="U$3" library="PJ-036ah" package="PJ-036AH" value="PJ-036AH" x="278.17318125" y="34.8589625" rot="R180"/>
+<element name="U$3" library="openag-connectors" library_urn="urn:adsk.eagle:library:4908154" package="BARREL-JACK-PJ-036AH" package3d_urn="urn:adsk.eagle:package:4908246/2" value="PJ-036AH" x="278.17318125" y="34.8589625" rot="R180">
+<attribute name="MANUFACTURER" value="CUI Inc." x="278.17318125" y="34.8589625" size="1.778" layer="27" rot="R180" display="off"/>
+<attribute name="MPN" value="PJ-036AH-SMT-TR" x="278.17318125" y="34.8589625" size="1.778" layer="27" rot="R180" display="off"/>
+<attribute name="VALUE" value="PJ-036AH" x="278.17318125" y="34.8589625" size="1.778" layer="27" rot="R180" display="off"/>
+<attribute name="VENDOR" value="Digikey" x="278.17318125" y="34.8589625" size="1.778" layer="27" rot="R180" display="off"/>
+<attribute name="VLINK" value="https://www.digikey.com/product-detail/en/cui-inc/PJ-036AH-SMT-TR/CP-036AHPJCT-ND/1530994" x="278.17318125" y="34.8589625" size="1.778" layer="27" rot="R180" display="off"/>
+<attribute name="VPN" value="CP-036AHPJCT-ND" x="278.17318125" y="34.8589625" size="1.778" layer="27" rot="R180" display="off"/>
+</element>
 <element name="U$9" library="openag-frames" package="OPENAG-LOGO-750-MIL" value="" x="140.07338125" y="3.0835625"/>
 <element name="U9" library="openag-sensors" library_urn="urn:adsk.eagle:library:4911564" package="CCS811" package3d_urn="urn:adsk.eagle:package:4911589/1" value="CCS811" x="47.3608375" y="105.91038125">
@@
 <element name="PAD13" library="wirepad" library_urn="urn:adsk.eagle:library:412" package="SMD1,27-2,54" package3d_urn="urn:adsk.eagle:package:30839/1" value="" x="30.226" y="209.804" rot="R90"/>
 <element name="PAD14" library="wirepad" library_urn="urn:adsk.eagle:library:412" package="SMD1,27-2,54" package3d_urn="urn:adsk.eagle:package:30839/1" value="" x="30.226" y="206.756" rot="R90"/>
-<element name="U$4" library="openag-connectors" library_urn="urn:adsk.eagle:library:4908154" package="23PINHEADERSMD" package3d_urn="urn:adsk.eagle:package:4908238/1" value="BBB_SMD" x="275.082" y="177.038" rot="R90"/>
+<element name="U$4" library="openag-connectors" library_urn="urn:adsk.eagle:library:4908154" package="23PINHEADERSMD" package3d_urn="urn:adsk.eagle:package:4908238/3" value="BBB_SMD" x="275.082" y="177.038" rot="R90"/>
 <element name="R48" library="rcl" library_urn="urn:adsk.eagle:library:334" package="R0805W" package3d_urn="urn:adsk.eagle:package:23537/1" value="" x="269.24" y="263.906" rot="R180">
 <attribute name="SPICEPREFIX" value="R" x="269.24" y="263.906" size="1.778" layer="27" rot="R180" display="off"/>
@@
 <wire x1="33.909" y1="8.001" x2="33.655" y2="7.747" width="0.3048" layer="1"/>
 <contactref element="U4" pad="1"/>
-<wire x1="15.8242" y1="250.571" x2="14.605" y2="250.571" width="0.3048" layer="1"/>
 <contactref element="U14" pad="1"/>
+<wire x1="15.8242" y1="250.571" x2="14.605" y2="250.571" width="0.6096" layer="1"/>
 <wire x1="48.4204375" y1="104.70078125" x2="48.4108375" y2="104.71038125" width="0" layer="19" extent="1-1"/>
 <wire x1="245.999" y1="277.5458" x2="245.999" y2="278.511" width="0" layer="19" extent="1-1"/>
@@
 <via x="32.258" y="244.094" extent="1-16" drill="0.35"/>
 <wire x1="32.258" y1="244.094" x2="32.512" y2="243.84" width="0.3048" layer="16"/>
-<wire x1="32.512" y1="243.84" x2="46.228" y2="243.84" width="0.3048" layer="16"/>
+<wire x1="41.148" y1="243.84" x2="32.512" y2="243.84" width="0.3048" layer="16"/>
 <via x="46.228" y="243.84" extent="1-16" drill="0.35"/>
 <contactref element="PAD11" pad="1"/>
+<wire x1="46.228" y1="243.84" x2="43.18" y2="243.84" width="0.3048" layer="16"/>
 <wire x1="30.226" y1="216.916" x2="30.226" y2="221.996" width="0.8128" layer="1"/>
 <via x="30.226" y="221.996" extent="1-16" drill="0.35"/>
@@
 <wire x1="45.88058125" y1="262.18399375" x2="45.88058125" y2="271.43258125" width="0.6096" layer="1"/>
 <wire x1="45.88058125" y1="271.43258125" x2="45.974" y2="271.526" width="0.6096" layer="1"/>
+<wire x1="43.18" y1="243.84" x2="41.148" y2="243.84" width="0.6096" layer="16"/>
 </signal>
 <signal name="N$12">
@@
 <wire x1="255.231" y1="157.734" x2="255.396" y2="157.899" width="0.6096" layer="1"/>
 <wire x1="255.396" y1="157.899" x2="255.396" y2="159.7265" width="0.6096" layer="1"/>
+<wire x1="255.231" y1="157.734" x2="255.231" y2="156.757" width="0.3048" layer="1"/>
+<wire x1="255.231" y1="156.757" x2="255.524" y2="156.464" width="0.3048" layer="1"/>
+<wire x1="255.524" y1="156.464" x2="256.794" y2="156.464" width="0.3048" layer="1"/>
+<wire x1="256.794" y1="156.464" x2="257.81" y2="157.48" width="0.3048" layer="1"/>
+<wire x1="257.81" y1="157.48" x2="257.81" y2="160.0225" width="0.3048" layer="1"/>
+<wire x1="257.81" y1="160.0225" x2="257.556" y2="160.2765" width="0.3048" layer="1"/>
 </signal>
 <signal name="VSET_2">
@@
 <wire x1="35.7124" y1="12.0904" x2="32.1564" y2="12.0904" width="0.3048" layer="1"/>
 <wire x1="36.449" y1="12.827" x2="35.7124" y2="12.0904" width="0.3048" layer="1"/>
-<wire x1="36.449" y1="15.367" x2="36.83" y2="15.748" width="0.3048" layer="1"/>
+<wire x1="36.449" y1="15.367" x2="36.576" y2="15.494" width="0.3048" layer="1"/>
+<wire x1="36.576" y1="15.494" x2="36.83" y2="15.748" width="0.3048" layer="1"/>
 <wire x1="36.83" y1="15.748" x2="38.354" y2="15.748" width="0.3048" layer="1"/>
 <wire x1="38.354" y1="15.748" x2="38.862" y2="15.24" width="0.3048" layer="1"/>
@@
 <contactref element="U3" pad="6"/>
 <wire x1="36.449" y1="14.1478" x2="36.449" y2="12.827" width="0.3048" layer="1"/>
-<wire x1="36.449" y1="14.1478" x2="36.449" y2="15.367" width="0" layer="19" extent="1-1"/>
+<wire x1="36.449" y1="14.1478" x2="36.449" y2="15.367" width="0.3048" layer="1"/>
 </signal>
 <signal name="ISO_SDA_2">
@@
 <wire x1="249.174" y1="271.868" x2="245.999" y2="271.868" width="0.5588" layer="1"/>
 <wire x1="244.2718" y1="269.4178" x2="237.3122" y2="269.4178" width="0.5588" layer="1"/>
-<wire x1="245.999" y1="271.145" x2="244.2718" y2="269.4178" width="0.5588" layer="1"/>
+<wire x1="244.2718" y1="269.4178" x2="245.618" y2="270.764" width="0.5588" layer="1"/>
 <wire x1="253.072" y1="271.868" x2="250.444" y2="271.868" width="0.5588" layer="1"/>
 <wire x1="250.444" y1="271.868" x2="249.174" y2="271.868" width="0.5588" layer="1"/>
@@
 <wire x1="250.4598" y1="273.558" x2="250.4598" y2="274.828" width="0.5588" layer="1"/>
 <contactref element="U14" pad="8"/>
-<wire x1="245.999" y1="272.6182" x2="245.999" y2="271.145" width="0.3048" layer="1"/>
+<wire x1="245.999" y1="271.145" x2="245.999" y2="272.6182" width="0.6096" layer="1"/>
+<wire x1="245.618" y1="270.764" x2="245.999" y2="271.145" width="0.6096" layer="1"/>
 <wire x1="245.999" y1="271.145" x2="245.999" y2="271.868" width="0" layer="19" extent="1-1"/>
 </signal>

Commit message: PFCEDUandLightController
PFCEDU
Connections:
- removed net LED+: C72.2, RS2.1, U$25.4
- net CH1+: now also C72.2, RS2.1, U$25.4
Routing:
- net CH1+: track 120.1 -> 131.5 mm
- net LED+: track 11.4 -> 0.00 mm
- net ISO_3V3_2: track 32.2 -> 33.4 mm
Other:
- outline, holes or cut-outs redrawn
Changed lines of the file:
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@@
 <drawing>
 <settings>
-<setting alwaysvectorfont="yes"/>
+<setting alwaysvectorfont="no"/>
 <setting keepoldvectorfont="yes"/>
 <setting verticaltext="up"/>
@@
 <layer number="29" name="tStop" color="7" fill="3" visible="no" active="yes"/>
 <layer number="30" name="bStop" color="7" fill="6" visible="no" active="yes"/>
-<layer number="31" name="tCream" color="7" fill="4" visible="no" active="yes"/>
+<layer number="31" name="tCream" color="7" fill="4" visible="yes" active="yes"/>
 <layer number="32" name="bCream" color="7" fill="5" visible="no" active="yes"/>
 <layer number="33" name="tFinish" color="6" fill="3" visible="no" active="yes"/>
@@
 <wire x1="284.734" y1="284.734" x2="224.536" y2="284.734" width="0" layer="109"/>
 <wire x1="224.7269875" y1="284.734" x2="189.98856875" y2="284.790740625" width="0" layer="109"/>
-<circle x="275.203146875" y="8.548271875" radius="3.175" width="0.025" layer="20"/>
+<circle x="276.981146875" y="9.310271875" radius="5.08" width="0.025" layer="20"/>
 <circle x="119.747796875" y="235.69623125" radius="1.1994" width="0.025" layer="20"/>
 <circle x="95.75750625" y="259.684240625" radius="1.1994" width="0.025" layer="20"/>
@@
 <wire x1="284.734" y1="284.734" x2="284.734" y2="0" width="0.1524" layer="20"/>
 <wire x1="284.734" y1="0" x2="0" y2="0" width="0.1524" layer="20"/>
+<rectangle x1="280.416" y1="26.416" x2="281.178" y2="29.972" layer="31"/>
+<rectangle x1="281.432" y1="25.4" x2="283.464" y2="26.162" layer="31"/>
+<rectangle x1="280.67" y1="39.624" x2="281.432" y2="43.18" layer="31"/>
+<rectangle x1="281.686" y1="43.688" x2="283.464" y2="44.196" layer="31"/>
 </plain>
 <attributes>
@@
 <wire x1="253.8397" y1="151.1602" x2="254.6985" y2="152.019" width="0.6096" layer="1"/>
 <wire x1="235.8723" y1="151.1602" x2="253.8397" y2="151.1602" width="0.6096" layer="1"/>
+<contactref element="U$25" pad="4"/>
+<contactref element="C72" pad="2"/>
+<contactref element="RS2" pad="1"/>
+<wire x1="255.396" y1="159.7265" x2="256.6885" y2="159.7265" width="0.6096" layer="1"/>
+<wire x1="256.6885" y1="159.7265" x2="257.556" y2="160.2765" width="0.6096" layer="1"/>
+<wire x1="255.231" y1="157.734" x2="255.396" y2="157.899" width="0.6096" layer="1"/>
+<wire x1="255.396" y1="157.899" x2="255.396" y2="159.7265" width="0.6096" layer="1"/>
+<wire x1="255.231" y1="157.734" x2="255.231" y2="156.757" width="0.3048" layer="1"/>
+<wire x1="255.231" y1="156.757" x2="255.524" y2="156.464" width="0.3048" layer="1"/>
+<wire x1="255.524" y1="156.464" x2="256.794" y2="156.464" width="0.3048" layer="1"/>
+<wire x1="256.794" y1="156.464" x2="257.81" y2="157.48" width="0.3048" layer="1"/>
+<wire x1="257.81" y1="157.48" x2="257.81" y2="160.0225" width="0.3048" layer="1"/>
+<wire x1="257.81" y1="160.0225" x2="257.556" y2="160.2765" width="0.3048" layer="1"/>
 </signal>
 <signal name="CH1-">
@@
 </polygon>
 </signal>
-<signal name="LED+">
-<contactref element="U$25" pad="4"/>
-<contactref element="C72" pad="2"/>
-<contactref element="RS2" pad="1"/>
-<wire x1="255.396" y1="159.7265" x2="256.6885" y2="159.7265" width="0.6096" layer="1"/>
-<wire x1="256.6885" y1="159.7265" x2="257.556" y2="160.2765" width="0.6096" layer="1"/>
-<wire x1="255.231" y1="157.734" x2="255.396" y2="157.899" width="0.6096" layer="1"/>
-<wire x1="255.396" y1="157.899" x2="255.396" y2="159.7265" width="0.6096" layer="1"/>
-<wire x1="255.231" y1="157.734" x2="255.231" y2="156.757" width="0.3048" layer="1"/>
-<wire x1="255.231" y1="156.757" x2="255.524" y2="156.464" width="0.3048" layer="1"/>
-<wire x1="255.524" y1="156.464" x2="256.794" y2="156.464" width="0.3048" layer="1"/>
-<wire x1="256.794" y1="156.464" x2="257.81" y2="157.48" width="0.3048" layer="1"/>
-<wire x1="257.81" y1="157.48" x2="257.81" y2="160.0225" width="0.3048" layer="1"/>
-<wire x1="257.81" y1="160.0225" x2="257.556" y2="160.2765" width="0.3048" layer="1"/>
-</signal>
 <signal name="VSET_2">
 <contactref element="U$26" pad="3"/>
@@
 <contactref element="U3" pad="8"/>
 <wire x1="33.909" y1="15.367" x2="33.909" y2="14.644" width="0.3048" layer="1"/>
-<wire x1="33.909" y1="14.644" x2="33.909" y2="14.1478" width="0" layer="19" extent="1-1"/>
+<wire x1="33.909" y1="14.1478" x2="33.909" y2="15.367" width="0.3048" layer="1"/>
 </signal>
 <signal name="PRB_2">
